File: hardware/servo-sigma-48v/mcu.sch (KiCad schematic (older format))
At the start: 40 parts, among them J2 CONN_02X05, J5 CONN_01X06, J6 629_105_150_921, U5 STM32F411RETx, Y1 ABM3-8.000MHZ-D2Y-T

Commit message: Finished routing of the servo controller
Parts:
- removed J5: CONN_01X06, symbol conn:CONN_01X06
- removed R17, R20, R28, R30, R38, R40: 10, Resistors_SMD:R_0603, symbol device:R
- added J5: CONN_01X05, Pin_Headers:Pin_Header_Angled_1x05_Pitch2.54mm, symbol conn:CONN_01X05
Connections:
- net labels added: AUX_H, AUX_L, IR_FB
- wire segments 203 -> 198
- no-connect marks 28 -> 20
Changed lines of the file:
@@
 $EndComp
 NoConn ~ 7150 4150
-NoConn ~ 7150 4950
-NoConn ~ 7150 5050
 NoConn ~ 7150 5350
 NoConn ~ 7150 5450
 NoConn ~ 7150 5550
-NoConn ~ 12950 3350
 NoConn ~ 12950 4650
-NoConn ~ 12950 5250
-NoConn ~ 12950 5350
 NoConn ~ 12950 5450
 NoConn ~ 12950 5550
@@
 	12950 4650 13350 4650
 Wire Wire Line
-	12950 5250 13350 5250
-Wire Wire Line
-	12950 5350 13350 5350
-Wire Wire Line
 	12950 5450 13350 5450
 Wire Wire Line
@@
 	13350 3150 12950 3150
 Wire Wire Line
-	13350 3250 12950 3250
-Wire Wire Line
-	13350 3350 12950 3350
-Wire Wire Line
 	13350 4050 12950 4050
 Wire Wire Line
@@
 Wire Wire Line
 	6750 4850 7150 4850
-Wire Wire Line
-	6750 4950 7150 4950
-Wire Wire Line
-	6750 5050 7150 5050
 Wire Wire Line
 	7150 5150 6750 5150
@@
 	10500 1550 10500 1800
 Connection ~ 11000 1800
-NoConn ~ 7150 5750
-NoConn ~ 7150 5850
 Text Label 6750 5750 0    60   ~ 0
 PC14
 Text Label 6750 5850 0    60   ~ 0
 PC15
-Wire Wire Line
-	7150 5750 6750 5750
-Wire Wire Line
-	7150 5850 6750 5850
 Wire Wire Line
 	5600 3900 5600 3850
@@
 Connection ~ 5850 2800
 $Comp
-L device:R R40
-U 1 1 5AB8EC9A
-P 13900 3550
-F 0 "R40" V 13850 3700 50  0000 C CNN
-F 1 "10" V 13900 3550 50  0000 C CNN
-F 2 "Resistors_SMD:R_0603" V 13830 3550 50  0001 C CNN
-F 3 "http://www.yageo.com/documents/recent/PYu-RC_Group_51_RoHS_L_8.pdf" H 13900 3550 50  0001 C CNN
-F 4 "311-10.0HRCT-ND" V 13900 3550 60  0001 C CNN "Part"
-F 5 "DigiKey" V 13900 3550 60  0001 C CNN "Provider"
-	1    13900 3550
-	0    -1   -1   0
-$EndComp
-$Comp
-L device:R R30
-U 1 1 59FA59CB
-P 13900 3650
-F 0 "R30" V 13850 3800 50  0000 C CNN
-F 1 "10" V 13900 3650 50  0000 C CNN
-F 2 "Resistors_SMD:R_0603" V 13830 3650 50  0001 C CNN
-F 3 "http://www.yageo.com/documents/recent/PYu-RC_Group_51_RoHS_L_8.pdf" H 13900 3650 50  0001 C CNN
-F 4 "311-10.0HRCT-ND" V 13900 3650 60  0001 C CNN "Part"
-F 5 "DigiKey" V 13900 3650 60  0001 C CNN "Provider"
-	1    13900 3650
-	0    -1   -1   0
-$EndComp
-$Comp
-L device:R R20
-U 1 1 59FA5A1B
-P 13900 3750
-F 0 "R20" V 13850 3900 50  0000 C CNN
-F 1 "10" V 13900 3750 50  0000 C CNN
-F 2 "Resistors_SMD:R_0603" V 13830 3750 50  0001 C CNN
-F 3 "http://www.yageo.com/documents/recent/PYu-RC_Group_51_RoHS_L_8.pdf" H 13900 3750 50  0001 C CNN
-F 4 "311-10.0HRCT-ND" V 13900 3750 60  0001 C CNN "Part"
-F 5 "DigiKey" V 13900 3750 60  0001 C CNN "Provider"
-	1    13900 3750
-	0    -1   -1   0
-$EndComp
-$Comp
-L device:R R38
-U 1 1 59FA5A6D
-P 13900 5650
-F 0 "R38" V 13850 5800 50  0000 C CNN
-F 1 "10" V 13900 5650 50  0000 C CNN
-F 2 "Resistors_SMD:R_0603" V 13830 5650 50  0001 C CNN
-F 3 "http://www.yageo.com/documents/recent/PYu-RC_Group_51_RoHS_L_8.pdf" H 13900 5650 50  0001 C CNN
-F 4 "311-10.0HRCT-ND" V 13900 5650 60  0001 C CNN "Part"
-F 5 "DigiKey" V 13900 5650 60  0001 C CNN "Provider"
-	1    13900 5650
-	0    -1   -1   0
-$EndComp
-$Comp
-L device:R R28
-U 1 1 5AB8EC9E
-P 13900 5750
-F 0 "R28" V 13850 5900 50  0000 C CNN
-F 1 "10" V 13900 5750 50  0000 C CNN
-F 2 "Resistors_SMD:R_0603" V 13830 5750 50  0001 C CNN
-F 3 "http://www.yageo.com/documents/recent/PYu-RC_Group_51_RoHS_L_8.pdf" H 13900 5750 50  0001 C CNN
-F 4 "311-10.0HRCT-ND" V 13900 5750 60  0001 C CNN "Part"
-F 5 "DigiKey" V 13900 5750 60  0001 C CNN "Provider"
-	1    13900 5750
-	0    -1   -1   0
-$EndComp
-$Comp
-L device:R R17
-U 1 1 5AB8EC9F
-P 13900 5850
-F 0 "R17" V 13850 6000 50  0000 C CNN
-F 1 "10" V 13900 5850 50  0000 C CNN
-F 2 "Resistors_SMD:R_0603" V 13830 5850 50  0001 C CNN
-F 3 "http://www.yageo.com/documents/recent/PYu-RC_Group_51_RoHS_L_8.pdf" H 13900 5850 50  0001 C CNN
-F 4 "311-10.0HRCT-ND" V 13900 5850 60  0001 C CNN "Part"
-F 5 "DigiKey" V 13900 5850 60  0001 C CNN "Provider"
-	1    13900 5850
-	0    -1   -1   0
-$EndComp
-Wire Wire Line
-	14950 3550 14050 3550
-Wire Wire Line
-	14950 3650 14050 3650
-Wire Wire Line
-	14950 3750 14050 3750
-Wire Wire Line
-	14950 5650 14050 5650
-Wire Wire Line
-	14950 5750 14050 5750
-Wire Wire Line
-	14950 5850 14050 5850
-$Comp
 L device:C C32
 U 1 1 5AB8ECA0
@@
 	0    1    1    0
 $EndComp
-NoConn ~ 12950 3050
-NoConn ~ 12950 3150
-NoConn ~ 12950 3250
 NoConn ~ 7150 5150
 NoConn ~ 7150 5250
@@
 $EndComp
 Text Label 2950 6350 2    60   ~ 0
-PC13
+PA4
 $Comp
 L device:R R9
@@
 Text Label 7400 9600 0    60   ~ 0
 IC_FB
-NoConn ~ 5600 9050
-NoConn ~ 5150 10950
-$Comp
-L conn:CONN_01X06 J5
-U 1 1 5BB280E1
-P 1150 8050
-F 0 "J5" H 1150 8450 50  0000 C CNN
-F 1 "CONN_01X06" H 1150 7700 50  0000 C CNN
-F 2 "" H 1150 8050 50  0001 C CNN
-F 3 "" H 1150 8050 50  0001 C CNN
-	1    1150 8050
-	-1   0    0    -1
-$EndComp
 Text Label 2100 7800 2    60   ~ 0
 ENCODER_B
@@
 Wire Wire Line
 	1350 8200 2100 8200
-NoConn ~ 1350 8300
 $Comp
 L power:+5V #PWR?
@@
 ENCODER_B
 Wire Wire Line
-	12950 3550 13750 3550
-Wire Wire Line
-	12950 3650 13750 3650
-Wire Wire Line
-	12950 3750 13750 3750
-Wire Wire Line
 	12950 3450 13350 3450
 Wire Wire Line
@@
 NoConn ~ 12950 4450
 NoConn ~ 12950 3450
-Wire Wire Line
-	12950 5650 13750 5650
-Wire Wire Line
-	12950 5750 13750 5750
-Wire Wire Line
-	12950 5850 13750 5850
 Wire Wire Line
 	12950 4750 13350 4750
@@
 Wire Wire Line
 	12950 3950 14650 3950
+Text HLabel 6500 5050 0    60   Output ~ 0
+AUX_L
+Text HLabel 6500 4950 0    60   Output ~ 0
+AUX_H
+$Comp
+L conn:CONN_01X05 J5
+U 1 1 5BCE27D8
+P 1150 8000
+F 0 "J5" H 1150 8300 50  0000 C CNN
+F 1 "CONN_01X05" H 1150 7700 50  0000 C CNN
+F 2 "Pin_Headers:Pin_Header_Angled_1x05_Pitch2.54mm" H 1150 8000 50  0001 C CNN
+F 3 "https://www.molex.com/pdm_docs/sd/705530002_sd.pdf" H 1150 8000 50  0001 C CNN
+F 4 "WM4903-ND" H 1150 8000 50  0001 C CNN "Part"
+F 5 "DigiKey" H 1150 8000 50  0001 C CNN "Provider"
+	1    1150 8000
+	-1   0    0    -1
+$EndComp
+Wire Wire Line
+	12950 3550 14950 3550
+Wire Wire Line
+	12950 3650 14950 3650
+Wire Wire Line
+	12950 3750 14950 3750
+Wire Wire Line
+	12950 5650 14950 5650
+Wire Wire Line
+	12950 5750 14950 5750
+Wire Wire Line
+	12950 5850 14950 5850
+Text Label 8700 9700 2    60   ~ 0
+PA3
+Text HLabel 7100 9700 0    60   Input ~ 0
+IR_FB
+Wire Wire Line
+	7100 9700 8700 9700
+Text Label 14650 3250 2    60   ~ 0
+LED_WARN
+Text Label 14650 3350 2    60   ~ 0
+LED_STATUS
+NoConn ~ 7150 5650
+Wire Wire Line
+	6500 4950 7150 4950
+Wire Wire Line
+	6500 5050 7150 5050
+Wire Wire Line
+	12950 5250 13350 5250
+Wire Wire Line
+	12950 5350 13350 5350
+NoConn ~ 12950 5250
+NoConn ~ 12950 5350
+Wire Wire Line
+	12950 3350 14650 3350
+Wire Wire Line
+	12950 3250 14650 3250
+Wire Wire Line
+	6750 5750 7150 5750
+Wire Wire Line
+	6750 5850 7150 5850
+NoConn ~ 7150 5750
+NoConn ~ 7150 5850
 $EndSCHEMATC

Commit message: Updated the footprints
Parts:
- C14, C19, C24, C25, C27, C3, C30, C32, C4: footprint Capacitors_SMD:C_0603 -> Capacitor_SMD:C_0603_1608Metric; symbol device:C -> servo-sigma-48v-rescue:C-device
- C15, C28, C29, C31: footprint Capacitors_SMD:C_0805 -> Capacitor_SMD:C_0805_2012Metric; symbol device:C -> servo-sigma-48v-rescue:C-device
- D1, D4: footprint LEDs:LED_0603 -> LED_SMD:LED_0603_1608Metric; symbol device:LED -> servo-sigma-48v-rescue:LED-device
- FB1: footprint Resistors_SMD:R_0805 -> Resistor_SMD:R_0603_1608Metric
- J2: footprint Pin_Headers:Pin_Header_Straight_2x05_Pitch1.27mm -> Connector_PinHeader_1.27mm:PinHeader_2x05_P1.27mm_Vertical; symbol conn:CONN_02X05 -> servo-sigma-48v-rescue:CONN_02X05-conn
- J5: footprint Pin_Headers:Pin_Header_Angled_1x05_Pitch2.54mm -> Connector_PinHeader_2.54mm:PinHeader_1x05_P2.54mm_Horizontal; symbol conn:CONN_01X05 -> servo-sigma-48v-rescue:CONN_01X05-conn
- R1, R10, R19, R2, R3, R4, R44, R47, R5, R50, R8, R9: footprint Resistors_SMD:R_0603 -> Resistor_SMD:R_0603_1608Metric; symbol device:R -> servo-sigma-48v-rescue:R-device
- U5: footprint Housings_QFP:LQFP-64_10x10mm_Pitch0.5mm -> Package_QFP:LQFP-64_10x10mm_P0.5mm; symbol stm32:STM32F411RETx -> servo-sigma-48v-rescue:STM32F411RETx-stm32
- Y1: footprint Crystals:Crystal_SMD_Abracon_ABM3-2pin_5.0x3.2mm -> Crystal:Crystal_SMD_Abracon_ABM3-2Pin_5.0x3.2mm; symbol device:Crystal -> servo-sigma-48v-rescue:Crystal-device

Commit message: Work on sigmadrive 2.0
Parts:
- added C51, C52: 100nF 50V, Capacitor_SMD:C_0603_1608Metric, symbol servo-sigma-48v-rescue:C-device
- added J8, J9: Conn_01x03, Connector_PinHeader_2.54mm:PinHeader_1x03_P2.54mm_Horizontal, symbol Connector_Generic:Conn_01x03
- added R17, R28: 10k, Resistor_SMD:R_0603_1608Metric, symbol servo-sigma-48v-rescue:R-device
- added R20, R30: 100, Resistor_SMD:R_0603_1608Metric, symbol servo-sigma-48v-rescue:R-device
Connections:
- net labels added: SW1, SW2, USART6_RX, USART6_TX, USER_BTN
- net labels removed: CURRENT_ADC, CURRENT_FAULT
- wire segments 198 -> 208
- no-connect marks 20 -> 12
Other:
- moved on the sheet: C27, C32, J2, R2, R3, R44, Y1

Commit message: work on rs485
Parts:
- removed J5: CONN_01X05, Connector_PinHeader_2.54mm:PinHeader_1x05_P2.54mm_Horizontal, symbol servo-sigma-48v-rescue:CONN_01X05-conn
- added C5, C8: 100nF 50V, Capacitor_SMD:C_0603_1608Metric, symbol servo-sigma-48v-rescue:C-device
- added J10, J11: Conn_01x03, Connector_PinHeader_2.54mm:PinHeader_1x03_P2.54mm_Horizontal, symbol Connector_Generic:Conn_01x03
- added J5: Conn_01x05, Connector_PinHeader_2.54mm:PinHeader_1x05_P2.54mm_Horizontal, symbol Connector_Generic:Conn_01x05
- added R14, R15, R84, R85: 10k, Resistor_SMD:R_0603_1608Metric, symbol servo-sigma-48v-rescue:R-device
- added R38, R40, R86, R87: 4.7k, Resistor_SMD:R_0603_1608Metric, symbol servo-sigma-48v-rescue:R-device
- added R81, R88: 100, Resistor_SMD:R_0603_1608Metric, symbol servo-sigma-48v-rescue:R-device
- added R83, R89: 21, Resistor_SMD:R_0603_1608Metric, symbol servo-sigma-48v-rescue:R-device
- added SW1, SW2: SW_DIP_x08, Button_Switch_SMD:SW_DIP_SPSTx08_Slide_Copal_CHS-08A_W5.08mm_P1.27mm_JPin, symbol Switch:SW_DIP_x08
- added U12, U3: SN65HVD75DGKR, Package_SO:SOIC-8_3.9x4.9mm_P1.27mm, symbol Interface_UART:MAX3485
Connections:
- net labels added: A_TERM_R120, BOOT0, B_TERM_R120, ENCODER_A_CON, ENCODER_B_CON, ENCODER_B_DE, ENCODER_DE, ENCODER_DI, ENCODER_RO, ENCODER_RS485_A, ENCODER_RS485_B, ENCODER_Z_CON, RS485_DE, RS485_DI, RS485_RO, USART1_RX, USART1_TX, USB_DP_USART1_RTS
- net labels removed: ENCODER_B, ENCODER_Z, USART6_RX, USART6_TX
- wire segments 208 -> 322
- no-connect marks 12 -> 23
Other:
- moved on the sheet: C4, C51, C52, D1, D4, J8, J9, R1, R10, R17, R20, R28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

Commit message: Changed the MCU to use 100 pin
Parts:
- removed SW2: SW_DIP_x08, Button_Switch_SMD:SW_DIP_SPSTx08_Slide_Copal_CHS-08A_W5.08mm_P1.27mm_JPin, symbol Switch:SW_DIP_x08
- removed U5: STM32F411RETx, Package_QFP:LQFP-64_10x10mm_P0.5mm, symbol servo-sigma-48v-rescue:STM32F411RETx-stm32
- added C10: 2.2uF, Capacitor_SMD:C_0603_1608Metric, symbol servo-sigma-48v-rescue:C-device
- added C53, C54: 100nF 50V, Capacitor_SMD:C_0603_1608Metric, symbol servo-sigma-48v-rescue:C-device
- added J12: Conn_01x05, Connector_PinHeader_2.54mm:PinHeader_1x05_P2.54mm_Horizontal, symbol Connector_Generic:Conn_01x05
- added R90, R91, R92: 10k, Resistor_SMD:R_0603_1608Metric, symbol servo-sigma-48v-rescue:R-device
- added U5: STM32F405VGTx, Package_QFP:LQFP-100_14x14mm_P0.5mm, symbol STM32LEGACY:STM32F405VGTx
- C15: value 4.7uF 25V -> 2.2uF; footprint Capacitor_SMD:C_0805_2012Metric -> Capacitor_SMD:C_0603_1608Metric; Part 1276-2415-1-ND -> 490-10731-1-ND
Connections:
- net PB2 is gone; now on net PB1: C52.2, J9.1 (Pin_1), R28.2
- net USART_RX is gone; now on net PB7: R2.1
- net USART_TX is gone; now on net PB6: R3.1
- net USB_DP is gone; now on net PA12: R50.2
- net +5V: now also J12.1 (Pin_1)
- net AUX_H: now also U5.37 (BOOT1/PB2)
- net AUX_L: now also U5.38 (PE7/FSMC_D4/FSMC_DA4/TIM1_ETR)
- net BOOT0: now also U5.94 (BOOT0)
- net ENCODER_A: now also J5.3 (Pin_3), R91.2, U5.23 (ADC1_IN0/ADC2_IN0/ADC3_IN0/SYS_WKUP/TIM2_CH1/TIM2_ETR/TIM5_CH1/TIM8_ETR/UART4_TX/USART2_CTS/PA0); no longer SW1.13
- net ENCODER_DE: now also U5.59 (PD12/FSMC_A17/FSMC_ALE/TIM4_CH1/USART3_RTS); no longer SW1.1
- net ENCODER_DI: now also U5.55 (PD8/FSMC_D13/FSMC_DA13/USART3_TX)
- net ENCODER_RO: now also U5.56 (PD9/DAC_EXTI9/FSMC_D14/FSMC_DA14/USART3_RX)
- net GND: now also C10.1, C53.1, C54.1, J12.4 (Pin_4), U5.10 (VSS), U5.20 (VSSA), U5.27 (VSS), U5.74 (VSS), U5.99 (VSS)
- net IA_FB: now also U5.30 (ADC1_IN5/ADC2_IN5/DAC_OUT2/SPI1_SCK/TIM2_CH1/TIM2_ETR/TIM8_CH1N/USB_OTG_HS_ULPI_CK/PA5)
- net IB_FB: now also U5.31 (ADC1_IN6/ADC2_IN6/SPI1_MISO/TIM13_CH1/TIM1_BKIN/TIM3_CH1/TIM8_BKIN/PA6)
- net IC_FB: now also U5.32 (ADC1_IN7/ADC2_IN7/SPI1_MOSI/TIM14_CH1/TIM1_CH1N/TIM3_CH2/TIM8_CH1N/PA7)
- net IR_FB: now also U5.33 (ADC1_IN14/ADC2_IN14/PC4)
- net LED_STATUS: now also U5.54 (ADC1_EXTI15/ADC2_EXTI15/ADC3_EXTI15/I2S2_SD/RTC_REFIN/SPI2_MOSI/TIM12_CH2/TIM1_CH3N/TIM8_CH3N/USB_OTG_HS_DP/PB15)
- net LED_WARN: now also U5.53 (I2S2_ext_SD/SPI2_MISO/TIM12_CH1/TIM1_CH2N/TIM8_CH2N/USART3_RTS/USB_OTG_HS_DM/PB14)
- net NRST: no longer C3.2, R8.1
- net PA11: now also U5.70 (ADC1_EXTI11/ADC2_EXTI11/ADC3_EXTI11/CAN1_RX/TIM1_CH4/USART1_CTS/USB_OTG_FS_DM/PA11)
- net PA12: now also U5.71 (CAN1_TX/TIM1_ETR/USART1_RTS/USB_OTG_FS_DP/PA12)
- net PA13: now also U5.72 (SYS_JTMS-SWDIO/PA13)
- net PA14: now also U5.76 (SYS_JTCK-SWCLK/PA14)
- net PA15: now also U5.77 (ADC1_EXTI15/ADC2_EXTI15/ADC3_EXTI15/I2S3_WS/SPI1_NSS/SPI3_NSS/SYS_JTDI/TIM2_CH1/TIM2_ETR/PA15)
- net PA4: now also U5.29 (ADC1_IN4/ADC2_IN4/DAC_OUT1/I2S3_WS/SPI1_NSS/SPI3_NSS/USART2_CK/USB_OTG_HS_SOF/PA4)
- net PB1: now also U5.36 (ADC1_IN9/ADC2_IN9/TIM1_CH3N/TIM3_CH4/TIM8_CH3N/USB_OTG_HS_ULPI_D2/PB1); no longer C51.2, J8.1 (Pin_1), R17.2
- net PB12: now also U5.51 (CAN2_RX/I2C2_SMBA/I2S2_WS/SPI2_NSS/TIM1_BKIN/USART3_CK/USB_OTG_HS_ID/USB_OTG_HS_ULPI_D5/PB12); no longer C4.2, R10.2, USR1.2
- net PB3: now also U5.89 (I2S3_CK/SPI1_SCK/SPI3_SCK/SYS_JTDO-SWO/TIM2_CH2/PB3)
- net PB5: now also U5.91 (CAN2_RX/I2C1_SMBA/I2S3_SD/SPI1_MOSI/SPI3_MOSI/TIM3_CH2/USB_OTG_HS_ULPI_D7/PB5)
- net PB6: now also U5.92 (CAN2_TX/I2C1_SCL/TIM4_CH1/USART1_TX/PB6)
- net PB7: now also U5.93 (FSMC_NL/I2C1_SDA/TIM4_CH2/USART1_RX/PB7)
- net PB8: now also U5.95 (CAN1_RX/I2C1_SCL/SDIO_D4/TIM10_CH1/TIM4_CH3/PB8)
- net PC10: now also U5.78 (I2S3_CK/SDIO_D2/SPI3_SCK/UART4_TX/USART3_TX/PC10)
- net PC11: now also U5.79 (ADC1_EXTI11/ADC2_EXTI11/ADC3_EXTI11/I2S3_ext_SD/SDIO_D3/SPI3_MISO/UART4_RX/USART3_RX/PC11)
- net PC12: now also U5.80 (I2S3_SD/SDIO_CK/SPI3_MOSI/UART5_TX/USART3_CK/PC12)
- net PC13: now also U5.7 (ANTI_TAMP/RTC_AF1/PC13)
- net PC7: now also U5.64 (I2S3_MCK/SDIO_D7/TIM3_CH2/TIM8_CH2/USART6_RX/PC7)
- net PC8: now also U5.65 (SDIO_D0/TIM3_CH3/TIM8_CH3/USART6_CK/PC8)
- net PC9: now also U5.66 (DAC_EXTI9/I2C3_SDA/I2S_CKIN/RCC_MCO_2/SDIO_D1/TIM3_CH4/TIM8_CH4/PC9)
- net PD2: now also U5.83 (PD2/SDIO_CMD/TIM3_ETR/UART5_RX)
- net PWM: now also U5.63 (I2S2_MCK/SDIO_D6/TIM3_CH1/TIM8_CH1/USART6_TX/PC6)
- net PWM_AH: now also U5.40 (PE9/DAC_EXTI9/FSMC_D6/FSMC_DA6/TIM1_CH1)
- net PWM_AL: now also U5.39 (PE8/FSMC_D5/FSMC_DA5/TIM1_CH1N)
- net PWM_BH: now also U5.42 (PE11/ADC1_EXTI11/ADC2_EXTI11/ADC3_EXTI11/FSMC_D8/FSMC_DA8/TIM1_CH2)
- net PWM_BL: now also U5.41 (PE10/FSMC_D7/FSMC_DA7/TIM1_CH2N)
- net PWM_CH: now also U5.44 (PE13/FSMC_D10/FSMC_DA10/TIM1_CH3)
- net PWM_CL: now also U5.43 (PE12/FSMC_D9/FSMC_DA9/TIM1_CH3N)
- net SENSE_A: now also U5.17 (ADC1_IN12/ADC2_IN12/ADC3_IN12/I2S2_ext_SD/SPI2_MISO/USB_OTG_HS_ULPI_DIR/PC2)
- net SENSE_B: now also U5.16 (ADC1_IN11/ADC2_IN11/ADC3_IN11/PC1)
- net SENSE_C: now also U5.15 (ADC1_IN10/ADC2_IN10/ADC3_IN10/USB_OTG_HS_ULPI_STP/PC0)
- net VBAT_ADC: now also U5.34 (ADC1_IN15/ADC2_IN15/PC5)
- net VDD: now also C53.2, C54.2, R90.1, R91.1, R92.1, U5.100 (VDD), U5.11 (VDD), U5.19 (VDD), U5.22 (VDDA), U5.28 (VDD), U5.50 (VDD), U5.6 (VBAT), U5.75 (VDD)
- net at C27.1, Y1.1: now also U5.12 (PH0/RCC_OSC_IN)
- net at C32.1, Y1.2: now also U5.13 (PH1/RCC_OSC_OUT)
- net at C30.1, C31.1, FB1.2: now also U5.21 (VREF+)
- net at C15.2: now also U5.73 (VCAP_2)
- net at R5.1: now also C3.2, R8.1, U5.14 (NRST)
- removed net ENCODER_A_CON: J5.3 (Pin_3), SW1.4, SW1.5
- removed net ENCODER_B_CON: J5.1 (Pin_1), SW1.2, SW1.3
- net ENCODER_B_DE: no longer names the net of SW1.15
- net ENCODER_B_DE: no longer SW1.16
- net ENCODER_RS485_A: no longer names the net of R40.2, R83.2, U3.6 (A)
- net ENCODER_RS485_A: now also J12.2 (Pin_2); no longer SW1.12
- net ENCODER_RS485_B: no longer names the net of R38.1, R81.1, U3.7 (B)
- net ENCODER_RS485_B: now also J12.3 (Pin_3); no longer SW1.14
- net ENCODER_Z_CON renamed ENCODER_Z
- net ENCODER_Z: now also R90.2, U5.25 (ADC1_IN2/ADC2_IN2/ADC3_IN2/TIM2_CH3/TIM5_CH3/TIM9_CH1/USART2_TX/PA2)
- net RS485_DE renamed PD4
- net PD4: now also U5.85 (PD4/FSMC_NOE/USART2_RTS)
- net RS485_DI renamed PD5
- net PD5: now also U5.86 (PD5/FSMC_NWE/USART2_TX)
- net RS485_RO renamed PD6
- net PD6: now also U5.87 (PD6/FSMC_NWAIT/USART2_RX)
- new net: C10.2, U5.49 (VCAP_1)
- new net ENCODER_B: J5.1 (Pin_1), R92.2, U5.24 (ADC1_IN1/ADC2_IN1/ADC3_IN1/TIM2_CH2/TIM5_CH2/UART4_RX/USART2_RTS/PA1)
- new net ENCODER_RS485_MCLR: J12.5 (Pin_5), U5.60 (PD13/FSMC_A18/TIM4_CH2)
- new net PA10: U5.69 (TIM1_CH3/USART1_RX/USB_OTG_FS_ID/PA10)
- new net PA3: U5.26 (ADC1_IN3/ADC2_IN3/ADC3_IN3/TIM2_CH4/TIM5_CH4/TIM9_CH2/USART2_RX/USB_OTG_HS_ULPI_D0/PA3)
- new net PA8: U5.67 (I2C3_SCL/RCC_MCO_1/TIM1_CH1/USART1_CK/USB_OTG_FS_SOF/PA8)
- new net PA9: U5.68 (DAC_EXTI9/I2C3_SMBA/TIM1_CH2/USART1_TX/USB_OTG_FS_VBUS/PA9)
- new net PB0: C51.2, J8.1 (Pin_1), R17.2, U5.35 (ADC1_IN8/ADC2_IN8/TIM1_CH2N/TIM3_CH3/TIM8_CH2N/USB_OTG_HS_ULPI_D1/PB0)
- new net PB10: U5.47 (I2C2_SCL/I2S2_CK/SPI2_SCK/TIM2_CH3/USART3_TX/USB_OTG_HS_ULPI_D3/PB10)
- new net PB11: U5.48 (ADC1_EXTI11/ADC2_EXTI11/ADC3_EXTI11/I2C2_SDA/TIM2_CH4/USART3_RX/USB_OTG_HS_ULPI_D4/PB11)
- new net PB13: U5.52 (CAN2_TX/I2S2_CK/SPI2_SCK/TIM1_CH1N/USART3_CTS/USB_OTG_HS_ULPI_D6/USB_OTG_HS_VBUS/PB13)
- new net PB4: U5.90 (I2S3_ext_SD/SPI1_MISO/SPI3_MISO/SYS_JTRST/TIM3_CH1/PB4)
- new net PB9: U5.96 (CAN1_TX/DAC_EXTI9/I2C1_SDA/I2S2_WS/SDIO_D5/SPI2_NSS/TIM11_CH1/TIM4_CH4/PB9)
- new net PC14: U5.8 (RCC_OSC32_IN/PC14)
- new net PC15: U5.9 (ADC1_EXTI15/ADC2_EXTI15/ADC3_EXTI15/RCC_OSC32_OUT/PC15)
- new net PC3: C4.2, R10.2, U5.18 (ADC1_IN13/ADC2_IN13/ADC3_IN13/I2S2_SD/SPI2_MOSI/USB_OTG_HS_ULPI_NXT/PC3), USR1.2
- new net PD0: U5.81 (PD0/CAN1_RX/FSMC_D2/FSMC_DA2)
- new net PD1: U5.82 (PD1/CAN1_TX/FSMC_D3/FSMC_DA3)
- new net PD10: U5.57 (PD10/FSMC_D15/FSMC_DA15/USART3_CK)
- new net PD11: U5.58 (PD11/ADC1_EXTI11/ADC2_EXTI11/ADC3_EXTI11/FSMC_A16/FSMC_CLE/USART3_CTS)
- new net PD14: U5.61 (PD14/FSMC_D0/FSMC_DA0/TIM4_CH3)
- new net PD15: U5.62 (PD15/ADC1_EXTI15/ADC2_EXTI15/ADC3_EXTI15/FSMC_D1/FSMC_DA1/TIM4_CH4)
- new net PD3: U5.84 (PD3/FSMC_CLK/USART2_CTS)
- new net PD7: U5.88 (PD7/FSMC_NCE2/FSMC_NE1/USART2_CK)
- new net PE0: U5.97 (PE0/FSMC_NBL0/TIM4_ETR)
- new net PE1: U5.98 (PE1/FSMC_NBL1)
- new net PE14: U5.45 (PE14/FSMC_D11/FSMC_DA11/TIM1_CH4)
- new net PE15: U5.46 (PE15/ADC1_EXTI15/ADC2_EXTI15/ADC3_EXTI15/FSMC_D12/FSMC_DA12/TIM1_BKIN)
- new net PE2: U5.1 (PE2/FSMC_A23/SYS_TRACECLK)
- new net PE3: U5.2 (PE3/FSMC_A19/SYS_TRACED0)
- new net PE4: U5.3 (PE4/FSMC_A20/SYS_TRACED1)
- new net PE5: U5.4 (PE5/FSMC_A21/SYS_TRACED2/TIM9_CH1)
- new net PE6: U5.5 (PE6/FSMC_A22/SYS_TRACED3/TIM9_CH2)
- no-connect marks 23 -> 61
Other:
- moved on the sheet: C14, C15, C19, C24, C25, C27, C28, C29, C3, C30, C31, C32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

Commit message: Routed version 2.0
Parts:
- removed SW1: SW_DIP_x08, Button_Switch_SMD:SW_DIP_SPSTx08_Slide_Copal_CHS-08A_W5.08mm_P1.27mm_JPin, symbol Switch:SW_DIP_x08
- added C55: 100nF 50V, Capacitor_SMD:C_0603_1608Metric, symbol servo-sigma-48v-rescue:C-device
- added SW1: SW_DIP_x04, Button_Switch_SMD:SW_DIP_SPSTx04_Slide_Copal_CHS-04A_W5.08mm_P1.27mm_JPin, symbol Switch:SW_DIP_x04
Connections:
- net A_TERM_R120: now also SW1.6
- net BOOT0: now also SW1.5
- net B_TERM_R120: now also SW1.3
- net GND: now also C55.1
- net VDD: now also C55.2, SW1.1, SW1.2, SW1.4
- net PE0 renamed GPIO_CONF_2
- net GPIO_CONF_2: now also SW1.7
- net PE1 renamed GPIO_CONF_1
- net GPIO_CONF_1: now also SW1.8
- no-connect marks 61 -> 42
Changed lines of the file:
@@
 PE15
 Wire Wire Line
-	8050 5150 8450 5150
-Wire Wire Line
-	8050 5250 8450 5250
-Wire Wire Line
 	8050 5350 8450 5350
 Wire Wire Line
@@
 Wire Wire Line
 	8050 6650 8450 6650
-NoConn ~ 8450 5150
-NoConn ~ 8450 5250
 NoConn ~ 8450 5350
 NoConn ~ 8450 5450
@@
 Wire Wire Line
 	17450 6250 17850 6250
-NoConn ~ 10100 14150
-NoConn ~ 9500 14150
-NoConn ~ 9500 14250
-NoConn ~ 9500 14350
-NoConn ~ 10100 14350
-NoConn ~ 10100 14250
-$Comp
-L Switch:SW_DIP_x08 SW1
-U 1 1 5D20434C
-P 9800 14050
-F 0 "SW1" H 9800 14717 50  0000 C CNN
-F 1 "SW_DIP_x08" H 9800 14626 50  0000 C CNN
-F 2 "Button_Switch_SMD:SW_DIP_SPSTx08_Slide_Copal_CHS-08A_W5.08mm_P1.27mm_JPin" H 9800 14050 50  0001 C CNN
-F 3 "http://www.grayhill.com/assets/1/7/DIP_Series_97.pdf" H 9800 14050 50  0001 C CNN
-F 4 "GH7645CT-ND" H 9800 14050 50  0001 C CNN "Part"
-F 5 "DigiKey" H 9800 14050 50  0001 C CNN "Provider"
-	1    9800 14050
-	1    0    0    -1
-$EndComp
-NoConn ~ 10100 13650
-NoConn ~ 10100 13750
-NoConn ~ 10100 13850
-NoConn ~ 10100 13950
-NoConn ~ 10100 14050
-NoConn ~ 9500 13650
-NoConn ~ 9500 13750
-NoConn ~ 9500 13850
-NoConn ~ 9500 13950
-NoConn ~ 9500 14050
-NoConn ~ 4350 10050
 NoConn ~ 8450 6850
 NoConn ~ 8450 6950
@@
 NoConn ~ 17450 3750
 NoConn ~ 17450 3850
+$Comp
+L servo-sigma-48v-rescue:C-device C55
+U 1 1 5C675569
+P 15750 1400
+F 0 "C55" H 15600 1300 50  0000 L CNN
+F 1 "100nF 50V" H 15300 1500 50  0000 L CNN
+F 2 "Capacitor_SMD:C_0603_1608Metric" H 15788 1250 50  0001 C CNN
+F 3 "http://psearch.en.murata.com/capacitor/product/GCM188R71H104KA57%23.pdf" H 15750 1400 50  0001 C CNN
+F 4 "490-4779-2-ND" H 15750 1400 60  0001 C CNN "Part"
+F 5 "DigiKey" H 15750 1400 60  0001 C CNN "Provider"
+	1    15750 1400
+	-1   0    0    1
+$EndComp
+Wire Wire Line
+	15150 950  15750 950
+Wire Wire Line
+	15750 950  15750 1250
+Connection ~ 15150 950
+Wire Wire Line
+	15150 1800 15750 1800
+Wire Wire Line
+	15750 1800 15750 1550
+Connection ~ 15150 1800
+$Comp
+L Switch:SW_DIP_x04 SW1
+U 1 1 5C6BDADE
+P 13200 11550
+F 0 "SW1" H 13200 12017 50  0000 C CNN
+F 1 "SW_DIP_x04" H 13200 11926 50  0000 C CNN
+F 2 "Button_Switch_SMD:SW_DIP_SPSTx04_Slide_Copal_CHS-04A_W5.08mm_P1.27mm_JPin" H 13200 11550 50  0001 C CNN
+F 3 "http://www.grayhill.com/assets/1/7/DIP_Series_97.pdf" H 13200 11550 50  0001 C CNN
+F 4 "GH7644CT-ND" H 13200 11550 50  0001 C CNN "Part"
+F 5 "DigiKey" H 13200 11550 50  0001 C CNN "Provider"
+	1    13200 11550
+	1    0    0    -1
+$EndComp
+Wire Wire Line
+	12900 11550 12100 11550
+Text Label 12100 11550 0    60   ~ 0
+B_TERM_R120
+Text Label 14200 11550 2    60   ~ 0
+A_TERM_R120
+Wire Wire Line
+	14200 11550 13500 11550
+Text Label 14200 11650 2    60   ~ 0
+BOOT0
+Wire Wire Line
+	13500 11650 14200 11650
+$Comp
+L power:VDD #PWR0134
+U 1 1 5C805834
+P 12100 11650
+F 0 "#PWR0134" H 12100 11500 50  0001 C CNN
+F 1 "VDD" H 12117 11823 50  0000 C CNN
+F 2 "" H 12100 11650 50  0001 C CNN
+F 3 "" H 12100 11650 50  0001 C CNN
+	1    12100 11650
+	0    -1   -1   0
+$EndComp
+Wire Wire Line
+	12100 11650 12900 11650
+$Comp
+L power:VDD #PWR0135
+U 1 1 5CA5B291
+P 12100 11350
+F 0 "#PWR0135" H 12100 11200 50  0001 C CNN
+F 1 "VDD" H 12117 11523 50  0000 C CNN
+F 2 "" H 12100 11350 50  0001 C CNN
+F 3 "" H 12100 11350 50  0001 C CNN
+	1    12100 11350
+	0    -1   -1   0
+$EndComp
+Wire Wire Line
+	12100 11350 12750 11350
+Wire Wire Line
+	12900 11450 12750 11450
+Wire Wire Line
+	12750 11450 12750 11350
+Connection ~ 12750 11350
+Wire Wire Line
+	12750 11350 12900 11350
+Text Label 14200 11450 2    60   ~ 0
+GPIO_CONF_2
+Text Label 14200 11350 2    60   ~ 0
+GPIO_CONF_1
+Text Label 6600 5150 0    60   ~ 0
+GPIO_CONF_2
+Text Label 6600 5250 0    60   ~ 0
+GPIO_CONF_1
+Wire Wire Line
+	6600 5150 8450 5150
+Wire Wire Line
+	6600 5250 8450 5250
+Wire Wire Line
+	13500 11350 14200 11350
+Wire Wire Line
+	13500 11450 14200 11450
 $EndSCHEMATC

Commit message: Added NPTH for mounting heat sink.
Parts:
- removed R86, R87: 4.7k, Resistor_SMD:R_0603_1608Metric, symbol servo-sigma-48v-rescue:R-device
- R38, R40: value 4.7k -> N/A
Connections:
- net A_TERM_R120: now also J10.2 (Pin_2), J11.2 (Pin_2), R40.2; no longer J10.1 (Pin_1), J11.1 (Pin_1)
- net GND: now also J10.1 (Pin_1), J11.1 (Pin_1), J8.1 (Pin_1), J9.1 (Pin_1); no longer J10.3 (Pin_3), J11.3 (Pin_3), J8.3 (Pin_3), J9.3 (Pin_3)
- net PB0: now also J8.3 (Pin_3); no longer J8.1 (Pin_1)
- net PB1: now also J9.3 (Pin_3); no longer J9.1 (Pin_1)
- net at R88.1, U12.7 (B): now also J10.3 (Pin_3), J11.3 (Pin_3), R38.1; no longer J10.2 (Pin_2), J11.2 (Pin_2)
- net at J12.2 (Pin_2), R83.2, U3.6 (A): no longer R40.2
- net at J12.3 (Pin_3), R81.1, U3.7 (B): no longer R38.1
Other:
- moved on the sheet: J10, J11
