File: hardware/servo-sigma-48v/mcu.sch (KiCad schematic (older format))
At the start: 67 parts, among them J10 Conn_01x03, J11 Conn_01x03, J12 Conn_01x05, J2 CONN_02X05, J5 Conn_01x05, J6 629_105_150_921, J8 Conn_01x03, J9 Conn_01x03, SW1 SW_DIP_x04, U12 SN65HVD75DGKR, U3 SN65HVD75DGKR, U5 STM32F405VGTx, Y1 ABM3-8.000MHZ-D2Y-T

Commit message: completed routing
Parts:
- removed R89: 21, Resistor_SMD:R_0603_1608Metric, symbol servo-sigma-48v-rescue:R-device
- added F1, F2, F3, F4: FIDUCIAL, Fiducials:Fiducial_0.5mm_Dia_1mm_Outer, symbol sigmadrone:FIDUCIAL
- added J4: Conn_01x03, Connector_PinHeader_2.54mm:PinHeader_1x03_P2.54mm_Horizontal, symbol Connector_Generic:Conn_01x03
Connections:
- net PD14 is gone; now on net LED_WARN: U5.61 (PD14/FSMC_D0/FSMC_DA0/TIM4_CH3)
- net PD15 is gone; now on net LED_STATUS: U5.62 (PD15/ADC1_EXTI15/ADC2_EXTI15/ADC3_EXTI15/FSMC_D1/FSMC_DA1/TIM4_CH4)
- net +5V: now also J4.2 (Pin_2)
- net B_TERM_R120: now also R88.2
- net GND: now also J4.1 (Pin_1)
- net IA_FB: now also U5.32 (ADC1_IN7/ADC2_IN7/SPI1_MOSI/TIM14_CH1/TIM1_CH1N/TIM3_CH2/TIM8_CH1N/PA7); no longer U5.30 (ADC1_IN5/ADC2_IN5/DAC_OUT2/SPI1_SCK/TIM2_CH1/TIM2_ETR/TIM8_CH1N/USB_OTG_HS_ULPI_CK/PA5)
- net IC_FB: now also U5.30 (ADC1_IN5/ADC2_IN5/DAC_OUT2/SPI1_SCK/TIM2_CH1/TIM2_ETR/TIM8_CH1N/USB_OTG_HS_ULPI_CK/PA5); no longer U5.32 (ADC1_IN7/ADC2_IN7/SPI1_MOSI/TIM14_CH1/TIM1_CH1N/TIM3_CH2/TIM8_CH1N/PA7)
- net LED_STATUS: no longer U5.54 (ADC1_EXTI15/ADC2_EXTI15/ADC3_EXTI15/I2S2_SD/RTC_REFIN/SPI2_MOSI/TIM12_CH2/TIM1_CH3N/TIM8_CH3N/USB_OTG_HS_DP/PB15)
- net LED_WARN: no longer U5.53 (I2S2_ext_SD/SPI2_MISO/TIM12_CH1/TIM1_CH2N/TIM8_CH2N/USART3_RTS/USB_OTG_HS_DM/PB14)
- net PB0: no longer C51.2, J8.3 (Pin_3), R17.2
- net PB1: no longer C52.2, J9.3 (Pin_3), R28.2
- net PB12: now also C51.2, J8.3 (Pin_3), R17.2
- net PB13: now also C52.2, J9.3 (Pin_3), R28.2
- net PB4: now also J4.3 (Pin_3)
- net PC3: no longer C4.2, R10.2, USR1.2
- net PD11: now also C4.2, R10.2, USR1.2
- net IR_FB renamed DRV_FAULT
- net PA3 renamed DRV2_CS
- net PA4 renamed DRV1_CS
- net PC10 renamed DRV_CLK
- net PC11 renamed DRV_SDO
- net PC12 renamed DRV_SDI
- net PE14 renamed GATE_ENABLE
- net PE15 renamed DRV_CAL
- net PWM renamed PC6
- net VDD renamed +3V3
- new net PB14: U5.53 (I2S2_ext_SD/SPI2_MISO/TIM12_CH1/TIM1_CH2N/TIM8_CH2N/USART3_RTS/USB_OTG_HS_DM/PB14)
- new net PB15: U5.54 (ADC1_EXTI15/ADC2_EXTI15/ADC3_EXTI15/I2S2_SD/RTC_REFIN/SPI2_MOSI/TIM12_CH2/TIM1_CH3N/TIM8_CH3N/USB_OTG_HS_DP/PB15)
- no-connect marks 42 -> 35
