File: hardware/servo-sigma-48v/mosfets_driving.sch (KiCad schematic (older format))
At the start: 73 parts, among them J7 CONN_01X02, Q1 STL160NS3LLH7, Q2 STL160NS3LLH7, Q3 STL160NS3LLH7, Q4 STL160NS3LLH7, Q5 STL160NS3LLH7, Q6 STL160NS3LLH7, Q7 STL160NS3LLH7, Q8 STL160NS3LLH7, U11 L6398, U4 L6398, U6 L6398, U7 L6398

Commit message: completed routing
Parts:
- removed C26, C36, C47, C50: 1uF 100V, Capacitor_SMD:C_0805_2012Metric, symbol servo-sigma-48v-rescue:C-device
- removed C35, C48, C49: 100pF 100V, Capacitor_SMD:C_0603_1608Metric, symbol servo-sigma-48v-rescue:C-device
- removed D10, D12, D13, D15, D16, D6, D7, D9: BAT30KFILM, Diodes_SMD:D_SOD-523, symbol servo-sigma-48v-rescue:D_Schottky-device
- removed D11, D14, D17, D8: STPS0560Z, Diodes_SMD:D_SOD-123, symbol servo-sigma-48v-rescue:D_Schottky-device
- removed R25, R26, R29, R35, R36, R39, R54, R55, R74, R75, R78: 5, Resistor_SMD:R_0603_1608Metric, symbol servo-sigma-48v-rescue:R-device
- removed R27, R32, R37, R42, R56, R79, R80: 10k, Resistor_SMD:R_0603_1608Metric, symbol servo-sigma-48v-rescue:R-device
- removed R33, R34, R43, R53, R76, R77: 21, Resistor_SMD:R_0603_1608Metric, symbol servo-sigma-48v-rescue:R-device
- removed R82: 0.010 1%, Resistor_SMD:R_2512_6332Metric, symbol servo-sigma-48v-rescue:R-device
- removed U11, U4, U6, U7: L6398, Package_SO:SOIC-8_3.9x4.9mm_P1.27mm, symbol sigmadrone:L6398
- added C1, C6: 4.7uF 50V, Capacitor_SMD:C_0805_2012Metric, symbol servo-sigma-48v-rescue:C-device
- added C11, C39, C40: 1uF 100V, Capacitor_SMD:C_1206_3216Metric, symbol servo-sigma-48v-rescue:C-device
- added C12, C2, C7, C9: 100nF, Capacitor_SMD:C_0603_1608Metric, symbol servo-sigma-48v-rescue:C-device
- added C13: 1uF 16V, Capacitor_SMD:C_0603_1608Metric, symbol servo-sigma-48v-rescue:C-device
- added C26, C35: 100uF, Capacitor_SMD:CP_Elec_6.3x7.7, symbol servo-sigma-48v-rescue:CP-device
- added C36, C37: 120uF, Capacitor_SMD:CP_Elec_10x10, symbol servo-sigma-48v-rescue:CP-device
- added D2, D3: STPS0560Z, Diode_SMD:D_SOD-123, symbol servo-sigma-48v-rescue:D_Schottky-device
- added D5: BAT30KFILM, Diode_SMD:D_SOD-523, symbol servo-sigma-48v-rescue:D_Schottky-device
- added J1: CONN_01X02, Sigmadrone:PhoenixContact_MKDS_02x7.62mm_Vertical, symbol servo-sigma-48v-rescue:CONN_01X02-conn
- added J3: CONN_01X03, Sigmadrone:PhoenixContact_MKDS_03x7.62mm_Vertical, symbol servo-sigma-48v-rescue:CONN_01X03-conn
- added L1, L2: 22uH, Inductor_SMD:L_Wuerth_WE-TPC-3816, symbol servo-sigma-48v-rescue:L-device
- added NT1, NT2, NT4, NT6: Net-Tie_2, NetTie:NetTie-2_SMD_Pad0.5mm, symbol Device:Net-Tie_2
- added R11, R12: 21, Resistor_SMD:R_0603_1608Metric, symbol servo-sigma-48v-rescue:R-device
- added R13: 28k, Resistor_SMD:R_0603_1608Metric, symbol servo-sigma-48v-rescue:R-device
- added R16: 8.45k, Resistor_SMD:R_0603_1608Metric, symbol servo-sigma-48v-rescue:R-device
- added R6, R7: 10k, Resistor_SMD:R_0603_1608Metric, symbol servo-sigma-48v-rescue:R-device
- added U1, U2: DRV8323RS, Package_DFN_QFN:QFN-48-1EP_7x7mm_P0.5mm_EP5.45x5.45mm_ThermalVias, symbol sigmadrone:DRV8323RS
- C16, C21: value 100pF 100V -> 0.047uF 100V; footprint Capacitor_SMD:C_0603_1608Metric -> Capacitor_SMD:C_0805_2012Metric; Part 399-7821-2-ND -> 490-4969-1-ND
- C17: value 1uF 100V -> 4.7uF 50V; Part 445-8887-1-ND -> 490-10751-2-ND; Value1 (none) -> 4.7uF 25V
- C18, C33: value 100pF 100V -> 1uF 16V; Part 399-7821-2-ND -> 732-7971-1-ND
- C20: value 1uF 100V -> 1uF 16V; footprint Capacitor_SMD:C_0805_2012Metric -> Capacitor_SMD:C_0603_1608Metric; Part 445-8887-1-ND -> 732-7971-1-ND
- C22, C34: value 1uF 100V -> 100nF; footprint Capacitor_SMD:C_0805_2012Metric -> Capacitor_SMD:C_0603_1608Metric; Part 445-8887-1-ND -> 490-4779-2-ND
- C23: value 100pF 100V -> 4.7uF 50V; footprint Capacitor_SMD:C_0603_1608Metric -> Capacitor_SMD:C_0805_2012Metric; Part 399-7821-2-ND -> 490-10751-2-ND; Value1 (none) -> 4.7uF 25V
- R18: value 5 -> 18k; Part 311-4.99HRCT-ND -> 311-18.0KHRCT-ND
- R22: value 10k -> 3.3k; Part 311-10.0KHRCT-ND -> 311-3.30KHRCT-ND
- R23: value 21 -> 47k; Part 311-21.0HRCT-ND -> 311-47KDCT-ND
- R24: value 21 -> 4.7k; Part 311-21.0HRCT-ND -> 311-2606-2-ND
Connections:
- net GATE_CL is gone; now on net VIN: R23.1
- net A_ISENSE_P: now also U2.11 (SPA)
- net B_ISENSE_P: now also U2.14 (SPB)
- net C_ISENSE_P: now also U2.21 (SPC)
- net GND: now also C17.2, C18.2, C23.2, C33.2, R22.1, R24.2, C2.2, C26.2, C35.2, C7.2, D2.2 (A), D3.2 (A), NT1.1, R16.1, U1.27 (DGND), U1.35 (AGND), U1.43 (BGND), U1.46 (BGND), U2.27 (DGND), U2.35 (AGND), U2.43 (BGND), U2.46 (BGND); no longer C16.1, C18.1, C20.1, C21.1, C23.1, C33.1, Q8.1 (S), R67.2, R68.2, R69.2
- net PHASE_A: now also J3.1 (P1), U2.9 (SHA); no longer C34.1
- net PHASE_B: now also J3.2 (P2), U2.16 (SHB); no longer C22.1
- net PHASE_C: now also J3.3 (P3), U2.19 (SHC); no longer C17.1, R22.2
- net PHASE_R: now also U1.19 (SHC)
- net PWM_AH: now also U2.37 (INHA)
- net PWM_AL: now also U2.38 (INLA); no longer C33.2
- net PWM_BH: now also U2.39 (INHB); no longer C23.2
- net PWM_BL: now also U2.40 (INLB); no longer C21.2
- net PWM_CH: now also U2.41 (INHC); no longer C18.2
- net PWM_CL: now also U2.42 (INLC); no longer C16.2
- net VIN: now also C17.1, C20.1, C1.1, C11.1, C12.1, C13.1, C36.1, C37.1, C39.1, C40.1, C6.1, C9.1, J1.2 (P2), U1.6 (VM), U1.7 (VDRAIN), U2.47 (VIN), U2.48 (~SHDN), U2.6 (VM), U2.7 (VDRAIN)
- net at C34.2: now also D2.1 (K), L1.1, U1.45 (SW)
- net at C22.2: now also D3.1 (K), L2.1, U2.45 (SW)
- net +5V: now reaches R18.2
- net +5V: now also C23.1, C26.1, D5.1 (K), L2.2, U1.47 (VIN), U1.48 (~SHDN)
- net GHA: now reaches Q5.2 (G)
- net GHA: now also U2.8 (GHA)
- net GHB: now reaches Q3.2 (G)
- net GHB: now also U2.17 (GHB)
- net GLA: now reaches Q6.2 (G)
- net GLA: now also U2.10 (GLA)
- net GLB: now reaches Q4.2 (G)
- net GLB: now also U2.15 (GLB)
- net GLC: now reaches Q2.2 (G)
- net GLC: now also U2.20 (GLC); no longer R23.2
- net GHR: now reaches Q7.2 (G)
- net GHR: now also U1.18 (GHC)
- net GLR: now reaches Q8.2 (G)
- net GLR: now also U1.20 (GLC)
- net +15V: no longer names the net of R18.1
- net +15V: now also R22.2, U2.1 (FB); no longer C20.2
- net GATE_CH renamed VBAT_ADC
- net VBAT_ADC: now also R23.2
- net R_ISENSE_P renamed PGND
- net PGND: now also Q8.1 (S), R67.2, R68.2, R69.2, C1.2, C11.2, C12.2, C36.2, C37.2, C39.2, C40.2, C6.2, C9.2, J1.1 (P1), NT1.2, NT2.2, NT4.2, NT6.2, U1.2 (PGND), U1.49 (PAD), U2.2 (PGND), U2.49 (PAD)
- new net: C22.1, U2.44 (CB)
- new net: C13.2, U2.5 (VCP)
- new net: R13.1, R16.2, U1.1 (FB)
- new net: C34.1, U1.44 (CB)
- new net: C20.2, U1.5 (VCP)
- new net: R12.2, U1.29 (SDO)
- new net: C21.2, U1.3 (CPL)
- new net: C33.1, U1.36 (DVDD)
- new net: C21.1, U1.4 (CPH)
- new net: R11.2, U2.29 (SDO)
- new net: C16.2, U2.3 (CPL)
- new net: C18.1, U2.36 (DVDD)
- new net: C16.1, U2.4 (CPH)
- new net +3V3: C2.1, C35.1, C7.1, L1.2, R13.2, R6.1, R7.1, U1.26 (VREF), U2.26 (VREF)
- new net A_ISENSE_N: NT2.1, U2.12 (SNA)
- new net B_ISENSE_N: NT4.1, U2.13 (SNB)
- new net C_ISENSE_N: NT6.1, U2.22 (SNC)
- new net DRV1_CS: U2.32 (~SCS)
- new net DRV2_CS: U1.32 (~SCS)
- new net DRV_CAL: U2.34 (CAL)
- new net DRV_CLK: U1.31 (SCLK), U2.31 (SCLK)
- new net DRV_FAULT: R7.2, U2.28 (~FAULT)
- new net DRV_SDI: U1.30 (SDI), U2.30 (SDI)
- new net DRV_SDO: R11.1, R12.1, R6.2
- new net DRV_SOA: U2.25 (SOA)
- new net DRV_SOB: U2.24 (SOB)
- new net DRV_SOC: U2.23 (SOC)
- new net EXT_5V: D5.2 (A)
- new net GATE_ENABLE: U1.33 (ENABLE), U2.33 (ENABLE)
- new net GHC: Q1.2 (G), U2.18 (GHC)
- new net PWM_RH: U1.41 (INHC)
- new net PWM_RL: U1.42 (INLC)
- no-connect marks 0 -> 21
Other:
- note added: "Power\nDecoupling\n"
- note added: "Voltage Sense"
- moved on the sheet: J7, Q1, Q2, Q3, Q4, Q5, Q6, Q7, Q8, R67, R68, R69
