File: hardware/servo-sigma-48v/servo-sigma-48v.kicad_pcb (KiCad board)
At the start: 4 copper layers, 64.7 x 71.7 mm, 176 parts, among them J1 CONN_01X02, J2 CONN_02X05, J3 CONN_01X03, J4 CONN_01X03_MALE, J5 CONN_01X05, J6 629_105_150_921, J7 CONN_01X02, Q1 STL160NS3LLH7, Q2 STL160NS3LLH7, Q3 STL160NS3LLH7, Q4 STL160NS3LLH7, Q5 STL160NS3LLH7, Q6 STL160NS3LLH7, Q7 STL160NS3LLH7, Q8 STL160NS3LLH7, U1 ST1S14, U10 OPA4374, U11 L6398, U2 TPS70950, U3 ACS711, U4 L6398, U5 STM32F411RETx, U6 L6398, U7 L6398, U8 TPS70933, U9 OPA4374, Y1 ABM3-8.000MHZ-D2Y-T

Commit message: Work on sigmadrive 2.0
Parts:
- removed C10: 100nF 50V, Capacitor_SMD:C_0603_1608Metric
- removed C5, C8: 1uF 100V, Capacitor_SMD:C_0805_2012Metric
- removed R14: 10k, Resistor_SMD:R_0603_1608Metric
- removed R15: 47k, Resistor_SMD:R_0603_1608Metric
- removed U3: ACS711, Package_SO:SOIC-8_3.9x4.9mm_P1.27mm
- added C51: 100nF 50V, Capacitor_SMD:C_0603_1608Metric, F.Cu at (188.0, 92.1)
- added C52: 100nF 50V, Capacitor_SMD:C_0603_1608Metric, F.Cu at (191.0, 92.1)
- added J8: Conn_01x03, Connector_PinHeader_2.54mm:PinHeader_1x03_P2.54mm_Horizontal, F.Cu at (181.1, 60.5)
- added J9: Conn_01x03, Connector_PinHeader_2.54mm:PinHeader_1x03_P2.54mm_Horizontal, F.Cu at (181.2, 69.6)
- added R17: 10k, Resistor_SMD:R_0603_1608Metric, F.Cu at (188.0, 93.6)
- added R20: 100, Resistor_SMD:R_0603_1608Metric, F.Cu at (191.0, 93.6)
- added R28: 10k, Resistor_SMD:R_0603_1608Metric, F.Cu at (194.0, 92.1)
- added R30: 100, Resistor_SMD:R_0603_1608Metric, F.Cu at (197.0, 92.1)
- R67, R68, R69, R82: value 0.0005 1% -> 0.010 1%
- moved C43 99.1 mm to (68.1, 143.6)
- moved R16 99.1 mm to (68.1, 145.1)
- moved R21 99.1 mm to (73.1, 145.1)
- moved U10 99.1 mm to (70.6, 150.6)
- moved C11 99.1 mm to (76.4, 147.7)
- moved C44 99.1 mm to (76.4, 153.5)
- moved C45 99.1 mm to (64.8, 147.7)
- moved C46 99.1 mm to (64.8, 153.5)
- moved R57 99.1 mm to (76.4, 151.7)
- moved R61 99.1 mm to (76.4, 149.5)
- moved R65 99.1 mm to (64.8, 149.5)
- moved R72 99.1 mm to (64.8, 151.7)
- moved R31 79.2 mm to (99.7, 152.3)
- moved R41 79.2 mm to (99.7, 150.8)
- moved R58 79.2 mm to (99.7, 153.8)
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Connections:
- C1 pad 1: +BATT -> VIN
- C12 pad 1: +BATT -> VIN
- C2 pad 1: +BATT -> VIN
- C4 pad 2: /MCU/PA4 -> /MCU/PB12
- C6 pad 1: +BATT -> VIN
- C7 pad 1: +BATT -> VIN
- C9 pad 1: +BATT -> VIN
- R10 pad 2: /MCU/PA4 -> /MCU/PB12
- U1 pad 5: +BATT -> VIN
- U1 pad 7: +BATT -> VIN
- U5 pad 14: /MCU/CURRENT_ADC -> /MCU/PA0
- U5 pad 15: /MCU/VBAT_ADC -> /MCU/PA1
- U5 pad 16: /MCU/CURRENT_FAULT -> /MCU/PA2
- U5 pad 17: /MCU/IR_FB -> /MCU/PA3
- U5 pad 21: /MCU/LED_WARN -> /MCU/PA5
- U5 pad 22: /MCU/LED_STATUS -> /MCU/IR_FB
- U5 pad 23: /MCU/PA7 -> /MCU/VBAT_ADC
- U5 pad 26: /MCU/PB0 -> /MCU/ENCODER_Z
- U5 pad 29: /MCU/PB10 -> /MCU/LED_STATUS
- U5 pad 3: /MCU/PC14 -> /MCU/AUX_H
- U5 pad 37: /MCU/AUX_H -> /MCU/PC6
- U5 pad 38: /MCU/AUX_L -> /MCU/PC7
- U5 pad 4: /MCU/PC15 -> /MCU/AUX_L
- U5 pad 57: /MCU/ENCODER_Z -> /MCU/PB5
- U5 pad 62: /MCU/PB9 -> /MCU/LED_WARN
- USR1 pad 2: /MCU/PA4 -> /MCU/PB12
Routing:
- net +3V3: track 207.1 -> 104.2 mm, vias 10 -> 6
- net /MCU/CURRENT_FAULT: track 60.4 -> 0.00 mm, vias 3 -> 0
- net /MCU/CURRENT_ADC: track 56.8 -> 0.00 mm, vias 2 -> 0
- net VIN: track 0.00 -> 44.5 mm
- net +BATT: track 44.5 -> 0.00 mm
- net /MCU/IR_FB: track 37.2 -> 0.00 mm, vias 2 -> 0
- net /MOSFETs/A_ISENSE_P: track 27.8 -> 0.00 mm, vias 2 -> 0
- net /MCU/PA4: track 24.2 -> 0.00 mm, vias 1 -> 0
- net Net-(R16-Pad1): track 21.6 -> 0.00 mm
- net /MCU/LED_STATUS: track 28.1 -> 13.0 mm
- net /MCU/LED_WARN: track 26.5 -> 12.2 mm
- net /MCU/IA_FB: track 41.2 -> 30.9 mm, vias 2 -> 1
- net /MCU/IB_FB: track 18.7 -> 9.46 mm, vias 2 -> 1
- net /MCU/AUX_L: track 27.0 -> 18.4 mm, vias 2 -> 1
- net /MCU/IC_FB: track 25.8 -> 17.8 mm
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- removed copper zone on F.Cu, net +BATT

Commit message: work on rs485
Parts:
- added C5: 100nF 50V, Capacitor_SMD:C_0603_1608Metric, B.Cu at (143.0, 66.7)
- added C8: 100nF 50V, Capacitor_SMD:C_0603_1608Metric, B.Cu at (143.7, 87.5)
- added J10: Conn_01x03, Connector_PinHeader_2.54mm:PinHeader_1x03_P2.54mm_Horizontal, F.Cu at (139.6, 82.7)
- added J11: Conn_01x03, Connector_PinHeader_2.54mm:PinHeader_1x03_P2.54mm_Horizontal, F.Cu at (139.6, 73.8)
- added R14: 10k, Resistor_SMD:R_0603_1608Metric, B.Cu at (142.4, 55.4)
- added R15: 10k, Resistor_SMD:R_0603_1608Metric, B.Cu at (144.0, 55.4)
- added R38: 4.7k, Resistor_SMD:R_0603_1608Metric, B.Cu at (147.8, 66.7)
- added R40: 4.7k, Resistor_SMD:R_0603_1608Metric, B.Cu at (146.7, 56.1)
- added R81: 100, Resistor_SMD:R_0603_1608Metric, B.Cu at (144.6, 66.7)
- added R83: 21, Resistor_SMD:R_0603_1608Metric, B.Cu at (146.2, 66.7)
- added R84: 10k, Resistor_SMD:R_0603_1608Metric, B.Cu at (142.9, 75.3)
- added R85: 10k, Resistor_SMD:R_0603_1608Metric, B.Cu at (144.6, 75.3)
- added R86: 4.7k, Resistor_SMD:R_0603_1608Metric, B.Cu at (142.0, 87.4)
- added R87: 4.7k, Resistor_SMD:R_0603_1608Metric, B.Cu at (145.3, 87.5)
- added R88: 100, Resistor_SMD:R_0603_1608Metric, B.Cu at (136.7, 76.3)
- added R89: 21, Resistor_SMD:R_0603_1608Metric, B.Cu at (135.1, 76.3)
- added SW1: SW_DIP_x08, Button_Switch_SMD:SW_DIP_SPSTx08_Slide_Copal_CHS-08A_W5.08mm_P1.27mm_JPin, F.Cu at (126.8, 65.9)
- added SW2: SW_DIP_x08, Button_Switch_SMD:SW_DIP_SPSTx08_Slide_Copal_CHS-08A_W5.08mm_P1.27mm_JPin, F.Cu at (126.8, 75.3)
- added U12: SN65HVD75DGKR, Package_SO:SOIC-8_3.9x4.9mm_P1.27mm, B.Cu at (144.8, 81.0)
- added U3: SN65HVD75DGKR, Package_SO:SOIC-8_3.9x4.9mm_P1.27mm, B.Cu at (144.9, 61.1)
- C11, C3, C43, C44, C45, C46, C51, C52, R16, R17, R20, R21, R28, R30, R47, R5, R50, R57, R61, R65, R72, R8, U10: moved to B.Cu
- J4: value CONN_01X03_MALE -> Conn_01x03; footprint Connector_PinHeader_2.54mm:PinHeader_1x03_P2.54mm_Vertical -> Connector_PinHeader_2.54mm:PinHeader_1x03_P2.54mm_Horizontal
- J5: value CONN_01X05 -> Conn_01x05
- moved C46 69.3 mm to (95.4, 91.3), turned to 180 degrees
- moved R65 68.0 mm to (95.4, 88.7)
- moved C45 68.0 mm to (95.4, 86.9), turned to 180 degrees
- moved R16 67.5 mm to (88.2, 80.7), turned to 0 degrees
- moved R72 65.9 mm to (95.4, 93.3)
- moved C43 64.6 mm to (88.2, 82.2), turned to 0 degrees
- moved U10 63.7 mm to (89.6, 89.8), turned to 0 degrees
- moved R21 63.2 mm to (88.2, 83.7), turned to 0 degrees
- moved C44 62.6 mm to (83.7, 91.3), turned to 0 degrees
- moved R73 62.6 mm to (83.7, 97.6), turned to 0 degrees
- moved R61 61.2 mm to (83.8, 88.7)
- moved C11 61.2 mm to (83.8, 86.9), turned to 0 degrees
- moved F1 60.4 mm to (80.3, 55.7)
- moved F3 60.4 mm to (80.3, 55.7)
- moved R70 59.9 mm to (83.7, 99.1), turned to 0 degrees
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Connections:
- net /MCU/ENCODER_Z renamed /MCU/ENCODER_Z_CON
- net Net-(R19-Pad1) renamed /MCU/BOOT0
- J5 pad 1: /MCU/ENCODER_B -> /MCU/ENCODER_B_CON
- J5 pad 3: /MCU/ENCODER_A -> /MCU/ENCODER_A_CON
- R2 pad 1: /MCU/PB3 -> /MCU/USART_RX
- R3 pad 1: /MCU/PA15 -> /MCU/USART_TX
- R31 pad 1: /MOSFETs/A_ISENSE_P -> /MOSFETs/C_ISENSE_P
- R50 pad 2: /MCU/PA12 -> /MCU/USB_DP
- R58 pad 2: /MCU/IA_FB -> /MCU/IC_FB
- R63 pad 1: /MOSFETs/C_ISENSE_P -> /MOSFETs/R_ISENSE_P
- R66 pad 2: /MCU/IC_FB -> /MCU/IR_FB
- R70 pad 1: /MOSFETs/R_ISENSE_P -> /MOSFETs/A_ISENSE_P
- R73 pad 2: /MCU/IR_FB -> /MCU/IA_FB
- U5 pad 14: /MCU/PA0 -> /MCU/ENCODER_A
- U5 pad 15: /MCU/PA1 -> /MCU/ENCODER_B_DE
- U5 pad 16: /MCU/PA2 -> /MCU/ENCODER_DI
- U5 pad 17: /MCU/PA3 -> /MCU/ENCODER_RO
- U5 pad 58: /MCU/ENCODER_A -> /MCU/PB6
- U5 pad 59: /MCU/ENCODER_B -> /MCU/PB7
- U9 pad 1: /MCU/IA_FB -> /MCU/IC_FB
- U9 pad 14: /MCU/IR_FB -> /MCU/IA_FB
- U9 pad 8: /MCU/IC_FB -> /MCU/IR_FB
Routing:
- net +3V3: track 104.2 -> 216.2 mm, vias 6 -> 11
- net +5V: track 60.5 -> 160.3 mm
- net /MOSFETs/PHASE_A: track 70.2 -> 9.99 mm, vias 10 -> 9
- net /MCU/IR_FB: track 0.00 -> 59.1 mm, vias 0 -> 1
- net /MOSFETs/C_ISENSE_P: track 63.0 -> 4.44 mm
- net /MOSFETs/PHASE_B: track 65.2 -> 10.0 mm, vias 10 -> 9
- net GND: track 268.7 -> 213.9 mm, vias 32 -> 25
- net /MCU/PB2: track 0.00 -> 52.0 mm
- net /MOSFETs/PHASE_C: track 59.5 -> 9.99 mm, vias 10 -> 9
- net /MOSFETs/A_ISENSE_P: track 0.00 -> 45.1 mm, vias 0 -> 2
- net /MCU/PB1: track 0.00 -> 43.7 mm
- net /MCU/IB_FB: track 9.46 -> 52.8 mm
- net /MCU/ENCODER_B: track 43.3 -> 0.00 mm
- net Net-(J2-Pad6): track 38.8 -> 3.37 mm, vias 1 -> 0
- net /MCU/ENCODER_RO: track 0.00 -> 33.1 mm
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- removed copper zone on In1.Cu, net GND
Other:
- board size 64.7 x 71.7 mm -> 71.7 x 73.2 mm
