File: hardware/sigmadrive-solo/sigmadrive-solo.sch (KiCad schematic (older format))
At the start: 0 parts

Commit message: Work on sigmadrive-solo 3.1
Changed lines of the file:
@@
 F24 "PWM_RH" I R 6650 2900 60
 F25 "PWM_RL" I R 6650 3000 60
+F26 "GATE2_ENABLE" I R 6650 3100 60
 $EndSheet
 $Sheet
@@
 F24 "GATE_ENABLE" O L 7700 3200 60
 F25 "DRV2_CS" O L 7700 3700 60
+F26 "GATE2_ENABLE" O L 7700 3100 60
 $EndSheet
 Wire Wire Line
@@
 Wire Wire Line
 	6650 3700 7700 3700
+Wire Wire Line
+	6650 3100 7700 3100
 $EndSCHEMATC
