File: hardware/sigmadrive-solo/mcu.sch (KiCad schematic (older format))
At the start: 71 parts, among them J10 Conn_01x03, J11 Conn_01x03, J12 Conn_01x05, J2 CONN_02X05, J4 Conn_01x03, J5 Conn_01x05, J6 629_105_150_921, J8 Conn_01x03, J9 Conn_01x03, SW1 SW_DIP_x04, U12 SN65HVD75DGKR, U3 SN65HVD75DGKR, U5 STM32F405VGTx, Y1 ABM3-8.000MHZ-D2Y-T

Commit message: Rerouted ADC and encoder connectors
Parts:
- removed C29: 4.7uF 25V, Capacitor_SMD:C_0805_2012Metric, symbol servo-sigma-48v-rescue:C-device
- added D6: GREEN, LED_SMD:LED_0603_1608Metric, symbol Device:LED
- added R21: 2.2k, Resistor_SMD:R_0603_1608Metric, symbol Device:R
- C10, C14, C15, C19, C24, C25, C27, C28, C3, C30, C31, C32, C4, C5, C51, C52, C53, C54, C55, C8: symbol servo-sigma-48v-rescue:C-device -> Device:C
- D1, D4: symbol servo-sigma-48v-rescue:LED-device -> Device:LED
- J2: symbol servo-sigma-48v-rescue:CONN_02X05-conn -> Connector_Generic:Conn_02x05_Odd_Even
- R1, R10, R14, R15, R17, R19, R2, R20, R28, R3, R30, R38, R4, R40, R44, R47, R5, R50, R8, R81, R83, R84, R85, R88, R9, R90, R91, R92: symbol servo-sigma-48v-rescue:R-device -> Device:R
- Y1: symbol servo-sigma-48v-rescue:Crystal-device -> Device:Crystal
Connections:
- net labels added: PWR_ON

Commit message: Added test points.
Changed lines of the file:
@@
 	-1   0    0    -1
 $EndComp
+Text HLabel 19450 3650 2    60   Input ~ 0
+IC_FB
+Wire Wire Line
+	19450 7150 17450 7150
 Text HLabel 19450 3450 2    60   Input ~ 0
-IC_FB
-Wire Wire Line
-	19450 7150 17450 7150
-Text HLabel 19450 3650 2    60   Input ~ 0
 IA_FB
 Text HLabel 19450 3550 2    60   Input ~ 0
@@
 Connection ~ 12750 11650
 Wire Wire Line
+	17450 3650 19450 3650
+Wire Wire Line
+	17450 3550 19450 3550
+Wire Wire Line
 	17450 3450 19450 3450
 Wire Wire Line
-	17450 3550 19450 3550
-Wire Wire Line
-	17450 3650 19450 3650
-Wire Wire Line
 	17450 3750 17850 3750

Commit message: Adding capacitors on the current sense lines.
Parts:
- C28, C31: Part 445-8887-1-ND -> 445-6804-2-ND
Changed lines of the file:
@@
 EESchema Schematic File Version 4
+LIBS:sigmadrive-solo-cache
 EELAYER 26 0
 EELAYER END
@@
 F 2 "Capacitor_SMD:C_0805_2012Metric" H 5488 3050 50  0001 C CNN
 F 3 "https://product.tdk.com/info/en/catalog/datasheets/mlcc_commercial_soft_en.pdf" H 5450 3200 50  0001 C CNN
-F 4 "445-8887-1-ND" H 5450 3200 60  0001 C CNN "Part"
+F 4 "445-6804-2-ND" H 5450 3200 60  0001 C CNN "Part"
 F 5 "DigiKey" H 5450 3200 60  0001 C CNN "Provider"
 	1    5450 3200
@@
 F 2 "Capacitor_SMD:C_0805_2012Metric" H 6788 3050 50  0001 C CNN
 F 3 "https://product.tdk.com/info/en/catalog/datasheets/mlcc_commercial_soft_en.pdf" H 6750 3200 50  0001 C CNN
-F 4 "445-8887-1-ND" H 6750 3200 60  0001 C CNN "Part"
+F 4 "445-6804-2-ND" H 6750 3200 60  0001 C CNN "Part"
 F 5 "DigiKey" H 6750 3200 60  0001 C CNN "Provider"
 	1    6750 3200

Commit message: Work on sigmadrive-solo 3.1
Parts:
- added C42, C43, C44: 100pF, Capacitor_SMD:C_0603_1608Metric, symbol Device:C
- added R25: 0, Resistor_SMD:R_0603_1608Metric, symbol Device:R
- added R27, R29, R31: 21, Resistor_SMD:R_0603_1608Metric, symbol Device:R
- added U4: TPD4S009, Package_SO:TSSOP-10_3x3mm_P0.5mm, symbol sigmadrone:TPD4S009
Connections:
- net labels added: ENCODER_RE, GATE2_ENABLE
- wire segments 365 -> 411
- no-connect marks 35 -> 33

Commit message: Updated Inductor footprints. Split RE/DE for RS485.
Parts:
- removed FB1: BEAD/0.6OHM/0.2A/2.2 kOhm @ 100MHz, Resistor_SMD:R_0603_1608Metric, symbol sigmadrone:FB_SMT
- added FB1: 0.6OHM/0.2A/2.2 kOhm @ 100MHz, Resistor_SMD:R_0603_1608Metric, symbol Device:Ferrite_Bead
- added R33, R34, R35: 0, Resistor_SMD:R_0603_1608Metric, symbol Device:R
- added R36: 21, Resistor_SMD:R_0603_1608Metric, symbol Device:R
- C42, C43, C44: value 100pF -> 1000pF/50V; Part 399-7821-2-ND -> 1276-1091-2-ND
Connections:
- net labels added: RS485_RE
- wire segments 411 -> 418
- no-connect marks 33 -> 32

Commit message: Added part number for TPD4S009
Parts:
- U4: Part (none) -> 296-24538-1-ND; Provider (none) -> DigiKey
Changed lines of the file:
@@
 F 2 "Package_SO:TSSOP-10_3x3mm_P0.5mm" H 20900 2200 60  0001 C CNN
 F 3 "http://www.ti.com/lit/ds/symlink/tpd4s009.pdf" H 20950 2100 60  0001 C CNN
+F 4 "296-24538-1-ND" H 21050 2650 50  0001 C CNN "Part"
+F 5 "DigiKey" H 21050 2650 50  0001 C CNN "Provider"
 	1    21050 2650
 	1    0    0    -1

Commit message: Changed MCU to STM32F745
Parts:
- removed C25: 100nF 50V, Capacitor_SMD:C_0603_1608Metric, symbol Device:C
- removed U5: STM32F405VGTx, Package_QFP:LQFP-100_14x14mm_P0.5mm, symbol STM32LEGACY:STM32F405VGTx
- added U5: STM32F745VETx, Package_QFP:LQFP-100_14x14mm_P0.5mm, symbol STM32LEGACY:STM32F745VETx
Connections:
- wire segments 418 -> 414
