File: hardware/sigmadrive-solo/mcu.sch (KiCad schematic (older format))
At the start: 83 parts, among them J10 Conn_01x03, J11 Conn_01x03, J12 Conn_01x05, J2 CONN_02X05, J4 Conn_01x03, J5 Conn_01x05, J6 629_105_150_921, J8 Conn_01x03, J9 Conn_01x03, SW1 SW_DIP_x04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

Commit message: Added DIR and BUSY lines.
Parts:
- removed J4: Conn_01x03, Connector_PinHeader_2.54mm:PinHeader_1x03_P2.54mm_Horizontal, symbol Connector_Generic:Conn_01x03
- added J4: Conn_01x05, Connector_PinHeader_2.54mm:PinHeader_1x05_P2.54mm_Horizontal, symbol Connector_Generic:Conn_01x05
- added R37: 10k, Resistor_SMD:R_0603_1608Metric, symbol Device:R
Connections:
- net labels added: BUSY, DIR
- wire segments 414 -> 419
- no-connect marks 32 -> 30
Changed lines of the file:
@@
 	12150 9100 12150 8950
 Connection ~ 12050 9100
-Wire Wire Line
-	6550 7150 6950 7150
 Text Label 17550 8350 2    60   ~ 0
 PC14
@@
 Text Label 4850 8450 0    60   ~ 0
 LED_STATUS
-Wire Wire Line
-	17150 6050 17550 6050
 $Comp
 L Connector_Generic:Conn_01x03 J8
@@
 NoConn ~ 17150 5050
 NoConn ~ 17150 7850
-NoConn ~ 17150 6050
 Text HLabel 4550 6150 0    60   Output ~ 0
 PWM_AH
@@
 Wire Wire Line
 	4550 6450 6950 6450
-Text Label 18850 5750 2    60   ~ 0
+Text Label 18850 6050 2    60   ~ 0
 ENCODER_Z
 Text Label 18850 6450 2    60   ~ 0
@@
 	1    13500 14400
 	0    1    1    0
-$EndComp
-$Comp
-L Connector_Generic:Conn_01x03 J4
-U 1 1 5D4ACCD8
-P 12150 14400
-AR Path="/58BE2779/5D4ACCD8" Ref="J4"  Part="1"
-AR Path="/58BE27E6/5D4ACCD8" Ref="J?"  Part="1"
-F 0 "J4" H 12150 14600 50  0000 C CNN
-F 1 "Conn_01x03" H 12150 14200 50  0000 C CNN
-F 2 "Connector_PinHeader_2.54mm:PinHeader_1x03_P2.54mm_Horizontal" H 12150 14400 50  0001 C CNN
-F 3 "https://www.molex.com/pdm_docs/sd/705530002_sd.pdf" H 12150 14400 50  0001 C CNN
-F 4 "WM4901-ND" H 12150 14400 50  0001 C CNN "Part"
-F 5 "DigiKey" H 12150 14400 50  0001 C CNN "Provider"
-	1    12150 14400
-	-1   0    0    -1
 $EndComp
 Wire Wire Line
@@
 	17150 5950 18850 5950
 Wire Wire Line
-	17150 5750 18850 5750
+	17150 6050 18850 6050
 Wire Wire Line
 	15250 14300 15250 14400
@@
 NoConn ~ 6950 6950
 NoConn ~ 6950 7050
-NoConn ~ 6950 7150
 NoConn ~ 6950 7650
 NoConn ~ 6950 7950
+$Comp
+L Connector_Generic:Conn_01x05 J4
+U 1 1 5CA2996D
+P 12150 14500
+F 0 "J4" H 12150 14800 50  0000 C CNN
+F 1 "Conn_01x05" H 12150 14200 50  0000 C CNN
+F 2 "Connector_PinHeader_2.54mm:PinHeader_1x05_P2.54mm_Horizontal" H 12150 14500 50  0001 C CNN
+F 3 "https://www.molex.com/pdm_docs/sd/705530002_sd.pdf" H 12150 14500 50  0001 C CNN
+F 4 "WM4903-ND" H 12150 14500 50  0001 C CNN "Part"
+F 5 "DigiKey" H 12150 14500 50  0001 C CNN "Provider"
+	1    12150 14500
+	-1   0    0    -1
+$EndComp
+Text Label 13500 14600 2    60   ~ 0
+DIR
+Wire Wire Line
+	12350 14600 13500 14600
+Text Label 13500 14700 2    60   ~ 0
+BUSY
+Wire Wire Line
+	12350 14700 12700 14700
+Wire Wire Line
+	12700 13800 12700 13900
+$Comp
+L Device:R R37
+U 1 1 5CAFBC64
+P 12700 14050
+F 0 "R37" V 12780 14050 50  0000 C CNN
+F 1 "10k" V 12700 14050 50  0000 C CNN
+F 2 "Resistor_SMD:R_0603_1608Metric" V 12630 14050 50  0001 C CNN
+F 3 "http://www.yageo.com.tw/exep/pages/download/literatures/PYu-R_INT-thick_7.pdf" H 12700 14050 50  0001 C CNN
+F 4 "311-10.0KHRCT-ND" V 12700 14050 60  0001 C CNN "Part"
+F 5 "DigiKey" V 12700 14050 60  0001 C CNN "Provider"
+	1    12700 14050
+	1    0    0    -1
+$EndComp
+$Comp
+L power:+3V3 #PWR?
+U 1 1 5CAFBC6A
+P 12700 13800
+AR Path="/58BE27E6/5CAFBC6A" Ref="#PWR?"  Part="1"
+AR Path="/58BF664D/5CAFBC6A" Ref="#PWR?"  Part="1"
+AR Path="/58BE2779/5CAFBC6A" Ref="#PWR0113"  Part="1"
+F 0 "#PWR0113" H 12700 13650 50  0001 C CNN
+F 1 "+3V3" H 12715 13973 50  0000 C CNN
+F 2 "" H 12700 13800 50  0001 C CNN
+F 3 "" H 12700 13800 50  0001 C CNN
+	1    12700 13800
+	1    0    0    -1
+$EndComp
+Wire Wire Line
+	12700 14200 12700 14700
+Connection ~ 12700 14700
+Wire Wire Line
+	12700 14700 13500 14700
+Text Label 4850 7150 0    60   ~ 0
+BUSY
+Text Label 18850 5750 2    60   ~ 0
+DIR
+Wire Wire Line
+	17150 5750 18850 5750
+Wire Wire Line
+	4850 7150 6950 7150
 $EndSCHEMATC

Commit message: Added temperature sensor.
Parts:
- removed R34: 0, Resistor_SMD:R_0603_1608Metric, symbol Device:R
- removed R36, R83: 21, Resistor_SMD:R_0603_1608Metric, symbol Device:R
- added C25: 100nF 50V, Capacitor_SMD:C_0603_1608Metric, symbol Device:C
- added RV1: Varistor, Resistor_SMD:R_0603_1608Metric, symbol Device:Varistor
- added SW2: SW_DIP_x04, Button_Switch_SMD:SW_DIP_SPSTx04_Slide_Copal_CHS-04A_W5.08mm_P1.27mm_JPin, symbol Switch:SW_DIP_x04
- added U6: SN65HVD232DR, Package_SO:SOIC-8_3.9x4.9mm_P1.27mm, symbol Interface_CAN_LIN:SN65HVD232
- R35: value 0 -> 3.3k; Part 311-0.0GRTR-ND -> 311-3.30KHRCT-ND
- R38, R40: value N/A -> 10k; Part 311-2606-2-ND -> 311-10.0KHRCT-ND
Connections:
- net labels added: +3.3VA, CAN_D, CAN_R, GNDA, GPIO_CONF_3, GPIO_CONF_4, PULL_A, PULL_B, READY, TEMP1
- net labels removed: BUSY, RS485_RE
- wire segments 419 -> 436
- no-connect marks 30 -> 26

Commit message: Updated part number for temperature termistor.
Parts:
- RV1: value Varistor -> 10K; Part 495-76110-1-ND -> P12014CT-ND
Changed lines of the file:
@@
 	-1   0    0    1
-$EndComp
-$Comp
-L Device:Varistor RV1
-U 1 1 5E4BF9BF
-P 1400 7650
-F 0 "RV1" H 1279 7696 50  0000 R CNN
-F 1 "Varistor" H 1279 7605 50  0000 R CNN
-F 2 "Resistor_SMD:R_0603_1608Metric" V 1330 7650 50  0001 C CNN
-F 3 "https://www.tdk-electronics.tdk.com/inf/50/db/ntc/NTC_SMD_Automotive_series_0603.pdf" H 1400 7650 50  0001 C CNN
-F 4 "495-76110-1-ND" H 1400 7650 50  0001 C CNN "Part"
-F 5 "DigiKey" H 1400 7650 50  0001 C CNN "Provider"
-	1    1400 7650
-	-1   0    0    -1
 $EndComp
 Wire Wire Line
@@
 	17150 5250 18850 5250
 NoConn ~ 17150 3850
+$Comp
+L Device:Varistor RV1
+U 1 1 5E4BF9BF
+P 1400 7650
+F 0 "RV1" H 1279 7696 50  0000 R CNN
+F 1 "10K" H 1279 7605 50  0000 R CNN
+F 2 "Resistor_SMD:R_0603_1608Metric" V 1330 7650 50  0001 C CNN
+F 3 "https://industrial.panasonic.com/cdbs/www-data/pdf/AUA0000/AUA0000C8.pdf" H 1400 7650 50  0001 C CNN
+F 4 "P12014CT-ND" H 1400 7650 50  0001 C CNN "Part"
+F 5 "DigiKey" H 1400 7650 50  0001 C CNN "Provider"
+	1    1400 7650
+	-1   0    0    -1
+$EndComp
 $EndSCHEMATC

Commit message: Added explanation for the resonator capacitance selection.
Other:
- note added: "CL = (CX1 * CX2) / (CX1 + CX2) + Cstray\nCX1 = CX2 = 2(CL - Cstray)\nCL=18pF, Cstray = 2pF to 5pF\nCX1 = CX2 = 2*(18 - 4.5) = 27pF\n(27pF * 27pF)/(27pF * 27pF) + 4.5pF = 18pF"
Changed lines of the file:
@@
 	-1   0    0    -1
 $EndComp
+Text Notes 1900 6000 0    40   ~ 0
+CL = (CX1 * CX2) / (CX1 + CX2) + Cstray\nCX1 = CX2 = 2(CL - Cstray)\nCL=18pF, Cstray = 2pF to 5pF\nCX1 = CX2 = 2*(18 - 4.5) = 27pF\n(27pF * 27pF)/(27pF * 27pF) + 4.5pF = 18pF
 $EndSCHEMATC

Commit message: sigmadrive-solo board 3.3
Parts:
- removed Y1: ABM3-8.000MHZ-D2Y-T, Crystal:Crystal_SMD_Abracon_ABM3-2Pin_5.0x3.2mm, symbol Device:Crystal
- added Y1: NX3225SA-12.000M-STD-CSR-1, Crystal:Crystal_SMD_3225-4Pin_3.2x2.5mm, symbol Device:Crystal_GND24
- C27, C32: value 27pF/50V/1% -> 10pF/50V/1%; Part 490-9719-1-ND -> 490-9713-1-ND
Connections:
- net labels removed: +3.3VA, GNDA
- wire segments 436 -> 442
Other:
- note added: "CL = (CX1 * CX2) / (CX1 + CX2) + Cstray\nCX1 = CX2 = 2(CL - Cstray)\nCL=8pF, Cstray = 2pF to 5pF\nCX1 = CX2 = 2*(8 - 3) = 10pF\n(10pF * 10pF)/(10pF + 10pF) + 3pF = 8pF"
- note removed: "CL = (CX1 * CX2) / (CX1 + CX2) + Cstray\nCX1 = CX2 = 2(CL - Cstray)\nCL=18pF, Cstray = 2pF to 5pF\nCX1 = CX2 = 2*(18 - 4.5) = 27pF\n(27pF * 27pF)/(27pF * 27pF) + 4.5pF = 18pF"

Commit message: added battery ADC filter.
Parts:
- C27, C32: value 10pF/50V/1% -> 27pF/50V/1%; Part 490-9713-1-ND -> 490-9719-1-ND
- Y1: value NX3225SA-12.000M-STD-CSR-1 -> ABM3-8.000MHZ-D2Y-T; footprint Crystal:Crystal_SMD_3225-4Pin_3.2x2.5mm -> Crystal:Crystal_SMD_Abracon_ABM3-2Pin_5.0x3.2mm; symbol Device:Crystal_GND24 -> Device:Crystal; Part ‎644-1047-1-ND‎ -> 535-10630-1-ND
Connections:
- wire segments 442 -> 440
Other:
- note added: "CL = (CX1 * CX2) / (CX1 + CX2) + Cstray\nCX1 = CX2 = 2(CL - Cstray)\nCL=18pF, Cstray = 2pF to 5pF\nCX1 = CX2 = 2*(18 - 4.5) = 27pF\n(27pF * 27pF)/(27pF + 27pF) + 4.5pF = 18pF"
- note removed: "CL = (CX1 * CX2) / (CX1 + CX2) + Cstray\nCX1 = CX2 = 2(CL - Cstray)\nCL=8pF, Cstray = 2pF to 5pF\nCX1 = CX2 = 2*(8 - 3) = 10pF\n(10pF * 10pF)/(10pF + 10pF) + 3pF = 8pF"
Changed lines of the file:
@@
 U 1 1 58EFF4C6
 P 2250 4950
-F 0 "C27" V 2200 5050 50  0000 C CNN
-F 1 "10pF/50V/1%" V 2400 4950 50  0000 C CNN
+F 0 "C27" V 2200 5100 50  0000 C CNN
+F 1 "27pF/50V/1%" V 2400 4950 50  0000 C CNN
 F 2 "Capacitor_SMD:C_0603_1608Metric" H 2288 4800 50  0001 C CNN
 F 3 "http://search.murata.co.jp/Ceramy/image/img/A01X/partnumbering_e_01.pdf" H 2250 4950 50  0001 C CNN
-F 4 "490-9713-1-ND" V 2250 4950 60  0001 C CNN "Part"
+F 4 "490-9719-1-ND" V 2250 4950 60  0001 C CNN "Part"
 F 5 "DigiKey" V 2250 4950 60  0001 C CNN "Provider"
 	1    2250 4950
@@
 	-1   0    0    -1
 $EndComp
-Text HLabel 22000 3550 2    60   Input ~ 0
-IC_FB
 Text HLabel 22000 3750 2    60   Input ~ 0
+IC_FB
+Text HLabel 22000 3550 2    60   Input ~ 0
 IA_FB
 Text HLabel 22000 3650 2    60   Input ~ 0
@@
 L Device:C C42
 U 1 1 5CAFE6A1
-P 18000 3250
+P 18000 2900
 AR Path="/58BE2779/5CAFE6A1" Ref="C42"  Part="1"
 AR Path="/58BF664D/5CAFE6A1" Ref="C?"  Part="1"
-F 0 "C42" H 18000 3350 50  0000 L CNN
-F 1 "1000pF/50V" V 17850 3050 50  0000 L CNN
-F 2 "Capacitor_SMD:C_0603_1608Metric" H 18038 3100 50  0001 C CNN
-F 3 "http://www.samsungsem.com/kr/support/product-search/mlcc/__icsFiles/afieldfile/2018/06/11/CL10C102JB8NNNC.pdf" H 18000 3250 50  0001 C CNN
-F 4 "1276-1091-2-ND" H 18000 3250 60  0001 C CNN "Part"
-F 5 "DigiKey" H 18000 3250 60  0001 C CNN "Provider"
-	1    18000 3250
+F 0 "C42" H 18000 3000 50  0000 L CNN
+F 1 "1000pF/50V" V 17850 2700 50  0000 L CNN
+F 2 "Capacitor_SMD:C_0603_1608Metric" H 18038 2750 50  0001 C CNN
+F 3 "http://www.samsungsem.com/kr/support/product-search/mlcc/__icsFiles/afieldfile/2018/06/11/CL10C102JB8NNNC.pdf" H 18000 2900 50  0001 C CNN
+F 4 "1276-1091-2-ND" H 18000 2900 60  0001 C CNN "Part"
+F 5 "DigiKey" H 18000 2900 60  0001 C CNN "Provider"
+	1    18000 2900
 	1    0    0    1
 $EndComp
@@
 L power:GND #PWR017
 U 1 1 5CC09724
-P 18450 2900
-F 0 "#PWR017" H 18450 2650 50  0001 C CNN
-F 1 "GND" H 18450 2750 50  0000 C CNN
-F 2 "" H 18450 2900 50  0001 C CNN
-F 3 "" H 18450 2900 50  0001 C CNN
-	1    18450 2900
+P 18450 2550
+F 0 "#PWR017" H 18450 2300 50  0001 C CNN
+F 1 "GND" H 18450 2400 50  0000 C CNN
+F 2 "" H 18450 2550 50  0001 C CNN
+F 3 "" H 18450 2550 50  0001 C CNN
+	1    18450 2550
 	1    0    0    1
 $EndComp
 Wire Wire Line
-	18000 3100 18000 3000
+	18000 2750 18000 2650
 Wire Wire Line
-	18000 3000 18450 3000
+	18000 2650 18450 2650
 Wire Wire Line
-	18850 3000 18850 3100
+	18850 2650 18850 2750
 Wire Wire Line
-	18450 3100 18450 3000
-Connection ~ 18450 3000
+	18450 2750 18450 2650
+Connection ~ 18450 2650
 Wire Wire Line
-	18450 3000 18850 3000
+	18450 2650 18850 2650
 Wire Wire Line
-	18450 3000 18450 2900
+	18450 2650 18450 2550
 $Comp
 L Device:R R27
@@
 	0    -1   -1   0
 $EndComp
-Wire Wire Line
-	19500 3650 20000 3650
 $Comp
 L Device:R R31
@@
 	20350 2750 20000 2750
 Wire Wire Line
-	20000 2750 20000 3650
-Wire Wire Line
 	21150 2750 21550 2750
 Wire Wire Line
@@
 	17150 3650 18450 3650
 Wire Wire Line
-	18450 3400 18450 3650
+	18450 3050 18450 3650
 Connection ~ 18450 3650
 Wire Wire Line
 	18450 3650 19200 3650
-Connection ~ 20000 3650
-Wire Wire Line
-	20000 3650 21550 3650
 Connection ~ 21550 3650
 Wire Wire Line
@@
 L Device:C C43
 U 1 1 5CD712BE
-P 18450 3250
+P 18450 2900
 AR Path="/58BE2779/5CD712BE" Ref="C43"  Part="1"
 AR Path="/58BF664D/5CD712BE" Ref="C?"  Part="1"
-F 0 "C43" H 18450 3350 50  0000 L CNN
-F 1 "1000pF/50V" V 18300 3050 50  0000 L CNN
-F 2 "Capacitor_SMD:C_0603_1608Metric" H 18488 3100 50  0001 C CNN
-F 3 "http://www.samsungsem.com/kr/support/product-search/mlcc/__icsFiles/afieldfile/2018/06/11/CL10C102JB8NNNC.pdf" H 18450 3250 50  0001 C CNN
-F 4 "1276-1091-2-ND" H 18450 3250 60  0001 C CNN "Part"
-F 5 "DigiKey" H 18450 3250 60  0001 C CNN "Provider"
-	1    18450 3250
+F 0 "C43" H 18450 3000 50  0000 L CNN
+F 1 "1000pF/50V" V 18300 2700 50  0000 L CNN
+F 2 "Capacitor_SMD:C_0603_1608Metric" H 18488 2750 50  0001 C CNN
+F 3 "http://www.samsungsem.com/kr/support/product-search/mlcc/__icsFiles/afieldfile/2018/06/11/CL10C102JB8NNNC.pdf" H 18450 2900 50  0001 C CNN
+F 4 "1276-1091-2-ND" H 18450 2900 60  0001 C CNN "Part"
+F 5 "DigiKey" H 18450 2900 60  0001 C CNN "Provider"
+	1    18450 2900
 	1    0    0    1
 $EndComp
@@
 L Device:C C44
 U 1 1 5CD72252
-P 18850 3250
+P 18850 2900
 AR Path="/58BE2779/5CD72252" Ref="C44"  Part="1"
 AR Path="/58BF664D/5CD72252" Ref="C?"  Part="1"
-F 0 "C44" H 18850 3350 50  0000 L CNN
-F 1 "1000pF/50V" V 18700 3050 50  0000 L CNN
-F 2 "Capacitor_SMD:C_0603_1608Metric" H 18888 3100 50  0001 C CNN
-F 3 "http://www.samsungsem.com/kr/support/product-search/mlcc/__icsFiles/afieldfile/2018/06/11/CL10C102JB8NNNC.pdf" H 18850 3250 50  0001 C CNN
-F 4 "1276-1091-2-ND" H 18850 3250 60  0001 C CNN "Part"
-F 5 "DigiKey" H 18850 3250 60  0001 C CNN "Provider"
-	1    18850 3250
+F 0 "C44" H 18850 3000 50  0000 L CNN
+F 1 "1000pF/50V" V 18700 2700 50  0000 L CNN
+F 2 "Capacitor_SMD:C_0603_1608Metric" H 18888 2750 50  0001 C CNN
+F 3 "http://www.samsungsem.com/kr/support/product-search/mlcc/__icsFiles/afieldfile/2018/06/11/CL10C102JB8NNNC.pdf" H 18850 2900 50  0001 C CNN
+F 4 "1276-1091-2-ND" H 18850 2900 60  0001 C CNN "Part"
+F 5 "DigiKey" H 18850 2900 60  0001 C CNN "Provider"
+	1    18850 2900
 	1    0    0    1
 $EndComp
@@
 	-1   0    0    -1
 $EndComp
-Text Notes 1400 4650 0    40   ~ 0
-CL = (CX1 * CX2) / (CX1 + CX2) + Cstray\nCX1 = CX2 = 2(CL - Cstray)\nCL=8pF, Cstray = 2pF to 5pF\nCX1 = CX2 = 2*(8 - 3) = 10pF\n(10pF * 10pF)/(10pF + 10pF) + 3pF = 8pF
+Text Notes 1650 5950 0    40   ~ 0
+CL = (CX1 * CX2) / (CX1 + CX2) + Cstray\nCX1 = CX2 = 2(CL - Cstray)\nCL=18pF, Cstray = 2pF to 5pF\nCX1 = CX2 = 2*(18 - 4.5) = 27pF\n(27pF * 27pF)/(27pF + 27pF) + 4.5pF = 18pF
 $Comp
 L Device:C C32
 U 1 1 5CBC7928
 P 2250 5350
-F 0 "C32" V 2200 5450 50  0000 C CNN
-F 1 "10pF/50V/1%" V 2400 5350 50  0000 C CNN
+F 0 "C32" V 2200 5500 50  0000 C CNN
+F 1 "27pF/50V/1%" V 2400 5350 50  0000 C CNN
 F 2 "Capacitor_SMD:C_0603_1608Metric" H 2288 5200 50  0001 C CNN
 F 3 "http://search.murata.co.jp/Ceramy/image/img/A01X/partnumbering_e_01.pdf" H 2250 5350 50  0001 C CNN
-F 4 "490-9713-1-ND" V 2250 5350 60  0001 C CNN "Part"
+F 4 "490-9719-1-ND" V 2250 5350 60  0001 C CNN "Part"
 F 5 "DigiKey" V 2250 5350 60  0001 C CNN "Provider"
 	1    2250 5350
@@
 $EndComp
 $Comp
-L Device:Crystal_GND24 Y1
+L Device:Crystal Y1
 U 1 1 5CBCDE71
 P 3050 5150
-F 0 "Y1" V 3200 5000 50  0000 L CNN
-F 1 "NX3225SA-12.000M-STD-CSR-1" V 2800 4300 50  0000 L CNN
-F 2 "Crystal:Crystal_SMD_3225-4Pin_3.2x2.5mm" H 3050 5150 50  0001 C CNN
-F 3 "https://media.digikey.com/pdf/Data%20Sheets/NDK%20PDFs/NX3225SA_STD-CSR-3.pdf" H 3050 5150 50  0001 C CNN
-F 4 "‎644-1047-1-ND‎" H 3050 5150 50  0001 C CNN "Part"
+F 0 "Y1" V 3150 4950 50  0000 L CNN
+F 1 "ABM3-8.000MHZ-D2Y-T" V 2750 4550 50  0000 L CNN
+F 2 "Crystal:Crystal_SMD_Abracon_ABM3-2Pin_5.0x3.2mm" H 3050 5150 50  0001 C CNN
+F 3 "http://www.abracon.com/Resonators/abm3.pdf" H 3050 5150 50  0001 C CNN
+F 4 "535-10630-1-ND" H 3050 5150 50  0001 C CNN "Part"
 F 5 "DigiKey" H 3050 5150 50  0001 C CNN "Provider"
 	1    3050 5150
 	0    -1   -1   0
 $EndComp
-$Comp
-L power:GND #PWR0149
-U 1 1 5CCA715E
-P 2750 5150
-F 0 "#PWR0149" H 2750 4900 50  0001 C CNN
-F 1 "GND" H 2750 5000 50  0000 C CNN
-F 2 "" H 2750 5150 50  0001 C CNN
-F 3 "" H 2750 5150 50  0001 C CNN
-	1    2750 5150
-	0    1    1    0
-$EndComp
-$Comp
-L power:GND #PWR0150
-U 1 1 5CCA7553
-P 3350 5150
-F 0 "#PWR0150" H 3350 4900 50  0001 C CNN
-F 1 "GND" H 3350 5000 50  0000 C CNN
-F 2 "" H 3350 5150 50  0001 C CNN
-F 3 "" H 3350 5150 50  0001 C CNN
-	1    3350 5150
-	0    -1   -1   0
-$EndComp
-Wire Wire Line
-	3250 5150 3350 5150
-Wire Wire Line
-	2750 5150 2850 5150
 Wire Wire Line
 	17150 7250 19150 7250
 Wire Wire Line
-	21450 2850 21450 3550
-Connection ~ 21450 3550
-Wire Wire Line
-	21450 3550 22000 3550
-Wire Wire Line
-	21650 2650 21650 3750
-Connection ~ 21650 3750
-Wire Wire Line
-	21650 3750 22000 3750
-Wire Wire Line
-	19500 3750 19900 3750
-Wire Wire Line
-	19500 3550 20100 3550
-Wire Wire Line
-	19900 2650 19900 3750
-Connection ~ 19900 3750
-Wire Wire Line
-	19900 3750 21650 3750
-Wire Wire Line
-	20100 2850 20100 3550
-Connection ~ 20100 3550
-Wire Wire Line
-	20100 3550 21450 3550
-Wire Wire Line
 	17150 3550 18000 3550
 Wire Wire Line
 	17150 3750 18850 3750
 Wire Wire Line
-	18850 3400 18850 3750
+	18850 3050 18850 3750
 Connection ~ 18850 3750
 Wire Wire Line
 	18850 3750 19200 3750
 Wire Wire Line
-	18000 3400 18000 3550
+	18000 3050 18000 3550
 Connection ~ 18000 3550
 Wire Wire Line
@@
 	12250 2900 12150 2900
 Connection ~ 12150 2900
+Wire Wire Line
+	21450 2850 21450 3750
+Connection ~ 21450 3750
+Wire Wire Line
+	21450 3750 22000 3750
+Wire Wire Line
+	21650 2650 21650 3550
+Connection ~ 21650 3550
+Wire Wire Line
+	21650 3550 22000 3550
+Wire Wire Line
+	19500 3750 20100 3750
+Wire Wire Line
+	20000 3650 21550 3650
+Wire Wire Line
+	19500 3650 20000 3650
+Connection ~ 20000 3650
+Wire Wire Line
+	20000 2750 20000 3650
+Wire Wire Line
+	19500 3550 19900 3550
+Wire Wire Line
+	20100 2850 20100 3750
+Connection ~ 20100 3750
+Wire Wire Line
+	20100 3750 21450 3750
+Wire Wire Line
+	19900 2650 19900 3550
+Connection ~ 19900 3550
+Wire Wire Line
+	19900 3550 21650 3550
 $EndSCHEMATC
