File: hardware/sigmadrive-solo/mcu.sch (KiCad schematic (older format))
At the start: 88 parts, among them J10 Conn_01x03, J11 Conn_01x03, J12 Conn_01x05, J2 CONN_02X05, J4 Conn_01x05, J5 Conn_01x05, J6 629_105_150_921, J8 Conn_01x03, J9 Conn_01x03, SW1 SW_DIP_x04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

Commit message: Review from ZEK.
Parts:
- removed C28: 1uF 100V, Capacitor_SMD:C_0805_2012Metric, symbol Device:C
- removed C53: 100nF 50V, Capacitor_SMD:C_0603_1608Metric, symbol Device:C
- removed FB2: 0.6OHM/0.2A/2.2 kOhm, Resistor_SMD:R_0603_1608Metric, symbol Device:Ferrite_Bead
- added C47: 1000pF/50V, Capacitor_SMD:C_0603_1608Metric, symbol Device:C
- added C48: 100nF 50V, Capacitor_SMD:C_0603_1608Metric, symbol Device:C
- added C50: 7pF/50V/5%, Capacitor_SMD:C_0603_1608Metric, symbol Device:C
- added U7: TPD4S009, Package_SO:TSSOP-10_3x3mm_P0.5mm, symbol sigmadrone:TPD4S009
- C49: value 4.7uF 50V -> 7pF/50V/5%; footprint Capacitor_SMD:C_0805_2012Metric -> Capacitor_SMD:C_0603_1608Metric; Part 490-10751-2-ND -> ‎1276-2137-1-ND‎
Connections:
- net labels removed: +3.3VP
- wire segments 453 -> 461
- no-connect marks 26 -> 30
Other:
- note added: "Place close to CPU.\nPut this capacitor to all analog pins.\nresistor and capacitor close to CPU."
