File: hardware/sigmadrive-solo/mosfets_driving.sch (KiCad schematic (older format))
At the start: 58 parts, among them J1 CONN_01X02, J3 CONN_01X03, J7 CONN_01X02, Q1 STL160NS3LLH7, Q2 STL160NS3LLH7, Q3 STL160NS3LLH7, Q4 STL160NS3LLH7, Q5 STL160NS3LLH7, Q6 STL160NS3LLH7, Q7 STL160NS3LLH7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

Commit message: Rerouted ADC and encoder connectors
Parts:
- C1, C11, C12, C13, C16, C17, C18, C2, C20, C21, C22, C23, C33, C34, C39, C40, C6, C7, C9: symbol servo-sigma-48v-rescue:C-device -> Device:C
- C26, C35, C36, C37: symbol servo-sigma-48v-rescue:CP-device -> Device:CP
- D2, D3, D5: symbol servo-sigma-48v-rescue:D_Schottky-device -> Device:D_Shockley
- J1, J7: symbol servo-sigma-48v-rescue:CONN_01X02-conn -> Connector_Generic:Conn_01x02
- J3: symbol servo-sigma-48v-rescue:CONN_01X03-conn -> Connector_Generic:Conn_01x03
- L1, L2: symbol servo-sigma-48v-rescue:L-device -> Device:L
- Q1, Q2, Q3, Q4, Q5, Q6, Q7, Q8: symbol servo-sigma-48v-rescue:Q_NMOS_SGD-device -> Device:Q_NMOS_SGD
- R11, R12, R13, R16, R18, R22, R23, R24, R6, R67, R68, R69, R7: symbol servo-sigma-48v-rescue:R-device -> Device:R
Changed lines of the file:
@@
 EESchema Schematic File Version 4
-LIBS:servo-sigma-48v-cache
+LIBS:sigmadrive-solo-cache
 EELAYER 26 0
 EELAYER END
@@
 	14700 2050 14700 2600
 $Comp
-L servo-sigma-48v-rescue:Q_NMOS_SGD-device Q5
+L Device:Q_NMOS_SGD Q5
 U 1 1 5A928DF8
 P 9350 1550
@@
 	14700 2050 15200 2050
 $Comp
-L servo-sigma-48v-rescue:R-device R67
+L Device:R R67
 U 1 1 5BC9D211
 P 9450 3450
@@
 	9450 3600 9450 3850
 $Comp
-L servo-sigma-48v-rescue:R-device R68
+L Device:R R68
 U 1 1 5BC9D51F
 P 12100 3450
@@
 	12100 3600 12100 3850
 $Comp
-L servo-sigma-48v-rescue:R-device R69
+L Device:R R69
 U 1 1 5BC9D5F5
 P 14700 3450
@@
 	11300 10950 11800 10950
 $Comp
-L servo-sigma-48v-rescue:CONN_01X02-conn J?
+L Connector_Generic:Conn_01x02 J?
 U 1 1 5BC5C1F6
-P 11850 11350
+P 11850 11400
 AR Path="/58BE27E6/5BC5C1F6" Ref="J?"  Part="1"
 AR Path="/58BF664D/5BC5C1F6" Ref="J7"  Part="1"
 AR Path="/5BC5C1F6" Ref="J7"  Part="1"
-F 0 "J7" H 11769 11615 50  0000 C CNN
-F 1 "CONN_01X02" H 11769 11524 50  0000 C CNN
-F 2 "Sigmadrone:PhoenixContact_MKDS_02x7.62mm_Vertical" H 11850 11350 50  0001 C CNN
-F 3 "https://media.digikey.com/PDF/Data%20Sheets/Phoenix%20Contact%20PDFs/1868076.pdf" H 11850 11350 50  0001 C CNN
-F 4 "277-5840-ND" H 11850 11350 50  0001 C CNN "Part"
-F 5 "DigiKey" H 11850 11350 50  0001 C CNN "Provider"
-	1    11850 11350
+F 0 "J7" H 11769 11665 50  0000 C CNN
+F 1 "CONN_01X02" H 11769 11574 50  0000 C CNN
+F 2 "Sigmadrone:PhoenixContact_MKDS_02x7.62mm_Vertical" H 11850 11400 50  0001 C CNN
+F 3 "https://media.digikey.com/PDF/Data%20Sheets/Phoenix%20Contact%20PDFs/1868076.pdf" H 11850 11400 50  0001 C CNN
+F 4 "277-5840-ND" H 11850 11400 50  0001 C CNN "Part"
+F 5 "DigiKey" H 11850 11400 50  0001 C CNN "Provider"
+	1    11850 11400
 	1    0    0    1
 $EndComp
@@
 $EndComp
 $Comp
-L servo-sigma-48v-rescue:Q_NMOS_SGD-device Q6
+L Device:Q_NMOS_SGD Q6
 U 1 1 5C792FA5
 P 9350 2800
@@
 $EndComp
 $Comp
-L servo-sigma-48v-rescue:Q_NMOS_SGD-device Q3
+L Device:Q_NMOS_SGD Q3
 U 1 1 5C79432A
 P 12000 1550
@@
 $EndComp
 $Comp
-L servo-sigma-48v-rescue:Q_NMOS_SGD-device Q4
+L Device:Q_NMOS_SGD Q4
 U 1 1 5C794408
 P 12000 2800
@@
 $EndComp
 $Comp
-L servo-sigma-48v-rescue:Q_NMOS_SGD-device Q1
+L Device:Q_NMOS_SGD Q1
 U 1 1 5C794DDD
 P 14600 1550
@@
 $EndComp
 $Comp
-L servo-sigma-48v-rescue:Q_NMOS_SGD-device Q2
+L Device:Q_NMOS_SGD Q2
 U 1 1 5C794EBD
 P 14600 2800
@@
 $EndComp
 $Comp
-L servo-sigma-48v-rescue:Q_NMOS_SGD-device Q7
+L Device:Q_NMOS_SGD Q7
 U 1 1 5C79539C
 P 9650 10450
@@
 $EndComp
 $Comp
-L servo-sigma-48v-rescue:Q_NMOS_SGD-device Q8
+L Device:Q_NMOS_SGD Q8
 U 1 1 5C795574
 P 9650 11700
@@
 $EndComp
 $Comp
-L servo-sigma-48v-rescue:L-device L?
+L Device:L L?
 U 1 1 5C6E5DEC
 P 6900 4550
@@
 	5550 4750 6600 4750
 $Comp
-L servo-sigma-48v-rescue:D_Schottky-device D3
+L Device:D_Shockley D3
 U 1 1 5C6F6ADB
 P 6600 5300
@@
 Connection ~ 6600 4750
 $Comp
-L servo-sigma-48v-rescue:R-device R?
+L Device:R R?
 U 1 1 5C70F366
 P 7650 4750
@@
 $EndComp
 $Comp
-L servo-sigma-48v-rescue:R-device R?
+L Device:R R?
 U 1 1 5C70F372
 P 7650 5300
@@
 	6600 5750 6600 5450
 $Comp
-L servo-sigma-48v-rescue:CP-device C?
+L Device:CP C?
 U 1 1 5C78B9CA
 P 7150 5300
@@
 	7150 5750 7150 5450
 $Comp
-L servo-sigma-48v-rescue:C-device C?
+L Device:C C?
 U 1 1 5C7D8909
 P 6100 4550
@@
 	7150 4550 7150 4450
 $Comp
-L servo-sigma-48v-rescue:C-device C?
+L Device:C C?
 U 1 1 5C865E6F
 P 3250 1450
@@
 $EndComp
 $Comp
-L servo-sigma-48v-rescue:C-device C?
+L Device:C C?
 U 1 1 5C86FE85
 P 2350 1450
@@
 $EndComp
 $Comp
-L servo-sigma-48v-rescue:C-device C?
+L Device:C C?
 U 1 1 5C879D46
 P 2800 1450
@@
 	2800 1650 2800 1600
 $Comp
-L servo-sigma-48v-rescue:C-device C?
+L Device:C C?
 U 1 1 5C971DF5
 P 3350 5250
@@
 	3800 4950 3350 4950
 $Comp
-L servo-sigma-48v-rescue:C-device C?
+L Device:C C?
 U 1 1 5CC4E978
 P 3250 2250
@@
 	3250 2450 3950 2450
 $Comp
-L servo-sigma-48v-rescue:C-device C?
+L Device:C C?
 U 1 1 5CC701F5
 P 3500 2650
@@
 	2550 3150 2550 4250
 $Comp
-L servo-sigma-48v-rescue:C-device C?
+L Device:C C?
 U 1 1 5CDFEE38
 P 2550 4900
@@
 	3500 7800 3500 7900
 $Comp
-L servo-sigma-48v-rescue:R-device R?
+L Device:R R?
 U 1 1 5D5E9150
 P 3500 7500
@@
 $EndComp
 $Comp
-L servo-sigma-48v-rescue:R-device R?
+L Device:R R?
 U 1 1 5D5E9159
 P 3500 8050
@@
 $EndComp
 $Comp
-L servo-sigma-48v-rescue:CONN_01X02-conn J?
+L Connector_Generic:Conn_01x02 J?
 U 1 1 5D5E9162
-P 1250 7600
+P 1250 7650
 AR Path="/58BE27E6/5D5E9162" Ref="J?"  Part="1"
 AR Path="/58BF664D/5D5E9162" Ref="J1"  Part="1"
-F 0 "J1" H 1169 7865 50  0000 C CNN
-F 1 "CONN_01X02" H 1169 7774 50  0000 C CNN
-F 2 "Sigmadrone:PhoenixContact_MKDS_02x7.62mm_Vertical" H 1250 7600 50  0001 C CNN
-F 3 "https://media.digikey.com/PDF/Data%20Sheets/Phoenix%20Contact%20PDFs/1868076.pdf" H 1250 7600 50  0001 C CNN
-F 4 "277-5840-ND" H 1250 7600 50  0001 C CNN "Part"
-F 5 "DigiKey" H 1250 7600 50  0001 C CNN "Provider"
-	1    1250 7600
+F 0 "J1" H 1169 7915 50  0000 C CNN
+F 1 "CONN_01X02" H 1169 7824 50  0000 C CNN
+F 2 "Sigmadrone:PhoenixContact_MKDS_02x7.62mm_Vertical" H 1250 7650 50  0001 C CNN
+F 3 "https://media.digikey.com/PDF/Data%20Sheets/Phoenix%20Contact%20PDFs/1868076.pdf" H 1250 7650 50  0001 C CNN
+F 4 "277-5840-ND" H 1250 7650 50  0001 C CNN "Part"
+F 5 "DigiKey" H 1250 7650 50  0001 C CNN "Provider"
+	1    1250 7650
 	-1   0    0    1
 $EndComp
 $Comp
-L servo-sigma-48v-rescue:CP-device C?
+L Device:CP C?
 U 1 1 5D5E916B
 P 2150 7800
@@
 $EndComp
 $Comp
-L servo-sigma-48v-rescue:CP-device C?
+L Device:CP C?
 U 1 1 5D5E9190
 P 2450 7800
@@
 	11600 4650 12250 4650
 $Comp
-L servo-sigma-48v-rescue:CONN_01X03-conn J?
+L Connector_Generic:Conn_01x03 J?
 U 1 1 5D5E91A8
 P 12450 4650
@@
 	8400 2050 9450 2050
 $Comp
-L servo-sigma-48v-rescue:C-device C?
+L Device:C C?
 U 1 1 5C79A319
 P 9900 1150
@@
 	12100 1150 12100 1350
 $Comp
-L servo-sigma-48v-rescue:C-device C?
+L Device:C C?
 U 1 1 5C8289D7
 P 12550 1150
@@
 	12700 1150 12900 1150
 $Comp
-L servo-sigma-48v-rescue:C-device C?
+L Device:C C?
 U 1 1 5C8453D9
 P 15150 1150
@@
 	9750 11900 9750 12850
 $Comp
-L servo-sigma-48v-rescue:L-device L?
+L Device:L L?
 U 1 1 5CA944B3
 P 6900 13350
@@
 	5550 13550 6600 13550
 $Comp
-L servo-sigma-48v-rescue:D_Schottky-device D2
+L Device:D_Shockley D2
 U 1 1 5CA944BD
 P 6600 14100
@@
 Connection ~ 6600 13550
 $Comp
-L servo-sigma-48v-rescue:R-device R?
+L Device:R R?
 U 1 1 5CA944C8
 P 7650 14100
@@
 $EndComp
 $Comp
-L servo-sigma-48v-rescue:R-device R?
+L Device:R R?
 U 1 1 5CA944D1
 P 7650 13550
@@
 	6600 14550 6600 14250
 $Comp
-L servo-sigma-48v-rescue:CP-device C?
+L Device:CP C?
 U 1 1 5CA944E8
 P 7150 14100
@@
 	7150 14550 7150 14250
 $Comp
-L servo-sigma-48v-rescue:C-device C?
+L Device:C C?
 U 1 1 5CA944F8
 P 6100 13350
@@
 	7150 13350 7150 13250
 $Comp
-L servo-sigma-48v-rescue:C-device C?
+L Device:C C?
 U 1 1 5CA94516
 P 3250 10250
@@
 $EndComp
 $Comp
-L servo-sigma-48v-rescue:C-device C?
+L Device:C C?
 U 1 1 5CA94520
 P 2350 10250
@@
 $EndComp
 $Comp
-L servo-sigma-48v-rescue:C-device C?
+L Device:C C?
 U 1 1 5CA94529
 P 2800 10250
@@
 	2800 10450 2800 10400
 $Comp
-L servo-sigma-48v-rescue:C-device C?
+L Device:C C?
 U 1 1 5CA94540
 P 3350 14050
@@
 	3800 13750 3350 13750
 $Comp
-L servo-sigma-48v-rescue:C-device C?
+L Device:C C?
 U 1 1 5CA94583
 P 3250 11050
@@
 	3250 11250 3950 11250
 $Comp
-L servo-sigma-48v-rescue:C-device C?
+L Device:C C?
 U 1 1 5CA94590
 P 3500 11450
@@
 PWM_RL
 Wire Wire Line
-	1450 12550 3950 12550
-Wire Wire Line
 	1450 12650 3950 12650
 Wire Wire Line
@@
 	2550 11950 2550 13050
 $Comp
-L servo-sigma-48v-rescue:C-device C?
+L Device:C C?
 U 1 1 5CA945D2
 P 2550 13700
@@
 $EndComp
 $Comp
-L servo-sigma-48v-rescue:R-device R?
+L Device:R R?
 U 1 1 5CD77F2C
 P 2200 3400
@@
 $EndComp
 $Comp
-L servo-sigma-48v-rescue:R-device R?
+L Device:R R?
 U 1 1 5CF2179F
 P 1850 3400
@@
 	7450 7100 7450 7400
 $Comp
-L servo-sigma-48v-rescue:R-device R?
+L Device:R R?
 U 1 1 5CD745A7
 P 3650 3650
@@
 	1850 3650 3500 3650
 $Comp
-L servo-sigma-48v-rescue:R-device R?
+L Device:R R?
 U 1 1 5CDB071A
 P 3650 12450
@@
 	3800 12450 3950 12450
 $Comp
-L servo-sigma-48v-rescue:D_Schottky-device D?
+L Device:D_Shockley D?
 U 1 1 5D088870
 P 8150 4550
@@
 Wire Wire Line
 	7450 7400 7450 7600
+Wire Wire Line
+	1450 12550 3950 12550
 $EndSCHEMATC

Commit message: Added test points.
Parts:
- added D7: STPS0560Z, Diode_SMD:D_SOD-123, symbol Device:D_Shockley
- added TP1, TP2, TP3, TP4, TP5, TP6, TP7, TP8, TP9: PAD, TestPoint:TestPoint_Pad_D1.0mm, symbol Connector:TestPoint_Probe
- D5: value BAT30KFILM -> STPS0560Z; footprint Diode_SMD:D_SOD-523 -> Diode_SMD:D_SOD-123; Part 497-5552-1-ND -> 497-3787-1-ND
Connections:
- wire segments 268 -> 279

Commit message: Changed MOSFETs to NTMFS5C628NLT1G
Parts:
- Q1, Q2, Q3, Q4, Q5, Q6, Q7, Q8: value STL160NS3LLH7 -> NTMFS5C628NLT1G; Part 497-14988-6-ND -> NTMFS5C628NLT1GOSDKR-ND
Changed lines of the file:
@@
 EESchema Schematic File Version 4
-LIBS:sigmadrive-solo-cache
 EELAYER 26 0
 EELAYER END
@@
 P 10000 1550
 F 0 "Q5" H 10200 1600 50  0000 L CNN
-F 1 "STL160NS3LLH7" H 10200 1500 50  0000 L CNN
+F 1 "NTMFS5C628NLT1G" H 10200 1500 50  0000 L CNN
 F 2 "Sigmadrone:PQFN_5x6_SGD" H 10200 1650 50  0001 C CNN
-F 3 "http://www.st.com/content/ccc/resource/technical/document/datasheet/6c/2c/68/6d/40/eb/44/cd/DM00087549.pdf/files/DM00087549.pdf/jcr:content/translations/en.DM00087549.pdf" H 10000 1550 50  0001 C CNN
+F 3 "https://www.onsemi.com/pub/Collateral/NTMFS5C628NL-D.PDF" H 10000 1550 50  0001 C CNN
 F 4 "DigiKey" H 10000 1550 60  0001 C CNN "Provider"
-F 5 "497-14988-6-ND" H 10000 1550 60  0001 C CNN "Part"
+F 5 "NTMFS5C628NLT1GOSDKR-ND" H 10000 1550 60  0001 C CNN "Part"
 F 6 "STL160N4F7" H 10000 1550 50  0001 C CNN "Value1"
 	1    10000 1550
@@
 P 10000 2800
 F 0 "Q6" H 10200 2850 50  0000 L CNN
-F 1 "STL160NS3LLH7" H 10200 2750 50  0000 L CNN
+F 1 "NTMFS5C628NLT1G" H 10200 2750 50  0000 L CNN
 F 2 "Sigmadrone:PQFN_5x6_SGD" H 10200 2900 50  0001 C CNN
-F 3 "http://www.st.com/content/ccc/resource/technical/document/datasheet/6c/2c/68/6d/40/eb/44/cd/DM00087549.pdf/files/DM00087549.pdf/jcr:content/translations/en.DM00087549.pdf" H 10000 2800 50  0001 C CNN
+F 3 "https://www.onsemi.com/pub/Collateral/NTMFS5C628NL-D.PDF" H 10000 2800 50  0001 C CNN
 F 4 "DigiKey" H 10000 2800 60  0001 C CNN "Provider"
-F 5 "497-14988-6-ND" H 10000 2800 60  0001 C CNN "Part"
+F 5 "NTMFS5C628NLT1GOSDKR-ND" H 10000 2800 60  0001 C CNN "Part"
 F 6 "STL160N4F7" H 10000 2800 50  0001 C CNN "Value1"
 	1    10000 2800
@@
 P 12650 1550
 F 0 "Q3" H 12850 1600 50  0000 L CNN
-F 1 "STL160NS3LLH7" H 12850 1500 50  0000 L CNN
+F 1 "NTMFS5C628NLT1G" H 12850 1500 50  0000 L CNN
 F 2 "Sigmadrone:PQFN_5x6_SGD" H 12850 1650 50  0001 C CNN
-F 3 "http://www.st.com/content/ccc/resource/technical/document/datasheet/6c/2c/68/6d/40/eb/44/cd/DM00087549.pdf/files/DM00087549.pdf/jcr:content/translations/en.DM00087549.pdf" H 12650 1550 50  0001 C CNN
+F 3 "https://www.onsemi.com/pub/Collateral/NTMFS5C628NL-D.PDF" H 12650 1550 50  0001 C CNN
 F 4 "DigiKey" H 12650 1550 60  0001 C CNN "Provider"
-F 5 "497-14988-6-ND" H 12650 1550 60  0001 C CNN "Part"
+F 5 "NTMFS5C628NLT1GOSDKR-ND" H 12650 1550 60  0001 C CNN "Part"
 F 6 "STL160N4F7" H 12650 1550 50  0001 C CNN "Value1"
 	1    12650 1550
@@
 P 12650 2800
 F 0 "Q4" H 12850 2850 50  0000 L CNN
-F 1 "STL160NS3LLH7" H 12850 2750 50  0000 L CNN
+F 1 "NTMFS5C628NLT1G" H 12850 2750 50  0000 L CNN
 F 2 "Sigmadrone:PQFN_5x6_SGD" H 12850 2900 50  0001 C CNN
-F 3 "http://www.st.com/content/ccc/resource/technical/document/datasheet/6c/2c/68/6d/40/eb/44/cd/DM00087549.pdf/files/DM00087549.pdf/jcr:content/translations/en.DM00087549.pdf" H 12650 2800 50  0001 C CNN
+F 3 "https://www.onsemi.com/pub/Collateral/NTMFS5C628NL-D.PDF" H 12650 2800 50  0001 C CNN
 F 4 "DigiKey" H 12650 2800 60  0001 C CNN "Provider"
-F 5 "497-14988-6-ND" H 12650 2800 60  0001 C CNN "Part"
+F 5 "NTMFS5C628NLT1GOSDKR-ND" H 12650 2800 60  0001 C CNN "Part"
 F 6 "STL160N4F7" H 12650 2800 50  0001 C CNN "Value1"
 	1    12650 2800
@@
 P 15250 1550
 F 0 "Q1" H 15450 1600 50  0000 L CNN
-F 1 "STL160NS3LLH7" H 15450 1500 50  0000 L CNN
+F 1 "NTMFS5C628NLT1G" H 15450 1500 50  0000 L CNN
 F 2 "Sigmadrone:PQFN_5x6_SGD" H 15450 1650 50  0001 C CNN
-F 3 "http://www.st.com/content/ccc/resource/technical/document/datasheet/6c/2c/68/6d/40/eb/44/cd/DM00087549.pdf/files/DM00087549.pdf/jcr:content/translations/en.DM00087549.pdf" H 15250 1550 50  0001 C CNN
+F 3 "https://www.onsemi.com/pub/Collateral/NTMFS5C628NL-D.PDF" H 15250 1550 50  0001 C CNN
 F 4 "DigiKey" H 15250 1550 60  0001 C CNN "Provider"
-F 5 "497-14988-6-ND" H 15250 1550 60  0001 C CNN "Part"
+F 5 "NTMFS5C628NLT1GOSDKR-ND" H 15250 1550 60  0001 C CNN "Part"
 F 6 "STL160N4F7" H 15250 1550 50  0001 C CNN "Value1"
 	1    15250 1550
@@
 P 15250 2800
 F 0 "Q2" H 15450 2850 50  0000 L CNN
-F 1 "STL160NS3LLH7" H 15450 2750 50  0000 L CNN
+F 1 "NTMFS5C628NLT1G" H 15450 2750 50  0000 L CNN
 F 2 "Sigmadrone:PQFN_5x6_SGD" H 15450 2900 50  0001 C CNN
-F 3 "http://www.st.com/content/ccc/resource/technical/document/datasheet/6c/2c/68/6d/40/eb/44/cd/DM00087549.pdf/files/DM00087549.pdf/jcr:content/translations/en.DM00087549.pdf" H 15250 2800 50  0001 C CNN
+F 3 "https://www.onsemi.com/pub/Collateral/NTMFS5C628NL-D.PDF" H 15250 2800 50  0001 C CNN
 F 4 "DigiKey" H 15250 2800 60  0001 C CNN "Provider"
-F 5 "497-14988-6-ND" H 15250 2800 60  0001 C CNN "Part"
+F 5 "NTMFS5C628NLT1GOSDKR-ND" H 15250 2800 60  0001 C CNN "Part"
 F 6 "STL160N4F7" H 15250 2800 50  0001 C CNN "Value1"
 	1    15250 2800
@@
 P 9650 10450
 F 0 "Q7" H 9850 10500 50  0000 L CNN
-F 1 "STL160NS3LLH7" H 9850 10400 50  0000 L CNN
+F 1 "NTMFS5C628NLT1G" H 9850 10400 50  0000 L CNN
 F 2 "Sigmadrone:PQFN_5x6_SGD" H 9850 10550 50  0001 C CNN
-F 3 "http://www.st.com/content/ccc/resource/technical/document/datasheet/6c/2c/68/6d/40/eb/44/cd/DM00087549.pdf/files/DM00087549.pdf/jcr:content/translations/en.DM00087549.pdf" H 9650 10450 50  0001 C CNN
+F 3 "https://www.onsemi.com/pub/Collateral/NTMFS5C628NL-D.PDF" H 9650 10450 50  0001 C CNN
 F 4 "DigiKey" H 9650 10450 60  0001 C CNN "Provider"
-F 5 "497-14988-6-ND" H 9650 10450 60  0001 C CNN "Part"
+F 5 "NTMFS5C628NLT1GOSDKR-ND" H 9650 10450 60  0001 C CNN "Part"
 F 6 "STL160N4F7" H 9650 10450 50  0001 C CNN "Value1"
 	1    9650 10450
@@
 P 9650 11700
 F 0 "Q8" H 9850 11750 50  0000 L CNN
-F 1 "STL160NS3LLH7" H 9850 11650 50  0000 L CNN
+F 1 "NTMFS5C628NLT1G" H 9850 11650 50  0000 L CNN
 F 2 "Sigmadrone:PQFN_5x6_SGD" H 9850 11800 50  0001 C CNN
-F 3 "http://www.st.com/content/ccc/resource/technical/document/datasheet/6c/2c/68/6d/40/eb/44/cd/DM00087549.pdf/files/DM00087549.pdf/jcr:content/translations/en.DM00087549.pdf" H 9650 11700 50  0001 C CNN
+F 3 "https://www.onsemi.com/pub/Collateral/NTMFS5C628NL-D.PDF" H 9650 11700 50  0001 C CNN
 F 4 "DigiKey" H 9650 11700 60  0001 C CNN "Provider"
-F 5 "497-14988-6-ND" H 9650 11700 60  0001 C CNN "Part"
+F 5 "NTMFS5C628NLT1GOSDKR-ND" H 9650 11700 60  0001 C CNN "Part"
 F 6 "STL160N4F7" H 9650 11700 50  0001 C CNN "Value1"
 	1    9650 11700

Commit message: Adding capacitors on the current sense lines.
Parts:
- added C29, C38, C41: 100pF, Capacitor_SMD:C_0603_1608Metric, symbol Device:C
- C1, C17, C23, C6: Value1 4.7uF 25V -> (none)
- C12, C2, C22, C34, C7, C9: value 100nF -> 100nF 50V
Connections:
- wire segments 279 -> 291
Changed lines of the file:
@@
 EESchema Schematic File Version 4
+LIBS:sigmadrive-solo-cache
 EELAYER 26 0
 EELAYER END
@@
 AR Path="/58BE2779/5C7D8909" Ref="C?"  Part="1"
 AR Path="/58BF664D/5C7D8909" Ref="C22"  Part="1"
-F 0 "C22" V 6150 4400 50  0000 L CNN
-F 1 "100nF" V 6050 4250 50  0000 L CNN
+F 0 "C22" V 6150 4350 50  0000 L CNN
+F 1 "100nF 50V" V 6050 4600 50  0000 L CNN
 F 2 "Capacitor_SMD:C_0603_1608Metric" H 6138 4400 50  0001 C CNN
 F 3 "http://psearch.en.murata.com/capacitor/product/GCM188R71H104KA57%23.pdf" H 6100 4550 50  0001 C CNN
@@
 F 4 "490-10751-2-ND" H 2350 1450 60  0001 C CNN "Part"
 F 5 "DigiKey" H 2350 1450 60  0001 C CNN "Provider"
-F 6 "4.7uF 25V" H 2350 1450 50  0001 C CNN "Value1"
+F 6 "" H 2350 1450 50  0001 C CNN "Value1"
 	1    2350 1450
 	1    0    0    -1
@@
 AR Path="/58BF664D/5C879D46" Ref="C12"  Part="1"
 F 0 "C12" H 2800 1550 50  0000 L CNN
-F 1 "100nF" V 2650 1350 50  0000 L CNN
+F 1 "100nF 50V" V 2650 1350 50  0000 L CNN
 F 2 "Capacitor_SMD:C_0603_1608Metric" H 2838 1300 50  0001 C CNN
 F 3 "http://psearch.en.murata.com/capacitor/product/GCM188R71H104KA57%23.pdf" H 2800 1450 50  0001 C CNN
@@
 F 4 "490-10751-2-ND" H 3350 5250 60  0001 C CNN "Part"
 F 5 "DigiKey" H 3350 5250 60  0001 C CNN "Provider"
-F 6 "4.7uF 25V" H 3350 5250 50  0001 C CNN "Value1"
+F 6 "" H 3350 5250 50  0001 C CNN "Value1"
 	1    3350 5250
 	1    0    0    -1
@@
 AR Path="/58BF664D/5CDFEE38" Ref="C7"  Part="1"
 F 0 "C7" H 2550 5000 50  0000 L CNN
-F 1 "100nF" V 2400 4800 50  0000 L CNN
+F 1 "100nF 50V" V 2400 4800 50  0000 L CNN
 F 2 "Capacitor_SMD:C_0603_1608Metric" H 2588 4750 50  0001 C CNN
 F 3 "http://psearch.en.murata.com/capacitor/product/GCM188R71H104KA57%23.pdf" H 2550 4900 50  0001 C CNN
@@
 Wire Wire Line
 	12750 3150 12750 3300
-Text Label 6200 3950 2    60   ~ 0
+Text Label 6600 3950 2    60   ~ 0
 A_ISENSE_P
-Text Label 6200 4350 2    60   ~ 0
+Text Label 6600 4350 2    60   ~ 0
 A_ISENSE_N
 Wire Wire Line
-	6200 4350 5550 4350
-Wire Wire Line
-	5550 3950 6200 3950
-Text Label 6200 3450 2    60   ~ 0
+	6600 4350 5750 4350
+Wire Wire Line
+	5550 3950 5750 3950
+Text Label 6600 3450 2    60   ~ 0
 B_ISENSE_P
-Text Label 6200 3850 2    60   ~ 0
+Text Label 6600 3850 2    60   ~ 0
 B_ISENSE_N
 Wire Wire Line
-	6200 3850 5550 3850
-Wire Wire Line
-	5550 3450 6200 3450
-Text Label 6200 2950 2    60   ~ 0
+	6600 3850 5750 3850
+Wire Wire Line
+	5550 3450 5750 3450
+Text Label 6600 2950 2    60   ~ 0
 C_ISENSE_P
-Text Label 6200 3350 2    60   ~ 0
+Text Label 6600 3350 2    60   ~ 0
 C_ISENSE_N
 Wire Wire Line
-	6200 3350 5550 3350
-Wire Wire Line
-	5550 2950 6200 2950
+	6600 3350 5750 3350
+Wire Wire Line
+	5550 2950 5750 2950
 Text Notes 2450 8300 0    60   ~ 0
 Power\nDecoupling\n
@@
 AR Path="/58BF664D/5CA944F8" Ref="C34"  Part="1"
 F 0 "C34" V 6150 13200 50  0000 L CNN
-F 1 "100nF" V 6050 13050 50  0000 L CNN
+F 1 "100nF 50V" V 6050 13050 50  0000 L CNN
 F 2 "Capacitor_SMD:C_0603_1608Metric" H 6138 13200 50  0001 C CNN
 F 3 "http://psearch.en.murata.com/capacitor/product/GCM188R71H104KA57%23.pdf" H 6100 13350 50  0001 C CNN
@@
 F 4 "490-10751-2-ND" H 2350 10250 60  0001 C CNN "Part"
 F 5 "DigiKey" H 2350 10250 60  0001 C CNN "Provider"
-F 6 "4.7uF 25V" H 2350 10250 50  0001 C CNN "Value1"
+F 6 "" H 2350 10250 50  0001 C CNN "Value1"
 	1    2350 10250
 	1    0    0    -1
@@
 AR Path="/58BF664D/5CA94529" Ref="C9"  Part="1"
 F 0 "C9" H 2800 10350 50  0000 L CNN
-F 1 "100nF" V 2650 10150 50  0000 L CNN
+F 1 "100nF 50V" V 2650 10150 50  0000 L CNN
 F 2 "Capacitor_SMD:C_0603_1608Metric" H 2838 10100 50  0001 C CNN
 F 3 "http://psearch.en.murata.com/capacitor/product/GCM188R71H104KA57%23.pdf" H 2800 10250 50  0001 C CNN
@@
 F 4 "490-10751-2-ND" H 3350 14050 60  0001 C CNN "Part"
 F 5 "DigiKey" H 3350 14050 60  0001 C CNN "Provider"
-F 6 "4.7uF 25V" H 3350 14050 50  0001 C CNN "Value1"
+F 6 "" H 3350 14050 50  0001 C CNN "Value1"
 	1    3350 14050
 	1    0    0    -1
@@
 AR Path="/58BF664D/5CA945D2" Ref="C2"  Part="1"
 F 0 "C2" H 2550 13800 50  0000 L CNN
-F 1 "100nF" V 2400 13600 50  0000 L CNN
+F 1 "100nF 50V" V 2400 13600 50  0000 L CNN
 F 2 "Capacitor_SMD:C_0603_1608Metric" H 2588 13550 50  0001 C CNN
 F 3 "http://psearch.en.murata.com/capacitor/product/GCM188R71H104KA57%23.pdf" H 2550 13700 50  0001 C CNN
@@
 Wire Wire Line
 	14300 3150 15350 3150
+$Comp
+L Device:C C?
+U 1 1 5C959C8D
+P 5750 3150
+AR Path="/58BE2779/5C959C8D" Ref="C?"  Part="1"
+AR Path="/58BF664D/5C959C8D" Ref="C29"  Part="1"
+F 0 "C29" H 5800 3250 50  0000 L CNN
+F 1 "100pF" H 5750 3050 50  0000 L CNN
+F 2 "Capacitor_SMD:C_0603_1608Metric" H 5788 3000 50  0001 C CNN
+F 3 "http://psearch.en.murata.com/capacitor/product/GCM188R71H104KA57%23.pdf" H 5750 3150 50  0001 C CNN
+F 4 "399-7821-2-ND" H 5750 3150 60  0001 C CNN "Part"
+F 5 "DigiKey" H 5750 3150 60  0001 C CNN "Provider"
+	1    5750 3150
+	1    0    0    -1
+$EndComp
+Wire Wire Line
+	5750 3000 5750 2950
+Connection ~ 5750 2950
+Wire Wire Line
+	5750 2950 6600 2950
+Wire Wire Line
+	5750 3300 5750 3350
+Connection ~ 5750 3350
+Wire Wire Line
+	5750 3350 5550 3350
+$Comp
+L Device:C C?
+U 1 1 5C99D9A4
+P 5750 3650
+AR Path="/58BE2779/5C99D9A4" Ref="C?"  Part="1"
+AR Path="/58BF664D/5C99D9A4" Ref="C38"  Part="1"
+F 0 "C38" H 5800 3750 50  0000 L CNN
+F 1 "100pF" H 5750 3550 50  0000 L CNN
+F 2 "Capacitor_SMD:C_0603_1608Metric" H 5788 3500 50  0001 C CNN
+F 3 "http://psearch.en.murata.com/capacitor/product/GCM188R71H104KA57%23.pdf" H 5750 3650 50  0001 C CNN
+F 4 "399-7821-2-ND" H 5750 3650 60  0001 C CNN "Part"
+F 5 "DigiKey" H 5750 3650 60  0001 C CNN "Provider"
+	1    5750 3650
+	1    0    0    -1
+$EndComp
+$Comp
+L Device:C C?
+U 1 1 5C99DB76
+P 5750 4150
+AR Path="/58BE2779/5C99DB76" Ref="C?"  Part="1"
+AR Path="/58BF664D/5C99DB76" Ref="C41"  Part="1"
+F 0 "C41" H 5800 4250 50  0000 L CNN
+F 1 "100pF" H 5750 4050 50  0000 L CNN
+F 2 "Capacitor_SMD:C_0603_1608Metric" H 5788 4000 50  0001 C CNN
+F 3 "http://psearch.en.murata.com/capacitor/product/GCM188R71H104KA57%23.pdf" H 5750 4150 50  0001 C CNN
+F 4 "399-7821-2-ND" H 5750 4150 60  0001 C CNN "Part"
+F 5 "DigiKey" H 5750 4150 60  0001 C CNN "Provider"
+	1    5750 4150
+	1    0    0    -1
+$EndComp
+Wire Wire Line
+	5750 3500 5750 3450
+Connection ~ 5750 3450
+Wire Wire Line
+	5750 3450 6600 3450
+Wire Wire Line
+	5750 3800 5750 3850
+Connection ~ 5750 3850
+Wire Wire Line
+	5750 3850 5550 3850
+Wire Wire Line
+	5750 4000 5750 3950
+Connection ~ 5750 3950
+Wire Wire Line
+	5750 3950 6600 3950
+Wire Wire Line
+	5750 4300 5750 4350
+Connection ~ 5750 4350
+Wire Wire Line
+	5750 4350 5550 4350
 $EndSCHEMATC
