File: hardware/sigmadrive-solo/mosfets_driving.sch (KiCad schematic (older format))
At the start: 71 parts, among them J1 CONN_01X02, J3 CONN_01X03, J7 CONN_01X02, Q1 NTMFS5C628NLT1G, Q2 NTMFS5C628NLT1G, Q3 NTMFS5C628NLT1G, Q4 NTMFS5C628NLT1G, Q5 NTMFS5C628NLT1G, Q6 NTMFS5C628NLT1G, Q7 NTMFS5C628NLT1G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

Commit message: Work on sigmadrive-solo 3.1
Parts:
- added R26: 28k, Resistor_SMD:R_0603_1608Metric, symbol Device:R
Connections:
- net labels added: GATE2_ENABLE
Changed lines of the file:
@@
 L Device:C C?
 U 1 1 5C971DF5
-P 3350 5250
+P 3450 5400
 AR Path="/58BE27E6/5C971DF5" Ref="C?"  Part="1"
 AR Path="/58BF664D/5C971DF5" Ref="C17"  Part="1"
-F 0 "C17" H 3350 5350 50  0000 L CNN
-F 1 "4.7uF 50V" V 3200 5000 50  0000 L CNN
-F 2 "Capacitor_SMD:C_0805_2012Metric" H 3388 5100 50  0001 C CNN
-F 3 "http://www.samsungsem.com/kr/support/product-search/mlcc/CL21A475KACLRNC.jsp" H 3350 5250 50  0001 C CNN
-F 4 "490-10751-2-ND" H 3350 5250 60  0001 C CNN "Part"
-F 5 "DigiKey" H 3350 5250 60  0001 C CNN "Provider"
-F 6 "" H 3350 5250 50  0001 C CNN "Value1"
-	1    3350 5250
-	1    0    0    -1
-$EndComp
-Wire Wire Line
-	3950 4950 3800 4950
-Wire Wire Line
-	3350 4950 3350 5100
+F 0 "C17" H 3450 5500 50  0000 L CNN
+F 1 "4.7uF 50V" V 3300 5150 50  0000 L CNN
+F 2 "Capacitor_SMD:C_0805_2012Metric" H 3488 5250 50  0001 C CNN
+F 3 "http://www.samsungsem.com/kr/support/product-search/mlcc/CL21A475KACLRNC.jsp" H 3450 5400 50  0001 C CNN
+F 4 "490-10751-2-ND" H 3450 5400 60  0001 C CNN "Part"
+F 5 "DigiKey" H 3450 5400 60  0001 C CNN "Provider"
+F 6 "" H 3450 5400 50  0001 C CNN "Value1"
+	1    3450 5400
+	1    0    0    -1
+$EndComp
 $Comp
 L power:GND #PWR042
 U 1 1 5C97DC3B
-P 3350 5500
-F 0 "#PWR042" H 3350 5250 50  0001 C CNN
-F 1 "GND" H 3350 5350 50  0000 C CNN
-F 2 "" H 3350 5500 50  0001 C CNN
-F 3 "" H 3350 5500 50  0001 C CNN
-	1    3350 5500
-	1    0    0    -1
-$EndComp
-Wire Wire Line
-	3350 5400 3350 5500
+P 3450 5650
+F 0 "#PWR042" H 3450 5400 50  0001 C CNN
+F 1 "GND" H 3450 5500 50  0000 C CNN
+F 2 "" H 3450 5650 50  0001 C CNN
+F 3 "" H 3450 5650 50  0001 C CNN
+	1    3450 5650
+	1    0    0    -1
+$EndComp
+Wire Wire Line
+	3450 5550 3450 5650
 Wire Wire Line
 	2350 1750 2350 1650
@@
 L sigmadrone:VIN #PWR?
 U 1 1 5CA64BF7
-P 3350 4850
+P 3450 4750
 AR Path="/58BE27E6/5CA64BF7" Ref="#PWR?"  Part="1"
 AR Path="/58BF664D/5CA64BF7" Ref="#PWR038"  Part="1"
-F 0 "#PWR038" H 3350 4700 50  0001 C CNN
-F 1 "VIN" H 3350 5000 50  0000 C CNN
-F 2 "" H 3350 4850 50  0000 C CNN
-F 3 "" H 3350 4850 50  0000 C CNN
-	1    3350 4850
-	1    0    0    -1
-$EndComp
-Connection ~ 3350 4950
-Wire Wire Line
-	3350 4850 3350 4950
+F 0 "#PWR038" H 3450 4600 50  0001 C CNN
+F 1 "VIN" H 3450 4900 50  0000 C CNN
+F 2 "" H 3450 4750 50  0000 C CNN
+F 3 "" H 3450 4750 50  0000 C CNN
+	1    3450 4750
+	1    0    0    -1
+$EndComp
 $Comp
 L sigmadrone:DRV8323RS U2
@@
 $EndComp
 Wire Wire Line
-	3950 5150 3800 5150
-Wire Wire Line
-	3800 5150 3800 4950
-Connection ~ 3800 4950
-Wire Wire Line
-	3800 4950 3350 4950
+	3950 5150 3850 5150
 $Comp
 L Device:C C?
@@
 Wire Wire Line
 	3650 11450 3950 11450
-Text HLabel 3600 11650 0    60   Input ~ 0
-GATE_ENABLE
-Wire Wire Line
-	3600 11650 3950 11650
+Text HLabel 1450 11650 0    60   Input ~ 0
+GATE2_ENABLE
+Wire Wire Line
+	1450 11650 3950 11650
 Text HLabel 1450 12550 0    60   Input ~ 0
 DRV_SDI
@@
 DRV_CLK
 Wire Wire Line
-	3600 12150 3950 12150
-Wire Wire Line
-	3600 12250 3950 12250
+	1450 12150 3950 12150
+Wire Wire Line
+	1450 12250 3950 12250
 Text HLabel 1450 12750 0    60   Input ~ 0
 DRV2_CS
-Text HLabel 3600 12150 0    60   Input ~ 0
+Text HLabel 1450 12150 0    60   Input ~ 0
 PWM_RH
-Text HLabel 3600 12250 0    60   Input ~ 0
+Text HLabel 1450 12250 0    60   Input ~ 0
 PWM_RL
 Wire Wire Line
@@
 Wire Wire Line
 	5750 4350 5550 4350
+$Comp
+L Device:R R?
+U 1 1 5C9E1FE1
+P 3700 5150
+AR Path="/58BF599E/5C9E1FE1" Ref="R?"  Part="1"
+AR Path="/58BE27E6/5C9E1FE1" Ref="R?"  Part="1"
+AR Path="/58BF664D/5C9E1FE1" Ref="R26"  Part="1"
+F 0 "R26" V 3780 5150 50  0000 C CNN
+F 1 "28k" V 3700 5150 50  0000 C CNN
+F 2 "Resistor_SMD:R_0603_1608Metric" V 3630 5150 50  0001 C CNN
+F 3 "http://www.yageo.com/documents/recent/PYu-RT_1-to-0.01_RoHS_L_7.pdf" H 3700 5150 50  0001 C CNN
+F 4 "311-28.0KHRCT-ND" V 3700 5150 60  0001 C CNN "Part"
+F 5 "DigiKey" V 3700 5150 60  0001 C CNN "Provider"
+	1    3700 5150
+	0    -1   -1   0
+$EndComp
+Wire Wire Line
+	3550 5150 3450 5150
+Wire Wire Line
+	3450 5150 3450 4950
+Wire Wire Line
+	3450 4950 3950 4950
+Wire Wire Line
+	3450 5250 3450 5150
+Connection ~ 3450 5150
+Wire Wire Line
+	3450 4750 3450 4950
+Connection ~ 3450 4950
 $EndSCHEMATC

Commit message: Updated Inductor footprints. Split RE/DE for RS485.
Parts:
- added R32: 28k, Resistor_SMD:R_0603_1608Metric, symbol Device:R
- C11, C39, C40: footprint Capacitor_SMD:C_1206_3216Metric -> Capacitor_SMD:C_0805_2012Metric; Part 445-4468-1-ND -> 445-6804-2-ND
- C29, C38, C41: value 100pF -> 1000pF/50V; Part 399-7821-2-ND -> 1276-1091-2-ND
- L1, L2: footprint Inductor_SMD:L_Wuerth_WE-TPC-3816 -> Sigmadrone:L_Wuerth_WE-TPC-4828

Commit message: Added DIR and BUSY lines.
Parts:
- removed J3: CONN_01X03, Sigmadrone:PhoenixContact_MKDS_03x7.62mm_Vertical, symbol Connector_Generic:Conn_01x03
- removed J7: CONN_01X02, Sigmadrone:PhoenixContact_MKDS_02x7.62mm_Vertical, symbol Connector_Generic:Conn_01x02
- J1: footprint Sigmadrone:PhoenixContact_MKDS_02x7.62mm_Vertical -> Sigmadrone:PhoenixContact_MKDS_07x7.62mm_Vertical; symbol Connector_Generic:Conn_01x02 -> Connector_Generic:Conn_01x07
Connections:
- wire segments 291 -> 289
Changed lines of the file:
@@
 Wire Wire Line
 	9750 10950 9750 11500
-Wire Wire Line
-	9750 10950 11300 10950
-Text Label 11800 10950 2    60   ~ 0
+Text Label 11050 10950 0    60   ~ 0
 PHASE_R
-Wire Wire Line
-	11300 11300 11300 10950
-Connection ~ 11300 10950
-Wire Wire Line
-	11300 10950 11800 10950
-$Comp
-L Connector_Generic:Conn_01x02 J?
-U 1 1 5BC5C1F6
-P 11850 11400
-AR Path="/58BE27E6/5BC5C1F6" Ref="J?"  Part="1"
-AR Path="/58BF664D/5BC5C1F6" Ref="J7"  Part="1"
-AR Path="/5BC5C1F6" Ref="J7"  Part="1"
-F 0 "J7" H 11769 11665 50  0000 C CNN
-F 1 "CONN_01X02" H 11769 11574 50  0000 C CNN
-F 2 "Sigmadrone:PhoenixContact_MKDS_02x7.62mm_Vertical" H 11850 11400 50  0001 C CNN
-F 3 "https://media.digikey.com/PDF/Data%20Sheets/Phoenix%20Contact%20PDFs/1868076.pdf" H 11850 11400 50  0001 C CNN
-F 4 "277-5840-ND" H 11850 11400 50  0001 C CNN "Part"
-F 5 "DigiKey" H 11850 11400 50  0001 C CNN "Provider"
-	1    11850 11400
-	1    0    0    1
-$EndComp
-Wire Wire Line
-	11300 11300 11650 11300
-Wire Wire Line
-	11300 11400 11650 11400
 $Comp
 L sigmadrone:VIN #PWR?
@@
 Wire Wire Line
 	5550 2950 5750 2950
-Text Notes 2450 8300 0    60   ~ 0
+Text Notes 11450 12250 2    60   ~ 0
 Power\nDecoupling\n
 $Comp
@@
 $EndComp
 $Comp
-L Connector_Generic:Conn_01x02 J?
+L Connector_Generic:Conn_01x07 J?
 U 1 1 5D5E9162
-P 1250 7650
+P 12900 11250
 AR Path="/58BE27E6/5D5E9162" Ref="J?"  Part="1"
 AR Path="/58BF664D/5D5E9162" Ref="J1"  Part="1"
-F 0 "J1" H 1169 7915 50  0000 C CNN
-F 1 "CONN_01X02" H 1169 7824 50  0000 C CNN
-F 2 "Sigmadrone:PhoenixContact_MKDS_02x7.62mm_Vertical" H 1250 7650 50  0001 C CNN
-F 3 "https://media.digikey.com/PDF/Data%20Sheets/Phoenix%20Contact%20PDFs/1868076.pdf" H 1250 7650 50  0001 C CNN
-F 4 "277-5840-ND" H 1250 7650 50  0001 C CNN "Part"
-F 5 "DigiKey" H 1250 7650 50  0001 C CNN "Provider"
-	1    1250 7650
-	-1   0    0    1
+F 0 "J1" H 12900 10850 50  0000 C CNN
+F 1 "CONN_01X02" H 12900 11650 50  0000 C CNN
+F 2 "Sigmadrone:PhoenixContact_MKDS_07x7.62mm_Vertical" H 12900 11250 50  0001 C CNN
+F 3 "https://media.digikey.com/PDF/Data%20Sheets/Phoenix%20Contact%20PDFs/1868076.pdf" H 12900 11250 50  0001 C CNN
+F 4 "277-5840-ND" H 12900 11250 50  0001 C CNN "Part"
+F 5 "DigiKey" H 12900 11250 50  0001 C CNN "Provider"
+	1    12900 11250
+	1    0    0    1
 $EndComp
 $Comp
 L Device:CP C?
 U 1 1 5D5E916B
-P 2150 7800
+P 11400 12550
 AR Path="/58BE27E6/5D5E916B" Ref="C?"  Part="1"
 AR Path="/58BF664D/5D5E916B" Ref="C36"  Part="1"
-F 0 "C36" H 2175 7900 50  0000 L CNN
-F 1 "120uF" H 2175 7700 50  0000 L CNN
-F 2 "Capacitor_SMD:CP_Elec_10x10" H 2188 7650 50  0001 C CNN
-F 3 "https://industrial.panasonic.com/cdbs/www-data/pdf/RDD0000/DMD0000COL92.pdf" H 2150 7800 50  0001 C CNN
-F 4 "P19316CT-ND" H 2150 7800 60  0001 C CNN "Part"
-F 5 "DigiKey" H 2150 7800 60  0001 C CNN "Provider"
-	1    2150 7800
-	1    0    0    -1
-$EndComp
-Wire Wire Line
-	1450 7650 1850 7650
-Wire Wire Line
-	1850 7650 1850 8050
-Wire Wire Line
-	2150 7950 2150 8050
-Wire Wire Line
-	2150 8050 2450 8050
-Wire Wire Line
-	2450 7950 2450 8050
-Wire Wire Line
-	2150 7650 2150 7550
-Wire Wire Line
-	2150 7550 2450 7550
-Wire Wire Line
-	2450 7650 2450 7550
+F 0 "C36" H 11425 12650 50  0000 L CNN
+F 1 "120uF" H 11425 12450 50  0000 L CNN
+F 2 "Capacitor_SMD:CP_Elec_10x10" H 11438 12400 50  0001 C CNN
+F 3 "https://industrial.panasonic.com/cdbs/www-data/pdf/RDD0000/DMD0000COL92.pdf" H 11400 12550 50  0001 C CNN
+F 4 "P19316CT-ND" H 11400 12550 60  0001 C CNN "Part"
+F 5 "DigiKey" H 11400 12550 60  0001 C CNN "Provider"
+	1    11400 12550
+	-1   0    0    -1
+$EndComp
+Wire Wire Line
+	11400 12700 11400 12800
+Wire Wire Line
+	11400 12800 11100 12800
+Wire Wire Line
+	11100 12700 11100 12800
+Wire Wire Line
+	11400 12400 11400 12300
+Wire Wire Line
+	11400 12300 11100 12300
+Wire Wire Line
+	11100 12400 11100 12300
 $Comp
 L sigmadrone:VIN #PWR?
 U 1 1 5D5E9181
-P 1850 7250
+P 11700 12150
 AR Path="/58BE27E6/5D5E9181" Ref="#PWR?"  Part="1"
 AR Path="/58BF664D/5D5E9181" Ref="#PWR058"  Part="1"
-F 0 "#PWR058" H 1850 7100 50  0001 C CNN
-F 1 "VIN" H 1865 7423 50  0000 C CNN
-F 2 "" H 1850 7250 50  0000 C CNN
-F 3 "" H 1850 7250 50  0000 C CNN
-	1    1850 7250
-	1    0    0    -1
+F 0 "#PWR058" H 11700 12000 50  0001 C CNN
+F 1 "VIN" H 11715 12323 50  0000 C CNN
+F 2 "" H 11700 12150 50  0000 C CNN
+F 3 "" H 11700 12150 50  0000 C CNN
+	1    11700 12150
+	-1   0    0    -1
 $EndComp
 $Comp
 L Device:CP C?
 U 1 1 5D5E9190
-P 2450 7800
+P 11100 12550
 AR Path="/58BE27E6/5D5E9190" Ref="C?"  Part="1"
 AR Path="/58BF664D/5D5E9190" Ref="C37"  Part="1"
-F 0 "C37" H 2475 7900 50  0000 L CNN
-F 1 "120uF" H 2475 7700 50  0000 L CNN
-F 2 "Capacitor_SMD:CP_Elec_10x10" H 2488 7650 50  0001 C CNN
-F 3 "https://industrial.panasonic.com/cdbs/www-data/pdf/RDD0000/DMD0000COL92.pdf" H 2450 7800 50  0001 C CNN
-F 4 "P19316CT-ND" H 2450 7800 60  0001 C CNN "Part"
-F 5 "DigiKey" H 2450 7800 60  0001 C CNN "Provider"
-	1    2450 7800
-	1    0    0    -1
-$EndComp
-Wire Wire Line
-	12250 4750 12900 4750
-Wire Wire Line
-	12250 4550 12900 4550
-Wire Wire Line
-	12250 4650 12900 4650
-$Comp
-L Connector_Generic:Conn_01x03 J?
-U 1 1 5D5E91A8
-P 13100 4650
-AR Path="/58BE27E6/5D5E91A8" Ref="J?"  Part="1"
-AR Path="/58BF664D/5D5E91A8" Ref="J3"  Part="1"
-F 0 "J3" H 13019 4965 50  0000 C CNN
-F 1 "CONN_01X03" H 13019 4874 50  0000 C CNN
-F 2 "Sigmadrone:PhoenixContact_MKDS_03x7.62mm_Vertical" H 13100 4650 50  0001 C CNN
-F 3 "https://media.digikey.com/PDF/Data%20Sheets/Phoenix%20Contact%20PDFs/1704936.pdf" H 13100 4650 50  0001 C CNN
-F 4 "277-5954-ND" H 13100 4650 50  0001 C CNN "Part"
-F 5 "DigiKey" H 13100 4650 50  0001 C CNN "Provider"
-	1    13100 4650
-	1    0    0    -1
-$EndComp
+F 0 "C37" H 11125 12650 50  0000 L CNN
+F 1 "120uF" H 11125 12450 50  0000 L CNN
+F 2 "Capacitor_SMD:CP_Elec_10x10" H 11138 12400 50  0001 C CNN
+F 3 "https://industrial.panasonic.com/cdbs/www-data/pdf/RDD0000/DMD0000COL92.pdf" H 11100 12550 50  0001 C CNN
+F 4 "P19316CT-ND" H 11100 12550 60  0001 C CNN "Part"
+F 5 "DigiKey" H 11100 12550 60  0001 C CNN "Provider"
+	1    11100 12550
+	-1   0    0    -1
+$EndComp
+Wire Wire Line
+	11050 11150 12700 11150
+Wire Wire Line
+	11050 11350 12700 11350
+Wire Wire Line
+	11050 11250 12700 11250
 $Comp
 L power:GND #PWR?
@@
 	6350 7100 6350 7600
 Wire Wire Line
-	1450 7550 1850 7550
-Wire Wire Line
-	1850 7550 1850 7250
-Wire Wire Line
-	1850 7550 2150 7550
-Connection ~ 1850 7550
-Connection ~ 2150 7550
+	11700 12300 11700 12150
+Wire Wire Line
+	11700 12300 11400 12300
+Connection ~ 11400 12300
 $Comp
 L sigmadrone:VIN #PWR?
@@
 	1    0    0    -1
 $EndComp
-Text Label 12250 4750 0    60   ~ 0
+Text Label 11050 11150 0    60   ~ 0
 PHASE_C
-Text Label 12250 4650 0    60   ~ 0
+Text Label 11050 11250 0    60   ~ 0
 PHASE_B
-Text Label 12250 4550 0    60   ~ 0
+Text Label 11050 11350 0    60   ~ 0
 PHASE_A
 Text Label 15850 2050 2    60   ~ 0
@@
 Text HLabel 15850 2050 2    60   Output ~ 0
 PHASE_C
-Wire Wire Line
-	11300 11400 11300 12850
 $Comp
 L power:PWR_FLAG #FLG?
@@
 Wire Wire Line
 	15350 1150 15350 1350
-Wire Wire Line
-	2150 8050 1850 8050
-Connection ~ 2150 8050
-Connection ~ 1850 8050
-Wire Wire Line
-	1850 8050 1850 8200
+Connection ~ 11400 12800
+Wire Wire Line
+	11100 12800 11100 12850
 Wire Wire Line
 	6250 5450 6250 5750
@@
 L sigmadrone:PGND #PWR0119
 U 1 1 5C8C7B0A
-P 1850 8200
-F 0 "#PWR0119" H 1850 7950 50  0001 C CNN
-F 1 "PGND" H 1855 8027 50  0000 C CNN
-F 2 "" H 1850 8200 50  0001 C CNN
-F 3 "" H 1850 8200 50  0001 C CNN
-	1    1850 8200
-	1    0    0    -1
+P 11100 12850
+F 0 "#PWR0119" H 11100 12600 50  0001 C CNN
+F 1 "PGND" H 11105 12677 50  0000 C CNN
+F 2 "" H 11100 12850 50  0001 C CNN
+F 3 "" H 11100 12850 50  0001 C CNN
+	1    11100 12850
+	-1   0    0    -1
 $EndComp
 $Comp
@@
 L sigmadrone:PGND #PWR034
 U 1 1 5CCF6FDE
-P 11300 12850
-F 0 "#PWR034" H 11300 12600 50  0001 C CNN
-F 1 "PGND" H 11300 12700 50  0000 C CNN
-F 2 "" H 11300 12850 50  0001 C CNN
-F 3 "" H 11300 12850 50  0001 C CNN
-	1    11300 12850
-	1    0    0    -1
+P 10950 11050
+F 0 "#PWR034" H 10950 10800 50  0001 C CNN
+F 1 "PGND" H 10950 10900 50  0000 C CNN
+F 2 "" H 10950 11050 50  0001 C CNN
+F 3 "" H 10950 11050 50  0001 C CNN
+	1    10950 11050
+	0    1    1    0
 $EndComp
 NoConn ~ 5550 13150
@@
 	1    0    0    1
 $EndComp
+Wire Wire Line
+	11700 12300 12000 12300
+Connection ~ 11700 12300
+Connection ~ 11100 12800
+Wire Wire Line
+	12700 11450 12000 11450
+Wire Wire Line
+	12000 11450 12000 12300
+Wire Wire Line
+	12700 11550 12350 11550
+Wire Wire Line
+	12350 11550 12350 12800
+Wire Wire Line
+	11400 12800 12350 12800
+Wire Wire Line
+	10950 11050 12700 11050
+Wire Wire Line
+	9750 10950 12700 10950
 $EndSCHEMATC

Commit message: Added temperature sensor.
Parts:
- added C45: 1uF 16V, Capacitor_SMD:C_0603_1608Metric, symbol Device:C
- added C46: 2.2uF, Capacitor_SMD:C_0603_1608Metric, symbol Device:C
- added NT3: Net-Tie_2, NetTie:NetTie-2_SMD_Pad0.5mm, symbol Device:Net-Tie_2
- added R34: N/A, Resistor_SMD:R_0603_1608Metric, symbol Device:R
- added U7: TPS70933, Package_TO_SOT_SMD:TSOT-23-5, symbol sigmadrone:TPS709
Connections:
- net labels added: +3.3VA, GNDA
- wire segments 289 -> 311
- no-connect marks 21 -> 22
