File: hardware/sigmadrive-solo/mosfets_driving.sch (KiCad schematic (older format))
At the start: 76 parts, among them J1 CONN_01X02, Q1 NTMFS5C628NLT1G, Q2 NTMFS5C628NLT1G, Q3 NTMFS5C628NLT1G, Q4 NTMFS5C628NLT1G, Q5 NTMFS5C628NLT1G, Q6 NTMFS5C628NLT1G, Q7 NTMFS5C628NLT1G, Q8 NTMFS5C628NLT1G, U1 DRV8323RS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

Commit message: Changed 18kOhm to 20kOhm part. Changed termistor value.
Parts:
- R18: value 18k -> 20k; Part 311-18.0KHRCT-ND -> 311-20.0KHRTR-ND
Changed lines of the file:
@@
 AR Path="/58BF664D/5C70F366" Ref="R18"  Part="1"
 F 0 "R18" V 7730 4750 50  0000 C CNN
-F 1 "18k" V 7650 4750 50  0000 C CNN
+F 1 "20k" V 7650 4750 50  0000 C CNN
 F 2 "Resistor_SMD:R_0603_1608Metric" V 7580 4750 50  0001 C CNN
 F 3 "http://www.yageo.com/documents/recent/PYu-RT_1-to-0.01_RoHS_L_7.pdf" H 7650 4750 50  0001 C CNN
-F 4 "311-18.0KHRCT-ND" V 7650 4750 60  0001 C CNN "Part"
+F 4 "311-20.0KHRTR-ND" V 7650 4750 60  0001 C CNN "Part"
 F 5 "DigiKey" V 7650 4750 60  0001 C CNN "Provider"
 	1    7650 4750

Commit message: sigmadrive-solo board 3.3
Parts:
- removed C45: 1uF 16V, Capacitor_SMD:C_0603_1608Metric, symbol Device:C
- removed C46: 2.2uF, Capacitor_SMD:C_0603_1608Metric, symbol Device:C
- removed NT3: Net-Tie_2, NetTie:NetTie-2_SMD_Pad0.5mm, symbol Device:Net-Tie_2
- removed R34: N/A, Resistor_SMD:R_0603_1608Metric, symbol Device:R
- removed U7: TPS70933, Package_TO_SOT_SMD:TSOT-23-5, symbol sigmadrone:TPS709
- R24: value 4.7k -> 3.3k; Part 311-2606-2-ND -> 311-3.30KHRCT-ND
Connections:
- net labels removed: +3.3VA, GNDA
- wire segments 311 -> 289
- no-connect marks 22 -> 21

Commit message: added battery ADC filter.
Parts:
- added C45: 1uF 16V, Capacitor_SMD:C_0603_1608Metric, symbol Device:C
- added R34: 47k, Resistor_SMD:R_0603_1608Metric, symbol Device:R
Connections:
- wire segments 289 -> 293
Changed lines of the file:
@@
 F 5 "DigiKey" V 12750 3450 60  0001 C CNN "Provider"
 	1    12750 3450
-	1    0    0    -1
+	-1   0    0    1
 $EndComp
 Wire Wire Line
@@
 Voltage Sense
 Wire Wire Line
-	1950 8400 1950 8150
+	1950 8400 1950 8200
 Wire Wire Line
 	1950 7100 1950 7300
@@
 AR Path="/58BE27E6/5D5E9150" Ref="R?"  Part="1"
 AR Path="/58BF664D/5D5E9150" Ref="R23"  Part="1"
-F 0 "R23" H 2100 7450 50  0000 C CNN
+F 0 "R23" V 1850 7450 50  0000 C CNN
 F 1 "47k" V 1950 7450 50  0000 C CNN
 F 2 "Resistor_SMD:R_0603_1608Metric" V 1880 7450 50  0001 C CNN
@@
 L Device:R R?
 U 1 1 5CE917D9
-P 1950 8000
+P 1950 8050
 AR Path="/58BF599E/5CE917D9" Ref="R?"  Part="1"
 AR Path="/58BE27E6/5CE917D9" Ref="R?"  Part="1"
 AR Path="/58BF664D/5CE917D9" Ref="R24"  Part="1"
-F 0 "R24" V 2030 8000 50  0000 C CNN
-F 1 "3.3k" V 1950 8000 50  0000 C CNN
-F 2 "Resistor_SMD:R_0603_1608Metric" V 1880 8000 50  0001 C CNN
-F 3 "http://www.yageo.com/documents/recent/PYu-RT_1-to-0.01_RoHS_L_7.pdf" H 1950 8000 50  0001 C CNN
-F 4 "311-3.30KHRCT-ND" V 1950 8000 60  0001 C CNN "Part"
-F 5 "DigiKey" V 1950 8000 60  0001 C CNN "Provider"
-	1    1950 8000
+F 0 "R24" V 2050 8050 50  0000 C CNN
+F 1 "3.3k" V 1950 8050 50  0000 C CNN
+F 2 "Resistor_SMD:R_0603_1608Metric" V 1880 8050 50  0001 C CNN
+F 3 "http://www.yageo.com/documents/recent/PYu-RT_1-to-0.01_RoHS_L_7.pdf" H 1950 8050 50  0001 C CNN
+F 4 "311-3.30KHRCT-ND" V 1950 8050 60  0001 C CNN "Part"
+F 5 "DigiKey" V 1950 8050 60  0001 C CNN "Provider"
+	1    1950 8050
 	-1   0    0    1
 $EndComp
@@
 	1950 7600 1950 7750
 Wire Wire Line
-	3500 7750 1950 7750
+	3500 7750 2950 7750
 Connection ~ 1950 7750
 Wire Wire Line
-	1950 7750 1950 7850
+	1950 7750 1950 7900
 $Comp
 L sigmadrone:PGND #PWR0151
@@
 	1    0    0    -1
 $EndComp
+$Comp
+L Device:R R?
+U 1 1 5CD33422
+P 2450 7750
+AR Path="/58BE27E6/5CD33422" Ref="R?"  Part="1"
+AR Path="/58BF664D/5CD33422" Ref="R34"  Part="1"
+F 0 "R34" V 2400 7950 50  0000 C CNN
+F 1 "47k" V 2450 7750 50  0000 C CNN
+F 2 "Resistor_SMD:R_0603_1608Metric" V 2380 7750 50  0001 C CNN
+F 3 "http://www.yageo.com/documents/recent/PYu-RT_1-to-0.01_RoHS_L_7.pdf" H 2450 7750 50  0001 C CNN
+F 4 "311-47KDCT-ND" V 2450 7750 60  0001 C CNN "Part"
+F 5 "DigiKey" V 2450 7750 60  0001 C CNN "Provider"
+	1    2450 7750
+	0    1    1    0
+$EndComp
+Wire Wire Line
+	2300 7750 1950 7750
+$Comp
+L Device:C C?
+U 1 1 5CD37F9B
+P 2950 8050
+AR Path="/58BE27E6/5CD37F9B" Ref="C?"  Part="1"
+AR Path="/58BF664D/5CD37F9B" Ref="C45"  Part="1"
+F 0 "C45" H 2950 8150 50  0000 L CNN
+F 1 "1uF 16V" V 2800 7800 50  0000 L CNN
+F 2 "Capacitor_SMD:C_0603_1608Metric" H 2988 7900 50  0001 C CNN
+F 3 "https://product.tdk.com/info/en/catalog/datasheets/mlcc_commercial_soft_en.pdf" H 2950 8050 50  0001 C CNN
+F 4 "732-7971-1-ND" H 2950 8050 60  0001 C CNN "Part"
+F 5 "DigiKey" H 2950 8050 60  0001 C CNN "Provider"
+	1    2950 8050
+	1    0    0    -1
+$EndComp
+$Comp
+L sigmadrone:PGND #PWR035
+U 1 1 5CD3C239
+P 2950 8400
+F 0 "#PWR035" H 2950 8150 50  0001 C CNN
+F 1 "PGND" H 2955 8227 50  0000 C CNN
+F 2 "" H 2950 8400 50  0001 C CNN
+F 3 "" H 2950 8400 50  0001 C CNN
+	1    2950 8400
+	1    0    0    -1
+$EndComp
+Wire Wire Line
+	2950 7900 2950 7750
+Connection ~ 2950 7750
+Wire Wire Line
+	2950 7750 2600 7750
+Wire Wire Line
+	2950 8200 2950 8400
 $EndSCHEMATC

Commit message: Added second net-tie between GND and PGND.
Parts:
- added NT3: Net-Tie_2, NetTie:NetTie-2_SMD_Pad0.5mm, symbol Device:Net-Tie_2
Connections:
- wire segments 293 -> 297
Changed lines of the file:
@@
 $EndComp
 Wire Wire Line
-	6900 7100 6900 7400
+	6900 7100 6900 7250
 $Comp
 L sigmadrone:VIN #PWR?
@@
 $EndComp
 Wire Wire Line
-	7450 7100 7450 7400
+	7450 7100 7450 7250
 $Comp
 L Device:R R?
@@
 L Device:Net-Tie_2 NT1
 U 1 1 5D4D5931
-P 7200 7400
-F 0 "NT1" H 7200 7578 50  0000 C CNN
-F 1 "Net-Tie_2" H 7200 7487 50  0000 C CNN
-F 2 "NetTie:NetTie-2_SMD_Pad0.5mm" H 7200 7400 50  0001 C CNN
-F 3 "~" H 7200 7400 50  0001 C CNN
-	1    7200 7400
-	1    0    0    -1
-$EndComp
-Wire Wire Line
-	7100 7400 6900 7400
-Connection ~ 6900 7400
-Wire Wire Line
-	6900 7400 6900 7600
-Wire Wire Line
-	7300 7400 7450 7400
-Connection ~ 7450 7400
-Wire Wire Line
-	7450 7400 7450 7600
+P 7200 7250
+F 0 "NT1" H 7200 7428 50  0000 C CNN
+F 1 "Net-Tie_2" H 7200 7337 50  0000 C CNN
+F 2 "NetTie:NetTie-2_SMD_Pad0.5mm" H 7200 7250 50  0001 C CNN
+F 3 "~" H 7200 7250 50  0001 C CNN
+	1    7200 7250
+	1    0    0    -1
+$EndComp
+Wire Wire Line
+	7100 7250 6900 7250
+Connection ~ 6900 7250
+Wire Wire Line
+	6900 7250 6900 7500
+Wire Wire Line
+	7300 7250 7450 7250
+Connection ~ 7450 7250
+Wire Wire Line
+	7450 7250 7450 7500
 Wire Wire Line
 	1450 12550 3950 12550
@@
 Wire Wire Line
 	2950 8200 2950 8400
+$Comp
+L Device:Net-Tie_2 NT3
+U 1 1 5CBF51EC
+P 7200 7500
+F 0 "NT3" H 7200 7678 50  0000 C CNN
+F 1 "Net-Tie_2" H 7200 7587 50  0000 C CNN
+F 2 "NetTie:NetTie-2_SMD_Pad0.5mm" H 7200 7500 50  0001 C CNN
+F 3 "~" H 7200 7500 50  0001 C CNN
+	1    7200 7500
+	1    0    0    -1
+$EndComp
+Wire Wire Line
+	7300 7500 7450 7500
+Connection ~ 7450 7500
+Wire Wire Line
+	7450 7500 7450 7600
+Wire Wire Line
+	7100 7500 6900 7500
+Connection ~ 6900 7500
+Wire Wire Line
+	6900 7500 6900 7600
 $EndSCHEMATC

Commit message: Routed version 3.4
Parts:
- removed C26, C35: 100uF, Capacitor_SMD:CP_Elec_6.3x7.7, symbol Device:CP
- removed NT3: Net-Tie_2, NetTie:NetTie-2_SMD_Pad0.5mm, symbol Device:Net-Tie_2
- added C26, C35, C47, C48: 10uF 35V, Capacitor_SMD:C_1206_3216Metric, symbol Device:C
- added C50: 1uF 100V, Capacitor_SMD:C_0805_2012Metric, symbol Device:C
- added C56: 4.7uF 50V, Capacitor_SMD:C_0805_2012Metric, symbol Device:C
- added D8: BAT30KFILM, Diode_SMD:D_SOD-523, symbol Device:D_Shockley
- added FB3, FB4: 0.6OHM/0.2A/2.2 kOhm, Resistor_SMD:R_0603_1608Metric, symbol Device:Ferrite_Bead
- added JP1, JP2: Jumper_2_Open, Jumper:SolderJumper-2_P1.3mm_Open_TrianglePad1.0x1.5mm, symbol Jumper:Jumper_2_Open
- added R36, R41: N/A, Resistor_SMD:R_0603_1608Metric, symbol Device:R
- added R39: 0, Resistor_SMD:R_0603_1608Metric, symbol Device:R
- added TP10: PAD, TestPoint:TestPoint_Pad_D1.0mm, symbol Connector:TestPoint_Probe
- added U7: TPS70933, Package_TO_SOT_SMD:SOT-23-5, symbol sigmadrive-solo-rescue:TPS793333-EP-regul
Connections:
- wire segments 297 -> 336
- no-connect marks 21 -> 23

Commit message: Review from ZEK.
Parts:
- removed C47, C48: 10uF 35V, Capacitor_SMD:C_1206_3216Metric, symbol Device:C
- removed C50: 1uF 100V, Capacitor_SMD:C_0805_2012Metric, symbol Device:C
- removed C56: 4.7uF 50V, Capacitor_SMD:C_0805_2012Metric, symbol Device:C
- removed D8: BAT30KFILM, Diode_SMD:D_SOD-523, symbol Device:D_Shockley
- removed FB3, FB4: 0.6OHM/0.2A/2.2 kOhm, Resistor_SMD:R_0603_1608Metric, symbol Device:Ferrite_Bead
- removed JP1, JP2: Jumper_2_Open, Jumper:SolderJumper-2_P1.3mm_Open_TrianglePad1.0x1.5mm, symbol Jumper:Jumper_2_Open
- removed R36: N/A, Resistor_SMD:R_0603_1608Metric, symbol Device:R
- removed R39: 0, Resistor_SMD:R_0603_1608Metric, symbol Device:R
- removed TP10: PAD, TestPoint:TestPoint_Pad_D1.0mm, symbol Connector:TestPoint_Probe
- removed U7: TPS70933, Package_TO_SOT_SMD:SOT-23-5, symbol sigmadrive-solo-rescue:TPS793333-EP-regul
- added NT3: Net-Tie_2, NetTie:NetTie-2_SMD_Pad0.5mm, symbol Device:Net-Tie_2
Connections:
- wire segments 336 -> 306
- no-connect marks 23 -> 21
