File: hardware/sigmadrive-duo/mosfets_driving.sch (KiCad schematic (older format))
At the start: 105 parts, among them M1 Conn_01x04, M2 Conn_01x04, Q1 NTMFS5C628NLT1G, Q10 NTMFS5C628NLT1G, Q11 NTMFS5C628NLT1G, Q12 NTMFS5C628NLT1G, Q2 NTMFS5C628NLT1G, Q3 NTMFS5C628NLT1G, Q4 NTMFS5C628NLT1G, Q5 NTMFS5C628NLT1G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

Commit message: Work on duo drive.
Parts:
- removed R11, R12: 21, Resistor_SMD:R_0603_1608Metric, symbol Device:R
- removed R6: 10k, Resistor_SMD:R_0603_1608Metric, symbol Device:R
Connections:
- net DRV_SDO: now also U1.29 (SDO), U2.29 (SDO)
Changed lines of the file:
@@
 	1    0    0    -1
 $EndComp
-Wire Wire Line
-	2250 3550 2250 3650
-Wire Wire Line
-	2250 3150 2250 3250
-$Comp
-L power:+3.3V #PWR020
-U 1 1 5CF217A6
-P 2250 3150
-F 0 "#PWR020" H 2250 3000 50  0001 C CNN
-F 1 "+3.3V" H 2265 3323 50  0000 C CNN
-F 2 "" H 2250 3150 50  0001 C CNN
-F 3 "" H 2250 3150 50  0001 C CNN
-	1    2250 3150
-	1    0    0    -1
-$EndComp
-$Comp
-L Device:R R?
-U 1 1 5CF2179F
-P 2250 3400
-AR Path="/58BE2779/5CF2179F" Ref="R?"  Part="1"
-AR Path="/58BF664D/5CF2179F" Ref="R6"  Part="1"
-F 0 "R6" V 2330 3400 50  0000 C CNN
-F 1 "10k" V 2250 3400 50  0000 C CNN
-F 2 "Resistor_SMD:R_0603_1608Metric" V 2180 3400 50  0001 C CNN
-F 3 "http://www.yageo.com.tw/exep/pages/download/literatures/PYu-R_INT-thick_7.pdf" H 2250 3400 50  0001 C CNN
-F 4 "311-10.0KHRCT-ND" V 2250 3400 60  0001 C CNN "Part"
-F 5 "DigiKey" V 2250 3400 60  0001 C CNN "Provider"
-	1    2250 3400
-	1    0    0    -1
-$EndComp
-Wire Wire Line
-	2250 9450 4300 9450
 $Comp
 L power:PWR_FLAG #FLG?
@@
 Wire Wire Line
 	6750 13250 6750 13550
-$Comp
-L Device:R R?
-U 1 1 5CD745A7
-P 4500 3650
-AR Path="/58BE2779/5CD745A7" Ref="R?"  Part="1"
-AR Path="/58BF664D/5CD745A7" Ref="R11"  Part="1"
-F 0 "R11" V 4550 3800 50  0000 C CNN
-F 1 "21" V 4500 3650 50  0000 C CNN
-F 2 "Resistor_SMD:R_0603_1608Metric" V 4430 3650 50  0001 C CNN
-F 3 "http://www.yageo.com.tw/exep/pages/download/literatures/PYu-R_INT-thick_7.pdf" H 4500 3650 50  0001 C CNN
-F 4 "311-21.0HRCT-ND" V 4500 3650 60  0001 C CNN "Part"
-F 5 "DigiKey" V 4500 3650 60  0001 C CNN "Provider"
-	1    4500 3650
-	0    -1   -1   0
-$EndComp
-Wire Wire Line
-	4800 3650 4650 3650
-Wire Wire Line
-	1850 3650 2250 3650
-Connection ~ 2250 3650
-Wire Wire Line
-	2250 3650 4350 3650
-$Comp
-L Device:R R?
-U 1 1 5CDB071A
-P 4450 9450
-AR Path="/58BE2779/5CDB071A" Ref="R?"  Part="1"
-AR Path="/58BF664D/5CDB071A" Ref="R12"  Part="1"
-F 0 "R12" V 4500 9600 50  0000 C CNN
-F 1 "21" V 4450 9450 50  0000 C CNN
-F 2 "Resistor_SMD:R_0603_1608Metric" V 4380 9450 50  0001 C CNN
-F 3 "http://www.yageo.com.tw/exep/pages/download/literatures/PYu-R_INT-thick_7.pdf" H 4450 9450 50  0001 C CNN
-F 4 "311-21.0HRCT-ND" V 4450 9450 60  0001 C CNN "Part"
-F 5 "DigiKey" V 4450 9450 60  0001 C CNN "Provider"
-	1    4450 9450
-	0    -1   -1   0
-$EndComp
-Wire Wire Line
-	4600 9450 4750 9450
 $Comp
 L Device:Net-Tie_2 NT1
@@
 Wire Wire Line
 	21250 14050 19850 14050
+Wire Wire Line
+	1850 3650 4800 3650
+Wire Wire Line
+	2250 9450 4750 9450
 $EndSCHEMATC

Commit message: Work on duo drive.
Parts:
- added R37, R51: 21, Resistor_SMD:R_0603_1608Metric, symbol Device:R
- added R52, R53: 0, Resistor_SMD:R_0603_1608Metric, symbol Device:R
Connections:
- net +3V3: now also R52.1; no longer C2.1, C7.1, U1.26 (VREF), U2.26 (VREF)
- net DRV_SDO: now also R37.1, R51.1; no longer U1.29 (SDO), U2.29 (SDO)
- net at C56.1, U7.5 (OUT): now also R53.2
- new net: R51.2, U1.29 (SDO)
- new net: R37.2, U2.29 (SDO)
- new net +3.3VA: C2.1, C7.1, R52.2, R53.1, U1.26 (VREF), U2.26 (VREF)
Other:
- moved on the sheet: C56, NT1

Commit message: PCB sigmadrive-duo, version 3.6
Parts:
- removed M2: Conn_01x04, Connector_Molex:Molex_Micro-Fit_3.0_43650-0400_1x04_P3.00mm_Horizontal, symbol Connector_Generic:Conn_01x04
- removed R37, R51: 21, Resistor_SMD:R_0603_1608Metric, symbol Device:R
- added C46, C67: 10uF 35V, Capacitor_SMD:C_0805_2012Metric, symbol Device:C
- added M2: Conn_01x03, Connector_Molex:Molex_Micro-Fit_3.0_43650-0300_1x03_P3.00mm_Horizontal, symbol Connector_Generic:Conn_01x03
- C26, C35, C47, C48: footprint Capacitor_SMD:C_1206_3216Metric -> Capacitor_SMD:C_0805_2012Metric
- M1: value Conn_01x04 -> Conn_01x03; footprint Connector_Molex:Molex_Micro-Fit_3.0_43650-0400_1x04_P3.00mm_Horizontal -> Connector_Molex:Molex_Micro-Fit_3.0_43650-0300_1x03_P3.00mm_Horizontal; symbol Connector_Generic:Conn_01x04 -> Connector_Generic:Conn_01x03
- R52: value 0 -> N/A
Connections:
- net +3V3: now also C46.1
- net +5V: now also C67.1
- net DRV_SDO: now also U1.29 (SDO), U2.29 (SDO)
- net GND: now also C46.2, C67.2
- net M1_A: now also M1.3 (Pin_3); no longer M1.4 (Pin_4)
- net M1_B: now also M1.2 (Pin_2); no longer M1.3 (Pin_3)
- net M1_C: now also M1.1 (Pin_1); no longer M1.2 (Pin_2)
- net M2_A: now also M2.3 (Pin_3)
- net M2_B: now also M2.2 (Pin_2)
- net M2_C: now also M2.1 (Pin_1)
- net PGND: no longer M1.1 (Pin_1)
Other:
- moved on the sheet: R13, R16, R18, R22
