File: hardware/sigmadrive-duo/mcu.sch (KiCad schematic (older format))
At the start: 87 parts, among them J10 Conn_01x03, J11 Conn_01x03, J12 Conn_02x05_Odd_Even, J2 CONN_02X05, J4 Conn_01x05, J6 629_105_150_921, J8 Conn_01x03, J9 Conn_01x03, SW1 SW_DIP_x04, SW2 SW_DIP_x04, U12 SN65HVD75DGKR, U3 SN65HVD75DGKR, U4 TPD4S009, U5 STM32F745VGTx, U6 TPD4S009, Y1 NX3225SA-12.000M-STD-CSR-1

Commit message: Work on duo drive.
Parts:
- removed SW1: SW_DIP_x04, Button_Switch_SMD:SW_DIP_SPSTx04_Slide_Copal_CHS-04A_W5.08mm_P1.27mm_JPin, symbol Switch:SW_DIP_x04
- added C4: 100nF 50V, Capacitor_SMD:C_0603_1608Metric, symbol Device:C
- added J1: Conn_02x05_Odd_Even, Connector_PinHeader_2.00mm:PinHeader_2x05_P2.00mm_Horizontal, symbol Connector_Generic:Conn_02x05_Odd_Even
- added R10, R25, R33, R48, R9: 10k, Resistor_SMD:R_0603_1608Metric, symbol Device:R
- added U8: SN65HVD75DGKR, Package_SO:SOIC-8_3.9x4.9mm_P1.27mm, symbol Interface_UART:MAX3485
Connections:
- net PA5 is gone; now on net M2_AL: U5.29 (ADC1_IN5/ADC2_IN5/DAC_OUT2/I2S1_CK/SPI1_SCK/TIM2_CH1/TIM2_ETR/TIM8_CH1N/USB_OTG_HS_ULPI_CK/PA5)
- net PA6 is gone; now on net M2_QUAD_A: U5.30 (ADC1_IN6/ADC2_IN6/DCMI_PIXCLK/SPI1_MISO/TIM13_CH1/TIM1_BKIN/TIM3_CH1/TIM8_BKIN/PA6)
- net PB10 is gone; now on net DRV_CLK: U5.46 (ETH_RX_ER/I2C2_SCL/I2S2_CK/SPI2_SCK/TIM2_CH3/USART3_TX/USB_OTG_HS_ULPI_D3/PB10)
- net PE7 is gone; now on net M2_QUAD_Z: U5.37 (PE7/FMC_D4/FMC_DA4/QUADSPI_BK2_IO0/TIM1_ETR/UART7_RX)
- net +3V3: now also SW2.3, C4.2, R25.1, R33.1, R48.1, R9.1, U8.8 (VCC); no longer SW2.2
- net +5V: now also J1.9 (Pin_9)
- net BOOT0: now also SW2.5
- net DIR: no longer U5.91 (CAN2_RX/DCMI_D10/ETH_PPS_OUT/FMC_SDCKE1/I2C1_SMBA/I2S1_SD/I2S3_SD/SPI1_MOSI/SPI3_MOSI/TIM3_CH2/USB_OTG_HS_ULPI_D7/PB5)
- net DRV_CAL: now also U5.44 (PE14/FMC_D11/FMC_DA11/SAI2_MCLK_B/SPI4_MOSI/TIM1_CH4); no longer U5.45 (PE15/FMC_D12/FMC_DA12/TIM1_BKIN)
- net DRV_CLK: no longer U5.78 (DCMI_D8/I2S3_CK/QUADSPI_BK1_IO1/SDMMC1_D2/SPI3_SCK/UART4_TX/USART3_TX/PC10)
- net DRV_SDI: now also U5.54 (I2S2_SD/RTC_REFIN/SPI2_MOSI/TIM12_CH2/TIM1_CH3N/TIM8_CH3N/USB_OTG_HS_DP/PB15); no longer U5.80 (DCMI_D9/I2S3_SD/SDMMC1_CK/SPI3_MOSI/SYS_TRACED3/UART5_TX/USART3_CK/PC12)
- net DRV_SDO: now also U5.53 (SPI2_MISO/TIM12_CH1/TIM1_CH2N/TIM8_CH2N/USART3_RTS/USB_OTG_HS_DM/PB14); no longer U5.79 (ADC1_EXTI11/ADC2_EXTI11/ADC3_EXTI11/DCMI_D4/QUADSPI_BK2_NCS/SDMMC1_D3/SPI3_MISO/UART4_RX/USART3_RX/PC11)
- net GATE1_ENABLE: now also U5.45 (PE15/FMC_D12/FMC_DA12/TIM1_BKIN); no longer U5.44 (PE14/FMC_D11/FMC_DA11/SAI2_MCLK_B/SPI4_MOSI/TIM1_CH4)
- net GND: now also SW2.2, C4.1, J1.1 (Pin_1), R10.2, U8.5 (GND); no longer SW2.3
- net M2_AL: no longer U5.31 (ADC1_IN7/ADC2_IN7/ETH_CRS_DV/ETH_RX_DV/FMC_SDNWE/I2S1_SD/SPI1_MOSI/TIM14_CH1/TIM1_CH1N/TIM3_CH2/TIM8_CH1N/PA7)
- net M2_QUAD_A: no longer U5.92 (CAN2_TX/CEC/DCMI_D5/FMC_SDNE1/I2C1_SCL/QUADSPI_BK1_NCS/TIM4_CH1/USART1_TX/PB6)
- net M2_QUAD_B: now also U5.31 (ADC1_IN7/ADC2_IN7/ETH_CRS_DV/ETH_RX_DV/FMC_SDNWE/I2S1_SD/SPI1_MOSI/TIM14_CH1/TIM1_CH1N/TIM3_CH2/TIM8_CH1N/PA7); no longer U5.93 (DCMI_VSYNC/FMC_NL/I2C1_SDA/TIM4_CH2/USART1_RX/PB7)
- net M2_QUAD_Z: no longer U5.88 (PD7/FMC_NE1/SPDIFRX_IN0/USART2_CK)
- net PA15: now also R85.1, U12.2 (~RE), U12.3 (DE)
- net PA4: no longer R36.2, RV2.2
- net PB4: no longer J4.3 (Pin_3)
- net PC4: now also R36.2, RV2.2
- net at U3.6 (A): now also J12.5 (Pin_5); no longer J12.7 (Pin_7)
- net at U3.7 (B): now also J12.7 (Pin_7); no longer J12.5 (Pin_5)
- net GPIO_CONF_1 renamed PE0
- net GPIO_CONF_2 renamed PE1
- net GPIO_CONF_3 renamed PE2
- net GPIO_CONF_4 renamed PE3
- net PE3: no longer SW2.5
- net PB14 renamed SW1
- net SW1: no longer U5.53 (SPI2_MISO/TIM12_CH1/TIM1_CH2N/TIM8_CH2N/USART3_RTS/USB_OTG_HS_DM/PB14)
- net PB15 renamed SW2
- net SW2: no longer U5.54 (I2S2_SD/RTC_REFIN/SPI2_MOSI/TIM12_CH2/TIM1_CH3N/TIM8_CH3N/USB_OTG_HS_DP/PB15)
- removed net PD4: R85.1, U12.2 (~RE), U12.3 (DE), U5.85 (PD4/FMC_NOE/USART2_RTS)
- net PD5 renamed M1_ENCODER_DI
- net M1_ENCODER_DI: now also U8.4 (DI); no longer U12.4 (DI)
- net PD6 renamed PC11
- net PC11: now also U5.79 (ADC1_EXTI11/ADC2_EXTI11/ADC3_EXTI11/DCMI_D4/QUADSPI_BK2_NCS/SDMMC1_D3/SPI3_MISO/UART4_RX/USART3_RX/PC11); no longer U5.87 (PD6/DCMI_D10/FMC_NWAIT/I2S3_SD/SAI1_SD_A/SPI3_MOSI/USART2_RX)
- new net: J1.5 (Pin_5), U8.6 (A)
- new net: J1.7 (Pin_7), U8.7 (B)
- new net M1_ENCODER_DE: R10.1, U5.85 (PD4/FMC_NOE/USART2_RTS), U8.2 (~RE), U8.3 (DE)
- new net M1_ENCODER_RO: R9.2, U5.87 (PD6/DCMI_D10/FMC_NWAIT/I2S3_SD/SAI1_SD_A/SPI3_MOSI/USART2_RX), U8.1 (RO)
- new net M1_QUAD_A: J1.4 (Pin_4), R33.2, U5.92 (CAN2_TX/CEC/DCMI_D5/FMC_SDNE1/I2C1_SCL/QUADSPI_BK1_NCS/TIM4_CH1/USART1_TX/PB6)
- new net M1_QUAD_B: J1.2 (Pin_2), R25.2, U5.93 (DCMI_VSYNC/FMC_NL/I2C1_SDA/TIM4_CH2/USART1_RX/PB7)
- new net M1_QUAD_Z: J1.6 (Pin_6), R48.2, U5.88 (PD7/FMC_NE1/SPDIFRX_IN0/USART2_CK)
- new net PB5: U5.91 (CAN2_RX/DCMI_D10/ETH_PPS_OUT/FMC_SDCKE1/I2C1_SMBA/I2S1_SD/I2S3_SD/SPI1_MOSI/SPI3_MOSI/TIM3_CH2/USB_OTG_HS_ULPI_D7/PB5)
- new net PC10: U12.4 (DI), U5.78 (DCMI_D8/I2S3_CK/QUADSPI_BK1_IO1/SDMMC1_D2/SPI3_SCK/UART4_TX/USART3_TX/PC10)
- new net PC12: U5.80 (DCMI_D9/I2S3_SD/SDMMC1_CK/SPI3_MOSI/SYS_TRACED3/UART5_TX/USART3_CK/PC12)
- new net PWM_IN: J4.3 (Pin_3)
- no-connect marks 34 -> 37
Other:
- note added: "Swapped in Duo\nPE14 <--> PE15\n"
- moved on the sheet: C5, C51, C52, D1, D4, D6, J12, J6, J8, J9, R1, R14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

Commit message: Work on duo drive.
Parts:
- removed J10, J11, J8, J9: Conn_01x03, Connector_PinHeader_2.54mm:PinHeader_1x03_P2.54mm_Horizontal, symbol Connector_Generic:Conn_01x03
- removed J4: Conn_01x05, Connector_PinHeader_2.54mm:PinHeader_1x05_P2.54mm_Horizontal, symbol Connector_Generic:Conn_01x05
- removed R37: 10k, Resistor_SMD:R_0603_1608Metric, symbol Device:R
- added C65, C66: 100nF 50V, Capacitor_SMD:C_0603_1608Metric, symbol Device:C
- added GPIO1: Conn_02x05_Odd_Even, Connector_PinHeader_2.00mm:PinHeader_2x05_P2.00mm_Horizontal, symbol Connector_Generic:Conn_02x05_Odd_Even
- added J1, J4, M1_SW1, M1_SW2, M2_SW1, M2_SW2: CONN_02X02, Connector_PinHeader_2.00mm:PinHeader_2x02_P2.00mm_Horizontal, symbol Connector_Generic:Conn_02x02_Odd_Even
- added J3, J5: Conn_02x03_Odd_Even, Connector_PinHeader_2.00mm:PinHeader_2x03_P2.00mm_Horizontal, symbol Connector_Generic:Conn_02x03_Odd_Even
- added R11, R49: 100, Resistor_SMD:R_0603_1608Metric, symbol Device:R
- added R12, R6: 10k, Resistor_SMD:R_0603_1608Metric, symbol Device:R
- added R54, R55: 21, Resistor_SMD:R_0603_1608Metric, symbol Device:R
- renumbered J12 to ENC1, J1 to ENC2
Connections:
- net PB11 is gone; now on net M2_QUAD_Z: U5.47 (ADC1_EXTI11/ADC2_EXTI11/ADC3_EXTI11/ETH_TX_EN/I2C2_SDA/TIM2_CH4/USART3_RX/USB_OTG_HS_ULPI_D4/PB11)
- net PB4 is gone; now on net M2_QUAD_A: U5.90 (I2S2_WS/SPI1_MISO/SPI2_NSS/SPI3_MISO/SYS_JTRST/TIM3_CH1/PB4)
- net PB5 is gone; now on net M2_QUAD_B: U5.91 (CAN2_RX/DCMI_D10/ETH_PPS_OUT/FMC_SDCKE1/I2C1_SMBA/I2S1_SD/I2S3_SD/SPI1_MOSI/SPI3_MOSI/TIM3_CH2/USB_OTG_HS_ULPI_D7/PB5)
- net SW1 is gone; now on net M2_SW1: C51.2, R17.2
- net SW2 is gone; now on net M2_SW2: C52.2, R28.2
- net +3.3VP: no longer C53.2, U5.21 (VDDA)
- net +3V3: now also J2.3 (Pin_3), R48.2; no longer J2.1 (Pin_1), R48.1
- net +5V: now also J1.3 (Pin_3), J4.3 (Pin_3), M1_SW1.3 (Pin_3), M1_SW2.3 (Pin_3), M2_SW1.3 (Pin_3), M2_SW2.3 (Pin_3), R12.1, R6.1
- net A_TERM_R120: now also J3.3 (Pin_3), J5.3 (Pin_3)
- net GND: now also J2.1 (Pin_1), GPIO1.1 (Pin_1), J1.1 (Pin_1), J3.1 (Pin_1), J4.1 (Pin_1), J5.1 (Pin_1), M1_SW1.1 (Pin_1), M1_SW2.1 (Pin_1), M2_SW1.1 (Pin_1), M2_SW2.1 (Pin_1), R11.2, R49.2; no longer J2.3 (Pin_3)
- net M1_QUAD_Z: now also R48.1; no longer R48.2
- net M2_AL: now also U5.31 (ADC1_IN7/ADC2_IN7/ETH_CRS_DV/ETH_RX_DV/FMC_SDNWE/I2S1_SD/SPI1_MOSI/TIM14_CH1/TIM1_CH1N/TIM3_CH2/TIM8_CH1N/PA7); no longer U5.29 (ADC1_IN5/ADC2_IN5/DAC_OUT2/I2S1_CK/SPI1_SCK/TIM2_CH1/TIM2_ETR/TIM8_CH1N/USB_OTG_HS_ULPI_CK/PA5)
- net M2_QUAD_A: no longer U5.30 (ADC1_IN6/ADC2_IN6/DCMI_PIXCLK/SPI1_MISO/TIM13_CH1/TIM1_BKIN/TIM3_CH1/TIM8_BKIN/PA6)
- net M2_QUAD_B: no longer U5.31 (ADC1_IN7/ADC2_IN7/ETH_CRS_DV/ETH_RX_DV/FMC_SDNWE/I2S1_SD/SPI1_MOSI/TIM14_CH1/TIM1_CH1N/TIM3_CH2/TIM8_CH1N/PA7)
- net M2_QUAD_Z: no longer U5.37 (PE7/FMC_D4/FMC_DA4/QUADSPI_BK2_IO0/TIM1_ETR/UART7_RX)
- net PA0: now also GPIO1.8 (Pin_8); no longer C42.1, R27.1
- net PA1: now also C42.1, R27.1; no longer C43.1, R29.1
- net PA10: now also R55.2
- net PA2: now also C43.1, R29.1; no longer C44.1, R31.1
- net PA3: now also C44.1, R31.1
- net PA9: now also R54.2
- net PC12: now also J3.6 (Pin_6), J5.6 (Pin_6)
- net PD0: now also J3.4 (Pin_4), J5.4 (Pin_4)
- net PD1: now also J3.2 (Pin_2), J5.2 (Pin_2)
- net PE0: now also J1.4 (Pin_4)
- net PE1: now also J1.2 (Pin_2)
- net PE2: now also GPIO1.10 (Pin_10)
- net PE3: now also GPIO1.9 (Pin_9)
- net PE4: now also GPIO1.7 (Pin_7)
- net PE5: now also GPIO1.5 (Pin_5)
- net PE6: now also GPIO1.3 (Pin_3)
- net at R38.1, R88.1, U12.7 (B): now also J3.5 (Pin_5), J5.5 (Pin_5)
- net PA4 renamed ADC1_IN4
- net ADC1_IN4: now also GPIO1.6 (Pin_6)
- net PD10 renamed M1_SW1
- net M1_SW1: now also C65.2, M1_SW1.2 (Pin_2), R6.2
- net PD11 renamed M1_SW2
- net M1_SW2: now also C66.2, M1_SW2.2 (Pin_2), R12.2
- net PD2 renamed M2_SW2
- net M2_SW2: now also M2_SW2.2 (Pin_2)
- net PD3 renamed M2_SW1
- net M2_SW1: now also M2_SW1.2 (Pin_2)
- new net: C65.1, R11.1
- new net: C66.1, R49.1
- new net: J4.2 (Pin_2), R54.1
- new net: J4.4 (Pin_4), R55.1
- new net +3.3VA: C53.2, U5.21 (VDDA)
- new net ADC1_IN6: GPIO1.2 (Pin_2), U5.30 (ADC1_IN6/ADC2_IN6/DCMI_PIXCLK/SPI1_MISO/TIM13_CH1/TIM1_BKIN/TIM3_CH1/TIM8_BKIN/PA6)
- new net PA5: GPIO1.4 (Pin_4), U5.29 (ADC1_IN5/ADC2_IN5/DAC_OUT2/I2S1_CK/SPI1_SCK/TIM2_CH1/TIM2_ETR/TIM8_CH1N/USB_OTG_HS_ULPI_CK/PA5)
- new net PE7: U5.37 (PE7/FMC_D4/FMC_DA4/QUADSPI_BK2_IO0/TIM1_ETR/UART7_RX)
- no-connect marks 37 -> 26
Other:
- moved on the sheet: C14, C19, C24, C42, C43, C44, C46, C49, C51, C52, C53, R17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

Commit message: Work on duo drive.
Parts:
- added R56, R57: 10k, Resistor_SMD:R_0603_1608Metric, symbol Device:R
Connections:
- net PB8 is gone; now on net M1_TIM_CH3: U5.95 (CAN1_RX/DCMI_D6/ETH_TXD3/I2C1_SCL/SDMMC1_D4/TIM10_CH1/TIM4_CH3/PB8)
- net +3V3: now also R56.2, R57.1
- net DRV_SDO: now also U5.18 (ADC1_IN13/ADC2_IN13/ADC3_IN13/ETH_TX_CLK/FMC_SDCKE0/I2S2_SD/SPI2_MOSI/USB_OTG_HS_ULPI_NXT/PC3); no longer U5.53 (SPI2_MISO/TIM12_CH1/TIM1_CH2N/TIM8_CH2N/USART3_RTS/USB_OTG_HS_DM/PB14)
- net M2_BL: now also U5.53 (SPI2_MISO/TIM12_CH1/TIM1_CH2N/TIM8_CH2N/USART3_RTS/USB_OTG_HS_DM/PB14); no longer U5.34 (ADC1_IN8/ADC2_IN8/ETH_RXD2/TIM1_CH2N/TIM3_CH3/TIM8_CH2N/UART4_CTS/USB_OTG_HS_ULPI_D1/PB0)
- net PB9: now also GPIO1.2 (Pin_2)
- net VBAT_ADC: now also U5.30 (ADC1_IN6/ADC2_IN6/DCMI_PIXCLK/SPI1_MISO/TIM13_CH1/TIM1_BKIN/TIM3_CH1/TIM8_BKIN/PA6); no longer U5.18 (ADC1_IN13/ADC2_IN13/ADC3_IN13/ETH_TX_CLK/FMC_SDCKE0/I2S2_SD/SPI2_MOSI/USB_OTG_HS_ULPI_NXT/PC3)
- net M1_TIM_CH3: now reaches ENC2.8 (Pin_8)
- net M1_TIM_CH3: now also R56.1
- net M2_TIM_CH3: now reaches ENC1.8 (Pin_8)
- net M2_TIM_CH3: now also U5.34 (ADC1_IN8/ADC2_IN8/ETH_RXD2/TIM1_CH2N/TIM3_CH3/TIM8_CH2N/UART4_CTS/USB_OTG_HS_ULPI_D1/PB0), R57.2
- removed net ADC1_IN6: GPIO1.2 (Pin_2), U5.30 (ADC1_IN6/ADC2_IN6/DCMI_PIXCLK/SPI1_MISO/TIM13_CH1/TIM1_BKIN/TIM3_CH1/TIM8_BKIN/PA6)
- no-connect marks 26 -> 22
Changed lines of the file:
@@
 Text HLabel 22300 3750 2    60   Input ~ 0
 M1_IB_FB
-Text HLabel 18100 7250 2    60   Input ~ 0
+Text HLabel 18100 4150 2    60   Input ~ 0
 VBAT_ADC
 Text Label 17800 4450 2    60   ~ 0
@@
 	1    0    0    -1
 $EndComp
-Text HLabel 17400 6750 2    60   Output ~ 0
+Text HLabel 18050 6750 2    60   Output ~ 0
 DRV_SDI
-Text HLabel 17400 6650 2    60   Input ~ 0
+Text HLabel 18050 7250 2    60   Input ~ 0
 DRV_SDO
-Text HLabel 18100 8350 2    60   Output ~ 0
+Text HLabel 18050 8350 2    60   Output ~ 0
 DRV2_CS
 Text HLabel 3500 6650 0    60   Output ~ 0
 DRV_CAL
-Text HLabel 18100 8450 2    60   Input ~ 0
+Text HLabel 18050 8450 2    60   Input ~ 0
 DRV_FAULT
 Text HLabel 3500 6750 0    60   Output ~ 0
@@
 Wire Wire Line
 	3800 8350 5900 8350
-Text HLabel 18100 8250 2    60   Output ~ 0
+Text HLabel 18050 8250 2    60   Output ~ 0
 DRV1_CS
 Wire Wire Line
@@
 	3500 6650 5900 6650
 Wire Wire Line
-	16100 6650 17400 6650
+	16100 7250 18050 7250
 Wire Wire Line
-	16100 6750 17400 6750
+	16100 6750 18050 6750
 $Comp
 L Device:LED D6
@@
 PWR_ON
 Wire Wire Line
-	16100 8350 18100 8350
+	16100 8350 18050 8350
 Wire Wire Line
-	16100 8250 18100 8250
+	16100 8250 18050 8250
 Wire Wire Line
-	16100 8450 18100 8450
+	16100 8450 18050 8450
 Wire Wire Line
 	16100 4550 17800 4550
@@
 NoConn ~ 16100 6550
 Wire Wire Line
-	16100 5250 18100 5250
+	16100 6650 18100 6650
 $Comp
 L Device:Varistor RV1
@@
 $EndComp
 Wire Wire Line
-	16100 7250 18100 7250
+	16100 4150 18100 4150
 Wire Wire Line
 	16100 3850 19300 3850
@@
 NoConn ~ 16600 12800
 Wire Wire Line
-	16100 6050 16500 6050
-Wire Wire Line
 	16100 6150 16500 6150
-NoConn ~ 16100 6050
-NoConn ~ 16100 6150
 Wire Wire Line
 	16100 5450 18100 5450
 Text HLabel 18100 5350 2    60   Output ~ 0
 M2_CL
-Text HLabel 18100 5250 2    60   Output ~ 0
+Text HLabel 18100 6650 2    60   Output ~ 0
 M2_BL
-Text HLabel 18100 4250 2    60   Output ~ 0
+Text HLabel 18050 4250 2    60   Output ~ 0
 M2_AL
 Wire Wire Line
-	16100 4250 18100 4250
-Text HLabel 18100 7550 2    60   Output ~ 0
+	16100 4250 18050 4250
+Text HLabel 18050 7550 2    60   Output ~ 0
 M2_AH
-Text HLabel 18100 7650 2    60   Output ~ 0
+Text HLabel 18050 7650 2    60   Output ~ 0
 M2_BH
-Text HLabel 18100 7750 2    60   Output ~ 0
+Text HLabel 18050 7750 2    60   Output ~ 0
 M2_CH
 Wire Wire Line
-	16100 7550 18100 7550
+	16100 7550 18050 7550
 Wire Wire Line
-	16100 7650 18100 7650
+	16100 7650 18050 7650
 Wire Wire Line
-	16100 7750 18100 7750
+	16100 7750 18050 7750
 $Comp
 L Device:R R?
@@
 Text Label 17800 3950 2    60   ~ 0
 ADC1_IN4
-Text Label 17800 4150 2    60   ~ 0
-ADC1_IN6
 Wire Wire Line
 	16100 3950 17800 3950
-Wire Wire Line
-	16100 4150 17800 4150
 $Comp
 L Connector_Generic:Conn_02x05_Odd_Even GPIO1
@@
 Text Label 17600 11700 2    60   ~ 0
 ADC1_IN4
-Text Label 17600 11900 2    60   ~ 0
-ADC1_IN6
 Wire Wire Line
 	17100 11700 17600 11700
-Wire Wire Line
-	17100 11900 17600 11900
 Text Label 17600 11600 2    60   ~ 0
 TIM5_CH1
@@
 Text Label 6750 10300 2    60   ~ 0
 M1_QUAD_Z
-NoConn ~ 4800 10200
 $Comp
 L power:PWR_FLAG #FLG0108
@@
 Wire Wire Line
 	5900 12650 6750 12650
-NoConn ~ 4850 12550
 Wire Wire Line
 	4800 10300 5900 10300
@@
 Wire Wire Line
 	5900 10300 6750 10300
+Text Label 17800 5250 2    60   ~ 0
+M2_TIM_CH3
+Wire Wire Line
+	16100 5250 17800 5250
+Text Label 17800 6050 2    60   ~ 0
+M1_TIM_CH3
+Wire Wire Line
+	16100 6050 17800 6050
+Text Label 6750 10200 2    60   ~ 0
+M1_TIM_CH3
+Wire Wire Line
+	4800 10200 6100 10200
+Text Label 6750 12550 2    60   ~ 0
+M2_TIM_CH3
+Wire Wire Line
+	4850 12550 6100 12550
+$Comp
+L Device:R R57
+U 1 1 5F901D96
+P 6100 12250
+F 0 "R57" V 6180 12250 50  0000 C CNN
+F 1 "10k" V 6100 12250 50  0000 C CNN
+F 2 "Resistor_SMD:R_0603_1608Metric" V 6030 12250 50  0001 C CNN
+F 3 "http://www.yageo.com.tw/exep/pages/download/literatures/PYu-R_INT-thick_7.pdf" H 6100 12250 50  0001 C CNN
+F 4 "311-10.0KHRCT-ND" V 6100 12250 60  0001 C CNN "Part"
+F 5 "DigiKey" V 6100 12250 60  0001 C CNN "Provider"
+	1    6100 12250
+	-1   0    0    -1
+$EndComp
+Wire Wire Line
+	5900 12000 6100 12000
+Wire Wire Line
+	6100 12000 6100 12100
+Connection ~ 5900 12000
+Wire Wire Line
+	6100 12400 6100 12550
+Connection ~ 6100 12550
+Wire Wire Line
+	6100 12550 6750 12550
+$Comp
+L Device:R R56
+U 1 1 5F994D74
+P 6100 9900
+F 0 "R56" V 6180 9900 50  0000 C CNN
+F 1 "10k" V 6100 9900 50  0000 C CNN
+F 2 "Resistor_SMD:R_0603_1608Metric" V 6030 9900 50  0001 C CNN
+F 3 "http://www.yageo.com.tw/exep/pages/download/literatures/PYu-R_INT-thick_7.pdf" H 6100 9900 50  0001 C CNN
+F 4 "311-10.0KHRCT-ND" V 6100 9900 60  0001 C CNN "Part"
+F 5 "DigiKey" V 6100 9900 60  0001 C CNN "Provider"
+	1    6100 9900
+	-1   0    0    1
+$EndComp
+Wire Wire Line
+	5900 9650 6100 9650
+Wire Wire Line
+	6100 9650 6100 9750
+Connection ~ 5900 9650
+Wire Wire Line
+	6100 10050 6100 10200
+Connection ~ 6100 10200
+Wire Wire Line
+	6100 10200 6750 10200
+Text Label 17600 11900 2    60   ~ 0
+PB9
+Wire Wire Line
+	17100 11900 17600 11900
 $EndSCHEMATC
