File: hardware/sigmadrive-duo/sigmadrive-duo.kicad_pcb (KiCad board)
At the start: 4 copper layers, 85 x 100 mm, 213 parts, among them J1 CONN_02X02, J2 CONN_02X05, J3 Conn_02x03_Odd_Even, J4 CONN_02X02, J5 Conn_02x03_Odd_Even, J6 629_105_150_921, M1 Conn_01x03, M1_SW1 CONN_02X02, M1_SW2 CONN_02X02, M2 Conn_01x03, M2_SW1 CONN_02X02, M2_SW2 CONN_02X02, Q1 NTMFS5C628NLT1G, Q10 NTMFS5C628NLT1G, Q11 NTMFS5C628NLT1G, Q12 NTMFS5C628NLT1G, Q2 NTMFS5C628NLT1G, Q3 NTMFS5C628NLT1G, Q4 NTMFS5C628NLT1G, Q5 NTMFS5C628NLT1G, Q6 NTMFS5C628NLT1G, Q7 NTMFS5C628NLT1G, Q8 NTMFS5C628NLT1G, Q9 NTMFS5C628NLT1G, SW2 SW_DIP_x04, U1 DRV8323RS, U12 SN65HVD75DGKR, U2 DRV8323RS, U3 SN65HVD75DGKR, U4 TPD4S009, U5 STM32F745VGTx, U6 TPD4S009, U7 TPS70933, U8 SN65HVD75DGKR, Y1 NX3225SA-12.000M-STD-CSR-1

Commit message: Hardware version 3.8. Adde support for external battery.
Parts:
- added BT2: Battery_Cell, Battery:Battery_Panasonic_CR1220-VCN_Vertical_CircularHoles, F.Cu at (69.4, 109.9)
- moved BT1 3.32 mm to (69.4, 114.3), turned to 0 degrees
- moved NT1 1.20 mm to (63.9, 112.8)
Routing:
- net GND: track 222.0 -> 213.3 mm
- net +BATT: track 146.8 -> 149.2 mm
